File: DATALOGGER_ADS_V1/DATALOGGER_ADS_V1.brd (EAGLE design)
At the start: 170 x 120 mm, 119 parts, among them IC1 OPA1632DR, IC10 DE10-NANO, IC11 RASPBERRY_PI_4, IC12 PCF8523, IC2 OPA1632DR, IC3 OPA1632DR, IC4 OPA1632DR, IC5 OPA1632DR, IC6 OPA1632DR, IC7 OPA1632DR, IC8 OPA1632DR, IC9 REF1004U, J1 22-29-2021, J2 22-29-2021, U1 OPA350EA/2K5, U2 OPA350EA/2K5, U3 ADS1178IPAPT

Commit message: tarjeta_v2
Parts:
- added C100, C75: 100uF, rcl:C1206
- added C101, C102, C104, C44, C48, C52, C56, C60, C64, C68, C72, C74, C76, C77, C79, C85, C89, C93, C97, C99: 0.1uF, rcl:C0603
- added C103, C105, C106, C107, C78, C80, C81, C82: 10uF, rcl:C0603
- added C42, C45, C46, C49, C50, C53, C54, C57, C58, C61, C62, C65, C66, C69, C70, C73, C83, C86, C87, C90, C91, C94, C95, C98: 2.7nF, rcl:C0603
- added C43, C47, C51, C55, C59, C63, C67, C71, C84, C88, C92, C96: 2.2nF, rcl:C0603
- added IC13, IC14, IC15, IC16, IC17, IC18, IC19, IC20, IC22, IC23, IC24, IC25: OPA1632DR, SamacSys_Parts:SOIC127P600X175-8N
- added IC21, IC26: REF1004U, burr-brown:SO08
- added R100, R101, R104, R106, R109, R110, R112, R113, R115, R116, R118, R119, R121, R122, R124, R125, R127, R128, R130, R131, R134, R136, R55, R56, R58, R59, R61, R62, R64, R65, R67, R68, R70, R71, R73, R74, R76, R77, R79, R80, R82, R83, R85, R86, R88, R89, R91, R92, R94, R95, R97, R98: 1K, rcl:R0603
- added R102, R111, R114, R117, R120, R123, R126, R129, R132, R57, R60, R63, R66, R69, R72, R75, R78, R81, R84, R87, R90, R93, R96, R99: 49.9, rcl:R0603
- added R103, R105, R108, R133, R135, R138: 100, rcl:R0603
- added R107, R137: 20K, rcl:R0603
- added U4, U5, U7, U8: OPA350EA/2K5, OPA350EA_2K5:DGK8_TEX
- added U6, U9: ADS1178IPAPT, ADS1178IPAPT:PAP64_TEX
Connections:
- new net AINN2_1: C43.2, R59.1, R60.1, U6.4
- new net AINN2_2: C47.2, R65.1, R66.1, U6.2
- new net AINN2_3: C51.2, R71.1, R72.1, U6.64
- new net AINN2_4: C55.2, R77.1, R78.1, U6.62
- new net AINN2_5: C59.2, R83.1, R84.1, U6.52
- new net AINN2_6: C63.2, R89.1, R90.1, U6.50
- new net AINN2_7: C67.2, R95.1, R96.1, U6.48
- new net AINN2_8: C71.2, R101.1, R102.1, U6.46
- new net AINN3_1: C84.2, R113.1, R114.1, U9.4
- new net AINN3_2: C88.2, R119.1, R120.1, U9.2
- new net AINN3_3: C92.2, R125.1, R126.1, U9.64
- new net AINN3_4: C96.2, R131.1, R132.1, U9.62
- new net AINN3_5: U9.52
- new net AINN3_6: U9.50
- new net AINN3_7: U9.48
- new net AINN3_8: U9.46
- new net AINP2_1: C43.1, R56.1, R57.1, U6.3
- new net AINP2_2: C47.1, R62.1, R63.1, U6.1
- new net AINP2_3: C51.1, R68.1, R69.1, U6.63
- new net AINP2_4: C55.1, R74.1, R75.1, U6.61
- new net AINP2_5: C59.1, R80.1, R81.1, U6.51
- new net AINP2_6: C63.1, R86.1, R87.1, U6.49
- new net AINP2_7: C67.1, R92.1, R93.1, U6.47
- new net AINP2_8: C71.1, R98.1, R99.1, U6.45
- new net AINP3_1: C84.1, R110.1, R111.1, U9.3
- new net AINP3_2: C88.1, R116.1, R117.1, U9.1
- new net AINP3_3: C92.1, R122.1, R123.1, U9.63
- new net AINP3_4: C96.1, R128.1, R129.1, U9.61
- new net AINP3_5: U9.51
- new net AINP3_6: U9.49
- new net AINP3_7: U9.47
- new net AINP3_8: U9.45
- new net CLK2: U6.27
- new net CLK3: U9.27
- new net DOUT2_1: U6.20
- new net DOUT2_2: U6.19
- new net DOUT2_3: U6.18
- new net DOUT2_4: U6.17
- new net DOUT2_5: U6.16
- new net DOUT2_6: U6.15
- new net DOUT2_7: U6.14
- new net DOUT2_8: U6.13
- new net DOUT3_1: U9.20
- new net DOUT3_2: U9.19
- new net DOUT3_3: U9.18
- new net DOUT3_4: U9.17
- new net DOUT3_5: U9.16
- new net DOUT3_6: U9.15
- new net DOUT3_7: U9.14
- new net DOUT3_8: U9.13
- new net DRDY2: U6.29
- new net DRDY3: U9.29
- new net INPUT10+: R61.2
- new net INPUT10-: R64.2
- new net INPUT11+: R67.2
- new net INPUT11-: R70.2
- new net INPUT12+: R73.2
- new net INPUT12-: R76.2
- new net INPUT13+: R79.2
- new net INPUT13-: R82.2
- new net INPUT14+: R85.2
- new net INPUT14-: R88.2
- new net INPUT15+: R91.2
- new net INPUT15-: R94.2
- new net INPUT16+: R97.2
- new net INPUT16-: R100.2
- new net INPUT17+: R109.2
- new net INPUT17-: R112.2
- new net INPUT18+: R115.2
- new net INPUT18-: R118.2
- new net INPUT19+: R121.2
- new net INPUT19-: R124.2
- new net INPUT20+: R127.2
- new net INPUT20-: R130.2
- new net INPUT9+: R55.2
- new net INPUT9-: R58.2
- new net N$100: C101.2, R135.1, U7.6
- new net N$101: R138.1, U8.2, U8.6
- new net N$40: C42.1, IC13.8, R55.1, R56.2
- new net N$41: C42.2, IC13.5, R57.2
- new net N$42: C45.1, IC13.1, R58.1, R59.2
- new net N$43: C45.2, IC13.4, R60.2
- new net N$44: C46.1, IC14.8, R61.1, R62.2
- new net N$45: C46.2, IC14.5, R63.2
- new net N$46: C49.1, IC14.1, R64.1, R65.2
- new net N$47: C49.2, IC14.4, R66.2
- new net N$48: C50.1, IC15.8, R67.1, R68.2
- new net N$49: C50.2, IC15.5, R69.2
- new net N$50: C53.1, IC15.1, R70.1, R71.2
- new net N$51: C53.2, IC15.4, R72.2
- new net N$52: C54.1, IC16.8, R73.1, R74.2
- new net N$53: C54.2, IC16.5, R75.2
- new net N$54: C57.1, IC16.1, R76.1, R77.2
- new net N$55: C57.2, IC16.4, R78.2
- new net N$56: C58.1, IC17.8, R79.1, R80.2
- new net N$57: C58.2, IC17.5, R81.2
- new net N$58: C61.1, IC17.1, R82.1, R83.2
- new net N$59: C61.2, IC17.4, R84.2
- new net N$60: C62.1, IC18.8, R85.1, R86.2
- new net N$61: C62.2, IC18.5, R87.2
- new net N$62: C65.1, IC18.1, R88.1, R89.2
- new net N$63: C65.2, IC18.4, R90.2
- new net N$64: C66.1, IC19.8, R91.1, R92.2
- new net N$65: C66.2, IC19.5, R93.2
- new net N$66: C69.1, IC19.1, R94.1, R95.2
- new net N$67: C69.2, IC19.4, R96.2
- new net N$68: C70.1, IC20.8, R97.1, R98.2
- new net N$69: C70.2, IC20.5, R99.2
- new net N$70: C73.1, IC20.1, R100.1, R101.2
- new net N$71: C73.2, IC20.4, R102.2
- new net N$72: R103.2, U4.3
- new net N$73: C74.1, C75.1, R103.1, R104.2
- new net N$74: IC21.6, R104.1
- new net N$75: IC21.8, R107.1
- new net N$76: C76.1, R106.1, U4.2
- new net N$77: C76.2, R105.1, U4.6
- new net N$78: R108.1, U5.2, U5.6
- new net N$79: C83.1, IC22.8, R109.1, R110.2
- new net N$80: C83.2, IC22.5, R111.2
- new net N$81: C86.1, IC22.1, R112.1, R113.2
- new net N$82: C86.2, IC22.4, R114.2
- new net N$83: C87.1, IC23.8, R115.1, R116.2
- new net N$84: C87.2, IC23.5, R117.2
- new net N$85: C90.1, IC23.1, R118.1, R119.2
- new net N$86: C90.2, IC23.4, R120.2
- new net N$87: C91.1, IC24.8, R121.1, R122.2
- new net N$88: C91.2, IC24.5, R123.2
- new net N$89: C94.1, IC24.1, R124.1, R125.2
- new net N$90: C94.2, IC24.4, R126.2
- new net N$91: C95.1, IC25.8, R127.1, R128.2
- new net N$92: C95.2, IC25.5, R129.2
- new net N$93: C98.1, IC25.1, R130.1, R131.2
- new net N$94: C98.2, IC25.4, R132.2
- new net N$95: R133.2, U7.3
- new net N$96: C100.1, C99.1, R133.1, R134.2
- new net N$97: IC26.6, R134.1
- new net N$98: IC26.8, R137.1
- new net N$99: C101.1, R136.1, U7.2
- new net SCLK2: U6.28
- new net SCLK3: U9.28
- new net SYNC2: U6.11
- new net SYNC3: U9.11
- new net VCOM2: C44.1, C48.1, C52.1, C56.1, C60.1, C64.1, C68.1, C72.1, IC13.2, IC14.2, IC15.2, IC16.2, IC17.2, IC18.2, IC19.2, IC20.2, R108.2
- new net VCOM3: C85.1, C89.1, C93.1, C97.1, IC22.2, IC23.2, IC24.2, IC25.2, R138.2
- new net VCOMM2: C79.1, U5.3, U6.55
- new net VCOMM3: C104.1, U8.3, U9.55
- new net VREFN2: C77.2, C78.2, U6.57
- new net VREFN3: C102.2, C103.2, U9.57
- new net VREFP2: C77.1, C78.1, R105.2, R106.2, U6.56
- new net VREFP3: C102.1, C103.1, R135.2, R136.2, U9.56
- net +12V: now also IC13.3, IC14.3, IC15.3, IC16.3, IC17.3, IC18.3, IC19.3, IC20.3, IC22.3, IC23.3, IC24.3, IC25.3
- net +1V8: now also C107.1, C82.1, U6.26, U9.26
- net +3V3: now also C106.1, C81.1, U6.10, U6.22, U6.23, U6.31, U6.35, U6.36, U6.37, U6.38, U6.39, U6.40, U6.41, U6.42, U9.10, U9.22, U9.23, U9.31, U9.35, U9.36, U9.37, U9.38, U9.39, U9.40, U9.41, U9.42
- net +5V: now also C105.1, C80.1, R107.2, R137.2, U4.7, U5.7, U6.44, U6.5, U6.53, U6.60, U7.7, U8.7, U9.44, U9.5, U9.53, U9.60
- net -12V: now also IC13.6, IC14.6, IC15.6, IC16.6, IC17.6, IC18.6, IC19.6, IC20.6, IC22.6, IC23.6, IC24.6, IC25.6
- net GND: now also C100.2, C104.2, C105.2, C106.2, C107.2, C44.2, C48.2, C52.2, C56.2, C60.2, C64.2, C68.2, C72.2, C74.2, C75.2, C79.2, C80.2, C81.2, C82.2, C85.2, C89.2, C93.2, C97.2, C99.2, IC21.4, IC26.4, U4.4, U5.4, U6.12, U6.21, U6.24, U6.25, U6.30, U6.32, U6.34, U6.43, U6.54, U6.58, U6.59, U6.6, U6.7, U6.8, U6.9, U6.EPAD, U7.4, U8.4, U9.12, U9.21, U9.24, U9.25, U9.30, U9.32, U9.34, U9.43, U9.54, U9.58, U9.59, U9.6, U9.7, U9.8, U9.9, U9.EPAD

Commit message: tarjeta_v3
Parts:
- removed JP5: (no value), pinhead:2X04
- removed JP7: (no value), pinhead:2X05
- added IC27: D36V28F5-5V-3.2A, myProyects:D36V28F5-5V-3.2A
- added IC28: D24V5F1-1.8V-500MA, myProyects:D24V5F1
- added IC29: D24V10F3-3.3V-1A, myProyects:D24V10F3-3.3V-1A
- added IC30: D24V25F5-5V-2.5A, myProyects:D24V25F5-5V-2.5A
- added J3: 1985027, SamacSys_Parts:1985027
- added J4: 1989764, 1989764:CONN_1989764_PXC
- added J5: 1755736, 1755736:CONN_1924305
- moved JP6 145.6 mm to (5.35, 121.7), turned to 270 degrees
- moved JP4 127.9 mm to (27.8, 133.7), flipped to the top
- moved IC12 125.0 mm to (105.5, 118.4), turned to 180 degrees
- moved R56 71.5 mm to (13.8, -23.3), turned to 90 degrees
- moved R57 69.4 mm to (11.4, -23.3), turned to 90 degrees
- moved C42 69.4 mm to (11.3, -14.9), turned to 180 degrees
- moved IC13 64.7 mm to (9.03, -18.9)
- moved C43 62.8 mm to (9.07, -23.4), turned to 90 degrees
- moved R58 61.3 mm to (7.25, -12.2), turned to 90 degrees
- moved R60 59.8 mm to (6.67, -23.4), turned to 90 degrees
- moved R59 52.9 mm to (4.41, -23.4), turned to 90 degrees
- moved C44 50.8 mm to (4.14, -17.4), turned to 90 degrees
- moved R55 49.5 mm to (10.8, -12.2), turned to 90 degrees
- moved C45 47.2 mm to (6.75, -15.0)
- moved IC14 32.3 mm to (-14.5, -19.2)
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Other:
- board size 170 x 120 mm -> 170 x 140 mm

Commit message: tarjeta_v4
Parts:
- added C108, C109, C110, C111: (no value), rcl:C0805
- added IC31, IC32, IC33, IC34: TLV2771CDBVR, SamacSys_Parts:SOT95P280X145-5N
- added IC35, IC36, IC37, IC38, IC39, IC40, IC41, IC42: FODM217DV, SamacSys_Parts:SOIC127P700X220-4N
- added R139, R140, R141, R142: (no value), rcl:R0603
- added R143, R144, R145, R146, R147, R148, R149, R150, R151, R152, R153, R154, R155, R156, R157, R158, R159, R160, R161, R162: (no value), rcl:R0805
Connections:
- new net 3.3V_RPI: IC12.2, JP1.1
- new net 5V_2.5A: J2.1
- new net 5V_3.2A: J1.1
- new net DOBLE1: C108.1, IC31.4, J4.1, R143.2
- new net DOBLE2: C109.1, IC32.4, J4.2, R144.2
- new net DOBLE3: C110.1, IC33.4, J4.3, R145.2
- new net DOBLE4: C111.1, IC34.4, J4.4, R146.2
- new net GPIO0_0: JP3.1
- new net GPIO0_1: JP3.2
- new net GPIO0_10: JP3.13
- new net GPIO0_11: JP3.14
- new net GPIO0_12: JP3.15
- new net GPIO0_13: JP3.16
- new net GPIO0_14: JP3.17
- new net GPIO0_15: JP3.18
- new net GPIO0_16: JP3.19
- new net GPIO0_17: JP3.20
- new net GPIO0_18: JP3.21
- new net GPIO0_19: JP3.22
- new net GPIO0_2: JP3.3
- new net GPIO0_20: JP3.23
- new net GPIO0_21: JP3.24
- new net GPIO0_22: JP3.25
- new net GPIO0_23: JP3.26
- new net GPIO0_24: JP3.27
- new net GPIO0_25: JP3.28
- new net GPIO0_26: JP3.31
- new net GPIO0_27: JP3.32
- new net GPIO0_28: JP3.33
- new net GPIO0_29: JP3.34
- new net GPIO0_3: JP3.4
- new net GPIO0_30: JP3.35
- new net GPIO0_31: JP3.36
- new net GPIO0_32: JP3.37
- new net GPIO0_33: JP3.38
- new net GPIO0_34: JP3.39
- new net GPIO0_35: JP3.40
- new net GPIO0_4: JP3.5
- new net GPIO0_5: JP3.6
- new net GPIO0_6: JP3.7
- new net GPIO0_7: JP3.8
- new net GPIO0_8: JP3.9
- new net GPIO0_9: JP3.10
- new net GPIO10: JP1.19
- new net GPIO17: JP1.11, R140.1
- new net GPIO1_0: JP2.1
- new net GPIO1_1: JP2.2
- new net GPIO1_10: JP2.13
- new net GPIO1_11: JP2.14
- new net GPIO1_12: JP2.15
- new net GPIO1_13: JP2.16
- new net GPIO1_14: JP2.17
- new net GPIO1_15: JP2.18
- new net GPIO1_16: JP2.19
- new net GPIO1_17: JP2.20
- new net GPIO1_18: JP2.21
- new net GPIO1_19: JP2.22
- new net GPIO1_2: JP2.3
- new net GPIO1_20: JP2.23
- new net GPIO1_21: JP2.24
- new net GPIO1_22: JP2.25
- new net GPIO1_23: JP2.26
- new net GPIO1_24: JP2.27
- new net GPIO1_25: JP2.28
- new net GPIO1_26: JP2.31
- new net GPIO1_27: JP2.32
- new net GPIO1_28: JP2.33
- new net GPIO1_29: JP2.34
- new net GPIO1_3: JP2.4
- new net GPIO1_30: JP2.35
- new net GPIO1_31: JP2.36
- new net GPIO1_32: JP2.37
- new net GPIO1_33: JP2.38
- new net GPIO1_34: JP2.39
- new net GPIO1_35: JP2.40
- new net GPIO1_4: JP2.5
- new net GPIO1_5: JP2.6
- new net GPIO1_6: JP2.7
- new net GPIO1_7: JP2.8
- new net GPIO1_8: JP2.9
- new net GPIO1_9: JP2.10
- new net GPIO22: JP1.15, R142.1
- new net GPIO27: JP1.13, R141.1
- new net GPIO4: JP1.7, R139.1
- new net GPIO9: JP1.21
- new net LAZO1: IC35.4, R148.1
- new net LAZO2: IC36.4, R150.1
- new net LAZO3: IC37.4, R152.1
- new net LAZO4: IC38.4, R154.1
- new net LAZO5: IC39.4, R156.1
- new net LAZO6: IC40.4, R158.1
- new net LAZO7: IC41.4, R160.1
- new net LAZO8: IC42.4, R162.1
- new net LOOP1: IC35.2, J3.1
- new net LOOP2: IC36.2, J3.2
- new net LOOP3: IC37.2, J3.3
- new net LOOP4: IC38.2, J3.4
- new net LOOP5: IC39.2, J3.5
- new net LOOP6: IC40.2, J3.6
- new net LOOP7: IC41.2, J3.7
- new net LOOP8: IC42.2, J3.8
- new net N$102: IC35.1, R147.2
- new net N$104: IC36.1, R149.2
- new net N$105: JP4.35, JP4.39
- new net N$106: JP6.1, R139.2
- new net N$107: JP6.3, R140.2
- new net N$108: JP6.5, R141.2
- new net N$109: JP6.7, R142.2
- new net N$110: JP4.33, JP4.37
- new net N$112: IC37.1, R151.2
- new net N$114: JP4.36, JP4.40
- new net N$115: JP4.34, JP4.38
- new net N$116: IC38.1, R153.2
- new net N$118: IC39.1, R155.2
- new net N$120: IC40.1, R157.2
- new net N$122: IC41.1, R159.2
- new net N$124: IC42.1, R161.2
- new net RX: JP1.10
- new net SCL: IC12.4, JP1.5
- new net SDA: IC12.3, JP1.3
- new net SQW: IC12.5
- new net TX: JP1.8
- net +3V3: now also R148.2, R150.2, R152.2, R154.2, R156.2, R158.2, R160.2, R162.2
- net +5V: now also IC31.5, IC32.5, IC33.5, IC34.5, R147.1, R149.1, R151.1, R153.1, R155.1, R157.1, R159.1, R161.1
- net GND: now also IC12.1, IC31.2, IC31.3, IC32.2, IC32.3, IC33.2, IC33.3, IC34.2, IC34.3, IC35.3, IC36.3, IC37.3, IC38.3, IC39.3, IC40.3, IC41.3, IC42.3, J1.2, J2.2, JP1.14, JP1.20, JP1.25, JP1.30, JP1.34, JP1.39, JP1.6, JP1.9, JP2.12, JP2.30, JP3.12, JP3.30, JP6.2, JP6.4, JP6.6, JP6.8
- net INPUT1+: now also JP4.1
- net INPUT1-: now also JP4.2
- net INPUT10+: now also JP4.19
- net INPUT10-: now also JP4.20
- net INPUT11+: now also JP4.21
- net INPUT11-: now also JP4.22
- net INPUT12+: now also JP4.23
- net INPUT12-: now also JP4.24
- net INPUT13+: now also JP4.25
- net INPUT13-: now also JP4.26
- net INPUT14+: now also JP4.27
- net INPUT14-: now also JP4.28
- net INPUT15+: now also JP4.29
- net INPUT15-: now also JP4.30
- net INPUT16+: now also JP4.31
- net INPUT16-: now also JP4.32
- net INPUT17+: now also C108.2, IC31.1, R143.1
- net INPUT18+: now also C109.2, IC32.1, R144.1
- net INPUT19+: now also C110.2, IC33.1, R145.1
- net INPUT2+: now also JP4.3
- net INPUT2-: now also JP4.4
- net INPUT20+: now also C111.2, IC34.1, R146.1
- net INPUT3+: now also JP4.5
- net INPUT3-: now also JP4.6
- net INPUT4+: now also JP4.7
- net INPUT4-: now also JP4.8
- net INPUT5+: now also JP4.9
- net INPUT5-: now also JP4.10
- net INPUT6+: now also JP4.11
- net INPUT6-: now also JP4.12
- net INPUT7+: now also JP4.13
- net INPUT7-: now also JP4.14
- net INPUT8+: now also JP4.15
- net INPUT8-: now also JP4.16
- net INPUT9+: now also JP4.17
- net INPUT9-: now also JP4.18

Commit message: tarjeta_v5
Parts:
- added C112: 10uF, rcl:C1206
- added C113: 22uF, rcl:C1206
- added IC43: D24V25F5-5V-2.5A, myProyects:D24V25F5-5V-2.5A
- added U$4: D36V6F12-12V-600MA, myProyects:D36V6F12-12V-600MA
- added U10: VXO78012-500, VXO78012-500:CONV_VXO78012-500
Connections:
- new net +24V: C112.1, IC27.3, IC28.2, IC29.3, IC30.VIN, IC43.VIN, J5.1, U$4.2, U10.1
- net +12V: now also U$4.4
- net +1V8: now also IC28.4
- net +3V3: now also IC29.5
- net +5V: now also IC43.VOUT
- net -12V: now also C113.2, U10.2
- net 5V_2.5A: now also IC30.VOUT
- net 5V_3.2A: now also IC27.6
- net GND: now also C112.2, C113.1, IC27.4, IC27.5, IC28.3, IC29.4, IC30.GND@3, IC30.GND@4, IC43.GND@3, IC43.GND@4, J5.2, U$4.3, U10.3

Commit message: tarjeta_v6
Parts:
- moved C112 580.7 mm to (104.3, 134.4)
- moved C113 576.8 mm to (103.3, 126.5)
- moved IC42 537.4 mm to (214.1, 46.0), turned to 90 degrees
- moved R162 536.3 mm to (213.4, 52.6), turned to 90 degrees
- moved IC41 532.2 mm to (209.9, 46.0), turned to 90 degrees
- moved R160 530.6 mm to (209.2, 52.6), turned to 90 degrees
- moved R161 528.0 mm to (213.4, 39.4), turned to 90 degrees
- moved R159 522.3 mm to (209.2, 39.3), turned to 90 degrees
- moved IC40 520.1 mm to (205.9, 46.0), turned to 90 degrees
- moved R158 519.0 mm to (205.2, 52.6), turned to 90 degrees
- moved IC39 515.1 mm to (201.9, 45.9), turned to 90 degrees
- moved R156 513.4 mm to (201.2, 52.6), turned to 90 degrees
- moved R157 510.6 mm to (205.2, 39.2), turned to 90 degrees
- moved R155 505.0 mm to (201.2, 39.2), turned to 90 degrees
- moved IC38 502.9 mm to (197.9, 45.9), turned to 90 degrees
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Routing:
- net +5V: track 29.8 -> 172.5 mm
- net +3V3: track 0.00 -> 94.6 mm
- net N$50: track 0.00 -> 18.8 mm
- net N$81: track 0.00 -> 18.5 mm
- net N$93: track 0.00 -> 18.5 mm
- net N$89: track 0.00 -> 18.4 mm
- net N$42: track 0.00 -> 18.3 mm
- net N$62: track 0.00 -> 18.2 mm
- net N$70: track 0.00 -> 18.2 mm
- net N$54: track 0.00 -> 18.1 mm
- net N$85: track 0.00 -> 17.9 mm
- net N$46: track 0.00 -> 16.3 mm
- net VCOM2: track 0.00 -> 16.0 mm
- net N$58: track 0.00 -> 15.3 mm
- net N$76: track 0.00 -> 14.1 mm
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
Commit message: tarjeta_v7
Parts:
- moved IC34 435.4 mm to (160.1, 30.1), turned to 270 degrees
- moved C111 432.8 mm to (160.2, 26.8)
- moved R146 427.5 mm to (160.2, 24.7), turned to 180 degrees
- moved IC33 422.3 mm to (154.2, 30.1), turned to 270 degrees
- moved C110 419.7 mm to (154.3, 26.8)
- moved R145 414.3 mm to (154.3, 24.6), turned to 180 degrees
- moved R142 414.2 mm to (9.85, 107.2), turned to 270 degrees
- moved IC32 409.3 mm to (148.7, 30.1), turned to 270 degrees
- moved R141 407.4 mm to (9.88, 103.8), turned to 90 degrees
- moved C109 406.7 mm to (148.8, 26.8)
- moved R144 401.3 mm to (148.8, 24.6), turned to 180 degrees
- moved R140 400.7 mm to (9.83, 100.5), turned to 90 degrees
- moved R143 394.3 mm to (142.5, 24.7), turned to 180 degrees
- moved R139 394.0 mm to (9.84, 97.2), turned to 90 degrees
- moved C108 392.7 mm to (142.5, 26.9)
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Connections:
- removed net INPUT17-: R112.2
- removed net INPUT18-: R118.2
- removed net INPUT19-: R124.2
- removed net INPUT20-: R130.2
- net GND: now also R112.2, R118.2, R124.2, R130.2
Routing:
- net +5V: track 172.5 -> 316.1 mm, vias 0 -> 3
- net +1V8: track 0.00 -> 132.4 mm, vias 0 -> 2
- net 5V_2.5A: track 0.00 -> 90.0 mm
- net INPUT8-: track 0.00 -> 85.7 mm
- net INPUT8+: track 0.00 -> 78.8 mm
- net INPUT6-: track 0.00 -> 75.5 mm
- net +3V3: track 94.6 -> 167.4 mm, vias 0 -> 1
- net +24V: track 0.00 -> 72.1 mm
- net INPUT6+: track 0.00 -> 69.0 mm
- net -12V: track 0.00 -> 68.1 mm, vias 0 -> 4
- net INPUT4-: track 0.00 -> 66.7 mm
- net INPUT2-: track 0.00 -> 62.9 mm
- net VCOM3: track 9.06 -> 70.5 mm, vias 0 -> 5
- net +12V: track 0.00 -> 60.5 mm, vias 0 -> 4
- net INPUT4+: track 0.00 -> 60.2 mm
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- added copper zone on layer 2, net GND
Other:
- board size 170 x 140 mm -> 170 x 130 mm
