File: DATALOGGER_ADS_V1/DATALOGGER_ADS_V1.brd (EAGLE design)
At the start: 170 x 130 mm, 339 parts, among them IC1 OPA1632DR, IC10 DE10-NANO, IC11 RASPBERRY_PI_4, IC12 PCF8523, IC13 OPA1632DR, IC14 OPA1632DR, IC15 OPA1632DR, IC16 OPA1632DR, IC17 OPA1632DR, IC18 OPA1632DR, IC19 OPA1632DR, IC2 OPA1632DR, IC20 OPA1632DR, IC21 REF1004U, IC22 OPA1632DR, IC23 OPA1632DR, IC24 OPA1632DR, IC25 OPA1632DR, IC26 REF1004U, IC27 D36V28F5-5V-3.2A, IC28 D24V5F1-1.8V-500MA, IC29 D24V10F3-3.3V-1A, IC3 OPA1632DR, IC30 D24V25F5-5V-2.5A, IC31 TLV2771CDBVR, IC32 TLV2771CDBVR, IC33 TLV2771CDBVR, IC34 TLV2771CDBVR, IC35 FODM217DV, IC36 FODM217DV, IC37 FODM217DV, IC38 FODM217DV, IC39 FODM217DV, IC4 OPA1632DR, IC40 FODM217DV, IC41 FODM217DV, IC42 FODM217DV, IC43 D24V25F5-5V-2.5A, IC5 OPA1632DR, IC6 OPA1632DR, IC7 OPA1632DR, IC8 OPA1632DR, IC9 REF1004U, J1 22-29-2021, J2 22-29-2021, J3 1985027, J4 1989764, J5 1755736, U1 OPA350EA/2K5, U10 VXO78012-500, U2 OPA350EA/2K5, U3 ADS1178IPAPT, U4 OPA350EA/2K5, U5 OPA350EA/2K5, U6 ADS1178IPAPT, U7 OPA350EA/2K5, U8 OPA350EA/2K5, U9 ADS1178IPAPT

Commit message: tarjeta_v9
Parts:
- moved C106 1.87 mm to (163.5, 60.6)
- moved C107 1.86 mm to (163.5, 62.7)
- moved C82 1.60 mm to (43.4, 35.7), turned to 270 degrees
- moved C41 0.67 mm to (41.4, 37.4)
- moved C80 0.22 mm to (54.1, 46.5)
Connections:
- net GPIO1_29 renamed LAZO_8
- removed net GPIO0_12: JP3.15
- removed net GPIO0_13: JP3.16
- removed net GPIO0_14: JP3.17
- removed net GPIO0_15: JP3.18
- removed net GPIO0_16: JP3.19
- removed net GPIO0_17: JP3.20
- removed net GPIO0_18: JP3.21
- removed net GPIO0_19: JP3.22
- removed net GPIO0_20: JP3.23
- removed net GPIO0_21: JP3.24
- removed net GPIO0_22: JP3.25
- removed net GPIO0_23: JP3.26
- removed net GPIO1_0: JP2.1
- removed net GPIO1_1: JP2.2
- removed net GPIO1_10: JP2.13
- removed net GPIO1_11: JP2.14
- removed net GPIO1_12: JP2.15
- removed net GPIO1_13: JP2.16
- removed net GPIO1_15: JP2.18
- removed net GPIO1_2: JP2.3
- removed net GPIO1_3: JP2.4
- removed net GPIO1_4: JP2.5
- removed net GPIO1_5: JP2.6
- removed net GPIO1_6: JP2.7
- removed net GPIO1_7: JP2.8
- removed net GPIO1_8: JP2.9
- removed net GPIO1_9: JP2.10
- removed net N$105: JP4.35, JP4.39
- removed net N$110: JP4.33, JP4.37
- removed net N$114: JP4.36, JP4.40
- removed net N$115: JP4.34, JP4.38
- net CLK2: now also JP3.24
- net CLK3: now also JP2.9
- net DOUT2_1: now also JP3.23
- net DOUT2_2: now also JP3.22
- net DOUT2_3: now also JP3.21
- net DOUT2_4: now also JP3.20
- net DOUT2_5: now also JP3.19
- net DOUT2_6: now also JP3.18
- net DOUT2_7: now also JP3.17
- net DOUT2_8: now also JP3.16
- net DOUT3_1: now also JP2.13
- net DOUT3_2: now also JP2.16
- net DOUT3_3: now also JP2.15
- net DOUT3_4: now also JP2.18
- net DRDY2: now also JP3.26
- net DRDY3: now also JP2.14
- net LAZO1: now also JP2.2
- net LAZO2: now also JP2.1
- net LAZO3: now also JP2.4
- net LAZO4: now also JP2.3
- net LAZO5: now also JP2.6
- net LAZO6: now also JP2.5
- net LAZO7: now also JP2.8
- net LAZO8: now also JP2.7
- net SCLK2: now also JP3.25
- net SCLK3: now also JP2.10
- net SYNC2: now also JP3.15
Routing:
- net +5V: track 409.0 -> 594.8 mm, vias 6 -> 9
- net GPIO17: track 0.00 -> 153.7 mm, vias 0 -> 1
- net GPIO4: track 0.00 -> 150.6 mm, vias 0 -> 1
- net GPIO27: track 0.00 -> 150.3 mm, vias 0 -> 1
- net DOUT3_4: track 0.00 -> 148.1 mm, vias 0 -> 4
- net GPIO22: track 0.00 -> 146.1 mm, vias 0 -> 1
- net DOUT3_1: track 0.00 -> 145.8 mm, vias 0 -> 1
- net DOUT3_2: track 0.00 -> 143.9 mm, vias 0 -> 1
- net DOUT3_3: track 0.00 -> 142.7 mm, vias 0 -> 1
- net CLK3: track 0.00 -> 128.5 mm, vias 0 -> 1
- net DRDY3: track 0.00 -> 125.7 mm, vias 0 -> 1
- net SCLK3: track 0.00 -> 124.1 mm, vias 0 -> 1
- net LAZO3: track 2.46 -> 101.7 mm, vias 0 -> 1
- net LAZO1: track 2.43 -> 100.6 mm, vias 0 -> 1
- net LAZO2: track 2.45 -> 99.1 mm, vias 0 -> 1
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
Commit message: tarjeta_v10
Parts:
- U$4: value D36V6F12-12V-600MA -> D24V22F12-12V-2.2A; device myProyects:D36V6F12-12V-600MA -> myProyects:D24V22F12
- moved J2 10.8 mm to (4.94, 5.47)
- moved J3 3.66 mm to (159.4, 123.8)
- moved U$4 2.58 mm to (78.1, 109.2)
- moved U10 2.19 mm to (104.6, 115.3)
- moved J4 0.54 mm to (164.3, 7.42)
Connections:
- net +12V: now also JP4.35, JP4.36, U$4.5; no longer U$4.4
- net +24V: now also U$4.3; no longer U$4.2
- net +5V: now also JP4.39, JP4.40
- net GND: now also JP4.33, JP4.34, JP4.37, JP4.38, U$4.4; no longer U$4.3
Routing:
- net +12V: track 670.7 -> 693.2 mm
- net +5V: track 594.8 -> 614.8 mm
- net 5V_2.5A: track 90.0 -> 83.8 mm
- net +24V: track 357.2 -> 361.2 mm
- net LOOP3: track 16.3 -> 20.0 mm
- net LOOP4: track 15.9 -> 19.6 mm
- net LOOP2: track 16.6 -> 20.4 mm
- net LOOP1: track 17.0 -> 20.7 mm
- net LOOP8: track 17.0 -> 20.6 mm
- net LOOP5: track 16.0 -> 19.6 mm
- net LOOP7: track 16.7 -> 20.3 mm
- net LOOP6: track 16.3 -> 19.9 mm
- net -12V: track 649.3 -> 650.9 mm
- net DOBLE2: track 27.0 -> 27.5 mm
- net DOBLE1: track 34.6 -> 35.2 mm
Other:
- board text added: "+24v"
- board text added: "1"
- board text added: "2"
- board text added: "3"
- board text added: "4"
- board text added: "5"
- board text added: "6"
- board text added: "7"
- board text added: "8"
- board text added: "GND"
- board text added: "LI"
- board text added: "SDR"
- board text added: "ver 1.0"

Commit message: tarjeta_v11
Parts:
- added J6: 22-29-2021, SamacSys_Parts:SHDR2W64P0X254_1X2_508X580X117
Connections:
- net +12V: now also J6.1
- net GND: now also J6.2
Routing:
- net +12V: track 693.2 -> 707.0 mm, vias 24 -> 25
Changed lines of the file:
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@@
 <?xml version="1.0" encoding="utf-8"?>
 <!DOCTYPE eagle SYSTEM "eagle.dtd">
-<eagle version="9.6.2">
+<eagle version="9.5.2">
 <drawing>
 <settings>
-<setting alwaysvectorfont="yes"/>
+<setting alwaysvectorfont="no"/>
 <setting verticaltext="up"/>
 </settings>
-<grid distance="1" unitdist="mil" unit="mil" style="lines" multiple="1" display="yes" altdistance="5" altunitdist="mil" altunit="mil"/>
+<grid distance="1" unitdist="mil" unit="mm" style="lines" multiple="1" display="yes" altdistance="5" altunitdist="mil" altunit="mil"/>
 <layers>
 <layer number="1" name="Top" color="4" fill="1" visible="yes" active="yes"/>
@@
 <attribute name="VALUE" x="98.72" y="107.86" size="1.27" layer="27"/>
 </element>
+<element name="J6" library="SamacSys_Parts" package="SHDR2W64P0X254_1X2_508X580X117" value="22-29-2021" x="5.0292" y="15.0876" smashed="yes">
+<attribute name="DESCRIPTION" value="Molex KK 254 6410, 2.54mm Pitch, 2 Way, 1 Row, Straight PCB Header, Through Hole" x="3.8354" y="15.0876" size="1.778" layer="27" display="off"/>
+<attribute name="HEIGHT" value="11.7mm" x="3.8354" y="15.0876" size="1.778" layer="27" display="off"/>
+<attribute name="MANUFACTURER_NAME" value="Molex" x="3.8354" y="15.0876" size="1.778" layer="27" display="off"/>
+<attribute name="MANUFACTURER_PART_NUMBER" value="22-29-2021" x="3.8354" y="15.0876" size="1.778" layer="27" display="off"/>
+<attribute name="MOUSER_PART_NUMBER" value="538-22-29-2021" x="3.8354" y="15.0876" size="1.778" layer="27" display="off"/>
+<attribute name="MOUSER_PRICE-STOCK" value="https://www.mouser.com/Search/Refine.aspx?Keyword=538-22-29-2021" x="3.8354" y="15.0876" size="1.778" layer="27" display="off"/>
+<attribute name="NAME" x="2.3622" y="17.78" size="0.6096" layer="25" align="center"/>
+<attribute name="VALUE" x="5.0292" y="15.0876" size="1.27" layer="27" align="center"/>
+</element>
 </elements>
 <signals>
@@
 <wire x1="48.06" y1="120.79" x2="48.06" y2="121.56" width="0.508" layer="1"/>
 <wire x1="48.06" y1="124.1" x2="48.06" y2="121.56" width="0.508" layer="1"/>
+<contactref element="J6" pad="1"/>
+<wire x1="5.0292" y1="15.0876" x2="10.7616" y2="20.82" width="0.508" layer="1"/>
+<wire x1="10.7616" y1="20.82" x2="16.41" y2="20.82" width="0.508" layer="1"/>
+<via x="16.41" y="20.82" extent="1-2" drill="0.35"/>
 </signal>
 <signal name="-12V">
@@
 <contactref element="JP4" pad="38"/>
 <contactref element="JP4" pad="37"/>
+<contactref element="J6" pad="2"/>
 </signal>
 <signal name="N$1">
