File: DATALOGGER_ADS_V1/DATALOGGER_ADS_V1.brd (EAGLE design)
At the start: 170 x 130 mm, 340 parts, among them IC1 OPA1632DR, IC10 DE10-NANO, IC11 RASPBERRY_PI_4, IC12 PCF8523, IC13 OPA1632DR, IC14 OPA1632DR, IC15 OPA1632DR, IC16 OPA1632DR, IC17 OPA1632DR, IC18 OPA1632DR, IC19 OPA1632DR, IC2 OPA1632DR, IC20 OPA1632DR, IC21 REF1004U, IC22 OPA1632DR, IC23 OPA1632DR, IC24 OPA1632DR, IC25 OPA1632DR, IC26 REF1004U, IC27 D36V28F5-5V-3.2A, IC28 D24V5F1-1.8V-500MA, IC29 D24V10F3-3.3V-1A, IC3 OPA1632DR, IC30 D24V25F5-5V-2.5A, IC31 TLV2771CDBVR, IC32 TLV2771CDBVR, IC33 TLV2771CDBVR, IC34 TLV2771CDBVR, IC35 FODM217DV, IC36 FODM217DV, IC37 FODM217DV, IC38 FODM217DV, IC39 FODM217DV, IC4 OPA1632DR, IC40 FODM217DV, IC41 FODM217DV, IC42 FODM217DV, IC43 D24V25F5-5V-2.5A, IC5 OPA1632DR, IC6 OPA1632DR, IC7 OPA1632DR, IC8 OPA1632DR, IC9 REF1004U, J1 22-29-2021, J2 22-29-2021, J3 1985027, J4 1989764, J5 1755736, J6 22-29-2021, U1 OPA350EA/2K5, U10 VXO78012-500, U2 OPA350EA/2K5, U3 ADS1178IPAPT, U4 OPA350EA/2K5, U5 OPA350EA/2K5, U6 ADS1178IPAPT, U7 OPA350EA/2K5, U8 OPA350EA/2K5, U9 ADS1178IPAPT

Commit message: tarjeta_v13
Parts:
- added R163: (no value), rcl:R0603
- JP6: device pinhead:2X04 -> pinhead:2X05
- moved JP6 0.60 mm to (5.64, 103.4)
Connections:
- new net N$105: JP6.9, R163.2
- net 3.3V_RPI: now also R163.1
- net GND: now also JP6.10
Routing:
- net 3.3V_RPI: track 106.5 -> 204.0 mm, vias 0 -> 1
- net N$105: track 0.00 -> 6.57 mm
- net N$108: track 2.92 -> 3.48 mm
Changed lines of the file:
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@@
 <drawing>
 <settings>
-<setting alwaysvectorfont="yes"/>
+<setting alwaysvectorfont="no"/>
 <setting verticaltext="up"/>
 </settings>
@@
 <attribute name="VALUE" x="104.02" y="109.6" size="1.27" layer="27" rot="R180"/>
 </element>
-<element name="JP6" library="pinhead" library_urn="urn:adsk.eagle:library:325" package="2X04" package3d_urn="urn:adsk.eagle:package:22461/2" value="" x="5.87" y="102.89" smashed="yes" rot="R90">
-<attribute name="NAME" x="2.695" y="97.81" size="0.6096" layer="25" ratio="10" rot="R90"/>
-<attribute name="POPULARITY" value="47" x="5.87" y="102.89" size="1.778" layer="27" rot="R90" display="off"/>
-<attribute name="VALUE" x="10.315" y="97.81" size="1.27" layer="27" rot="R90"/>
+<element name="JP6" library="pinhead" library_urn="urn:adsk.eagle:library:325" package="2X05" package3d_urn="urn:adsk.eagle:package:22470/2" value="" x="5.6414" y="103.4488" smashed="yes" rot="R90">
+<attribute name="NAME" x="2.4664" y="98.3688" size="0.6096" layer="25" ratio="10" rot="R90"/>
+<attribute name="POPULARITY" value="35" x="5.6414" y="103.4488" size="1.778" layer="27" rot="R90" display="off"/>
+<attribute name="VALUE" x="10.0864" y="98.3688" size="1.27" layer="27" rot="R90"/>
 </element>
 <element name="J1" library="SamacSys_Parts" package="SHDR2W64P0X254_1X2_508X580X117" value="22-29-2021" x="146.96" y="15.31" smashed="yes" rot="R90">
@@
 <attribute name="VALUE" x="5.0292" y="15.0876" size="1.27" layer="27" align="center"/>
 </element>
+<element name="R163" library="rcl" library_urn="urn:adsk.eagle:library:334" package="R0603" package3d_urn="urn:adsk.eagle:package:23555/3" value="" x="2.7432" y="111.252" smashed="yes" rot="R180">
+<attribute name="NAME" x="3.3782" y="110.617" size="1.27" layer="25" rot="R180"/>
+<attribute name="POPULARITY" value="77" x="2.7432" y="111.252" size="0.0508" layer="27" rot="R180" display="off"/>
+<attribute name="SPICEPREFIX" value="R" x="2.7432" y="111.252" size="0.0508" layer="27" rot="R180" display="off"/>
+<attribute name="VALUE" x="3.3782" y="113.157" size="1.27" layer="27" rot="R180"/>
+</element>
 </elements>
 <signals>
@@
 <contactref element="JP4" pad="37"/>
 <contactref element="J6" pad="2"/>
+<contactref element="JP6" pad="10"/>
 </signal>
 <signal name="N$1">
@@
 <wire x1="99.48" y1="106.33" x2="97.67" y2="104.52" width="0.2032" layer="1"/>
 <wire x1="117.41" y1="30.29" x2="121.4676" y2="34.3476" width="0.2032" layer="1"/>
+<contactref element="R163" pad="1"/>
+<wire x1="97.67" y1="104.52" x2="97.67" y2="105.5554" width="0.508" layer="15"/>
+<wire x1="97.67" y1="105.5554" x2="95.1992" y2="108.0262" width="0.508" layer="15"/>
+<wire x1="95.1992" y1="108.0262" x2="22.8346" y2="108.0262" width="0.508" layer="15"/>
+<wire x1="19.812" y1="111.0488" x2="4.9276" y2="111.0488" width="0.508" layer="15"/>
+<via x="4.9276" y="111.0488" extent="1-16" drill="0.35"/>
+<wire x1="4.9276" y1="111.0488" x2="3.7964" y2="111.0488" width="0.508" layer="1"/>
+<wire x1="3.7964" y1="111.0488" x2="3.5932" y2="111.252" width="0.508" layer="1"/>
+<wire x1="22.8346" y1="108.0262" x2="19.812" y2="111.0488" width="0.508" layer="15"/>
 </signal>
 <signal name="N$106">
 <contactref element="JP6" pad="1"/>
 <contactref element="R139" pad="2"/>
-<wire x1="9.84" y1="98.03" x2="8.19" y2="98.03" width="0.6096" layer="1"/>
-<wire x1="8.19" y1="98.03" x2="7.14" y2="99.08" width="0.6096" layer="1"/>
+<wire x1="9.84" y1="98.03" x2="7.2502" y2="98.03" width="0.508" layer="1"/>
+<wire x1="7.2502" y1="98.03" x2="6.9114" y2="98.3688" width="0.508" layer="1"/>
 </signal>
 <signal name="N$107">
 <contactref element="JP6" pad="3"/>
 <contactref element="R140" pad="2"/>
-<wire x1="9.83" y1="101.34" x2="7.42" y2="101.34" width="0.6096" layer="1"/>
-<wire x1="7.42" y1="101.34" x2="7.14" y2="101.62" width="0.6096" layer="1"/>
+<wire x1="9.83" y1="101.34" x2="7.3426" y2="101.34" width="0.508" layer="1"/>
+<wire x1="7.3426" y1="101.34" x2="6.9114" y2="100.9088" width="0.508" layer="1"/>
 </signal>
 <signal name="N$108">
 <contactref element="JP6" pad="5"/>
 <contactref element="R141" pad="2"/>
-<wire x1="9.88" y1="104.6" x2="7.58" y2="104.6" width="0.6096" layer="1"/>
-<wire x1="7.58" y1="104.6" x2="7.14" y2="104.16" width="0.6096" layer="1"/>
+<wire x1="9.88" y1="104.6" x2="9.8546" y2="104.5746" width="0.6096" layer="1"/>
+<wire x1="9.88" y1="104.6" x2="8.0626" y2="104.6" width="0.508" layer="1"/>
+<wire x1="8.0626" y1="104.6" x2="6.9114" y2="103.4488" width="0.508" layer="1"/>
 </signal>
 <signal name="N$109">
 <contactref element="JP6" pad="7"/>
 <contactref element="R142" pad="2"/>
-<wire x1="9.85" y1="106.34" x2="7.5" y2="106.34" width="0.6096" layer="1"/>
-<wire x1="7.5" y1="106.34" x2="7.14" y2="106.7" width="0.6096" layer="1"/>
+<wire x1="9.85" y1="106.34" x2="7.2626" y2="106.34" width="0.508" layer="1"/>
+<wire x1="7.2626" y1="106.34" x2="6.9114" y2="105.9888" width="0.508" layer="1"/>
 </signal>
 <signal name="DOBLE1">
@@
 <wire x1="104.6444" y1="115.3284" x2="85.7616" y2="115.3284" width="0.508" layer="1"/>
 </signal>
+<signal name="N$105">
+<contactref element="R163" pad="2"/>
+<contactref element="JP6" pad="9"/>
+<wire x1="6.9114" y1="108.5288" x2="5.4582" y2="109.982" width="0.508" layer="1"/>
+<wire x1="5.4582" y1="109.982" x2="2.4384" y2="109.982" width="0.508" layer="1"/>
+<wire x1="2.4384" y1="109.982" x2="1.8932" y2="110.5272" width="0.508" layer="1"/>
+<wire x1="1.8932" y1="110.5272" x2="1.8932" y2="111.252" width="0.508" layer="1"/>
+</signal>
 </signals>

Commit message: tarjeta_v15
Parts:
- R139, R140, R141, R142, R163: value (none) -> 330R
- R147, R148, R149, R150, R151, R152, R153, R154, R155, R156, R157, R158, R159, R160, R161, R162: value (none) -> 220R

Commit message: tarjeta_v17
Parts:
- removed IC1, IC2: OPA1632DR, SamacSys_Parts:SOIC127P600X175-8N
- removed IC21, IC26, IC9: REF1004U, burr-brown:SO08
- removed R103, R133, R49: 100, rcl:R0603
- removed R107, R137, R53: 20K, rcl:R0603
- added C114, C115, C116, C117, C118, C119: 1uF, rcl:C0603
- added U11: ADS1278IPAPR, ADS1278IPAPR:PAP64_7X7
- added U12, U13: REF5025AID, REF5025:D8
- added U14, U15: THS4521IDGKT, THS4521IDGKT:DGK8
- C33, C74, C99: value 0.1uF -> 10uF
- U3: value ADS1178IPAPT -> REF5025AID; device ADS1178IPAPT:PAP64_TEX -> REF5025:D8
- U6, U9: value ADS1178IPAPT -> ADS1278IPAPR; device ADS1178IPAPT:PAP64_TEX -> ADS1278IPAPR:PAP64_7X7
- moved U9 181.5 mm to (6.81, -47.0), turned to 0 degrees
- moved U6 128.2 mm to (6.81, -77.5), flipped to the top
- moved U3 71.3 mm to (2.44, -11.2)
Connections:
- removed net N$98: IC26.8, R137.1
- new net N$103: U11.31
- net +12V: no longer IC1.3, IC2.3
- net +1V8: now also U11.26; no longer U3.26
- net +3V3: now also U11.10, U11.22, U11.23, U11.35, U11.36, U11.37, U11.38, U11.39, U11.40, U11.41, U11.42; no longer U3.10, U3.22, U3.23, U3.31, U3.35, U3.36, U3.37, U3.38, U3.39, U3.40, U3.41, U3.42, U6.31, U9.31
- net +5V: now also C114.1, C117.1, C119.1, U11.44, U11.5, U11.53, U11.60, U12.2, U13.2, U14.3, U15.3, U3.2; no longer R107.2, R137.2, R53.2, U3.44, U3.5, U3.53, U3.60
- net -12V: no longer IC1.6, IC2.6
- net AINN1_1: now also R2.1, R3.1, U11.4; no longer R5.1, R6.1, U3.4
- net AINN1_2: now also R8.1, R9.1, U11.2; no longer R11.1, R12.1, U3.2
- net AINN1_3: now also U11.64; no longer U3.64
- net AINN1_4: now also U11.62; no longer U3.62
- net AINN1_5: now also U11.52; no longer U3.52
- net AINN1_6: now also U11.50; no longer U3.50
- net AINN1_7: now also U11.48; no longer U3.48
- net AINN1_8: now also U11.46; no longer U3.46
- net AINP1_1: now also R5.1, R6.1, U11.3; no longer R2.1, R3.1, U3.3
- net AINP1_2: now also R11.1, R12.1, U11.1; no longer R8.1, R9.1, U3.1
- net AINP1_3: now also U11.63; no longer U3.63
- net AINP1_4: now also U11.61; no longer U3.61
- net AINP1_5: now also U11.51; no longer U3.51
- net AINP1_6: now also U11.49; no longer U3.49
- net AINP1_7: now also U11.47; no longer U3.47
- net AINP1_8: now also U11.45; no longer U3.45
- net CLK1: now also U11.27; no longer U3.27
- net DOUT1_1: now also U11.20; no longer U3.20
- net DOUT1_2: now also U11.19; no longer U3.19
- net DOUT1_3: now also U11.18; no longer U3.18
- net DOUT1_4: now also U11.17; no longer U3.17
- net DOUT1_5: now also U11.16; no longer U3.16
- net DOUT1_6: now also U11.15; no longer U3.15
- net DOUT1_7: now also U11.14; no longer U3.14
- net DOUT1_8: now also U11.13; no longer U3.13
- net DRDY1: now also U11.29; no longer U3.29
- net GND: now also C114.2, C115.2, C116.2, C117.2, C118.2, C119.2, U11.12, U11.21, U11.24, U11.25, U11.30, U11.32, U11.33, U11.34, U11.43, U11.54, U11.57, U11.58, U11.59, U11.6, U11.65, U11.7, U11.8, U11.9, U12.4, U13.4, U14.6, U15.6, U3.4, U6.33, U6.65, U9.33, U9.65; no longer IC21.4, IC26.4, IC9.4, U3.12, U3.21, U3.24, U3.25, U3.30, U3.32, U3.34, U3.43, U3.54, U3.57, U3.58, U3.59, U3.6, U3.7, U3.8, U3.9, U3.EPAD, U6.EPAD, U9.EPAD
- net N$1: now also U14.1; no longer IC1.1
- net N$2: now also U14.8; no longer IC1.8
- net N$3: now also U14.5; no longer IC1.5
- net N$33: now also C34.1, R50.2; no longer R49.2
- net N$34: now also C99.1, R134.1, U12.6; no longer C33.1, C34.1, R49.1, R50.2
- net N$35: now also C115.1, U3.5; no longer IC9.6, R50.1
- net N$36: now also C33.1, R50.1, U3.6; no longer IC9.8, R53.1
- net N$4: now also U14.4; no longer IC1.4
- net N$5: now also U15.8; no longer IC2.8
- net N$6: now also U15.5; no longer IC2.5
- net N$7: now also U15.1; no longer IC2.1
- net N$72: now also C75.1, R104.2; no longer R103.2
- net N$73: now also R104.1, U13.6; no longer C75.1, R103.1, R104.2
- net N$74: now also C118.1, U13.5; no longer IC21.6, R104.1
- net N$75: now also U6.31; no longer IC21.8, R107.1
- net N$8: now also U15.4; no longer IC2.4
- net N$95: now also C100.1, R134.2; no longer R133.2
- net N$96: now also C116.1, U12.5; no longer C100.1, C99.1, R133.1, R134.2
- net N$97: now also U9.31; no longer IC26.6, R134.1
- net SCLK1: now also U11.28; no longer U3.28
- net SYNC1: now also U11.11; no longer U3.11
- net VCOM1: now also U14.2, U15.2; no longer IC1.2, IC2.2
- net VCOMM1: now also U11.55; no longer U3.55
- net VREFP1: now also U11.56; no longer U3.56
Routing:
- net +3V3: track 397.8 -> 281.2 mm
- net +5V: track 614.8 -> 539.7 mm
- net AINN1_1: track 65.0 -> 3.04 mm
- net AINN1_2: track 42.2 -> 3.28 mm
- net AINN2_3: track 88.9 -> 58.1 mm
- net AINN2_1: track 79.9 -> 50.8 mm
- net AINP2_1: track 82.0 -> 53.3 mm
- net AINN2_2: track 60.1 -> 31.8 mm
- net AINP2_2: track 61.6 -> 33.9 mm
- net GND: track 33.6 -> 10.1 mm, vias 30 -> 29
- net AINP1_8: track 47.3 -> 28.5 mm
- net AINN1_8: track 47.7 -> 29.1 mm
- net DRDY1: track 56.2 -> 39.0 mm
- net SCLK1: track 57.7 -> 41.5 mm
- net CLK1: track 53.0 -> 37.8 mm
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
Commit message: tarjeta_v17
Parts:
- removed IC13, IC14, IC15, IC16, IC17, IC18, IC19, IC20, IC22, IC23, IC24, IC25, IC3, IC4, IC5, IC6, IC7, IC8: OPA1632DR, SamacSys_Parts:SOIC127P600X175-8N
- added U16, U17, U18, U19, U20, U21, U22, U23, U24, U25, U26, U27, U28, U29, U30, U31, U32, U33: THS4521IDGKT, THS4521IDGKT:DGK8
- C108, C109, C110, C111: value (none) -> 20nF
- R143, R144, R145, R146: value (none) -> 10M
- moved U9 181.6 mm to (152.3, 61.6), turned to 90 degrees
- moved U14 179.0 mm to (19.2, 90.7)
- moved U15 165.5 mm to (19.9, 72.3)
- moved C117 114.1 mm to (-29.6, 72.6)
- moved C118 114.1 mm to (-29.6, 47.0)
- moved C119 114.1 mm to (-29.6, 42.1)
- moved C116 114.1 mm to (-29.6, 77.4)
- moved U12 114.1 mm to (-27.3, 82.5)
- moved U13 114.1 mm to (-27.3, 52.0)
- moved U6 111.5 mm to (-31.6, 27.2), turned to 90 degrees
- moved C115 104.3 mm to (57.0, 66.3)
- moved C114 102.5 mm to (60.7, 66.4)
- moved U3 92.6 mm to (58.3, 62.6), turned to 180 degrees
- moved R50 4.32 mm to (50.6, 61.9)
- moved C34 3.54 mm to (51.5, 66.0)
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Connections:
- removed net N$103: U11.31
- removed net N$97: U9.31
- net +12V: no longer IC13.3, IC14.3, IC15.3, IC16.3, IC17.3, IC18.3, IC19.3, IC20.3, IC22.3, IC23.3, IC24.3, IC25.3, IC3.3, IC4.3, IC5.3, IC6.3, IC7.3, IC8.3
- net +3V3: now also U11.31, U9.31
- net +5V: now also U16.3, U17.3, U18.3, U19.3, U20.3, U21.3, U22.3, U23.3, U24.3, U25.3, U26.3, U27.3, U28.3, U29.3, U30.3, U31.3, U32.3, U33.3
- net -12V: no longer IC13.6, IC14.6, IC15.6, IC16.6, IC17.6, IC18.6, IC19.6, IC20.6, IC22.6, IC23.6, IC24.6, IC25.6, IC3.6, IC4.6, IC5.6, IC6.6, IC7.6, IC8.6
- net AINN1_3: now also R14.1, R15.1; no longer R17.1, R18.1
- net AINN1_4: now also R20.1, R21.1; no longer R23.1, R24.1
- net AINN1_5: now also R26.1, R27.1; no longer R29.1, R30.1
- net AINN1_6: now also R32.1, R33.1; no longer R35.1, R36.1
- net AINN1_7: now also R38.1, R39.1; no longer R41.1, R42.1
- net AINN1_8: now also R44.1, R45.1; no longer R47.1, R48.1
- net AINN3_1: now also R110.1, R111.1; no longer R113.1, R114.1
- net AINN3_2: now also R116.1, R117.1; no longer R119.1, R120.1
- net AINP1_3: now also R17.1, R18.1; no longer R14.1, R15.1
- net AINP1_4: now also R23.1, R24.1; no longer R20.1, R21.1
- net AINP1_5: now also R29.1, R30.1; no longer R26.1, R27.1
- net AINP1_6: now also R35.1, R36.1; no longer R32.1, R33.1
- net AINP1_7: now also R41.1, R42.1; no longer R38.1, R39.1
- net AINP1_8: now also R47.1, R48.1; no longer R44.1, R45.1
- net AINP3_1: now also R113.1, R114.1; no longer R110.1, R111.1
- net AINP3_2: now also R119.1, R120.1; no longer R116.1, R117.1
- net GND: now also U16.6, U17.6, U18.6, U19.6, U20.6, U21.6, U22.6, U23.6, U24.6, U25.6, U26.6, U27.6, U28.6, U29.6, U30.6, U31.6, U32.6, U33.6
- net N$10: now also U16.5; no longer IC3.5
- net N$11: now also U16.1; no longer IC3.1
- net N$12: now also U16.4; no longer IC3.4
- net N$13: now also U17.8; no longer IC4.8
- net N$14: now also U17.5; no longer IC4.5
- net N$15: now also U17.1; no longer IC4.1
- net N$16: now also U17.4; no longer IC4.4
- net N$17: now also U18.8; no longer IC5.8
- net N$18: now also U18.5; no longer IC5.5
- net N$19: now also U18.1; no longer IC5.1
- net N$20: now also U18.4; no longer IC5.4
- net N$21: now also U19.8; no longer IC6.8
- net N$22: now also U19.5; no longer IC6.5
- net N$23: now also U19.1; no longer IC6.1
- net N$24: now also U19.4; no longer IC6.4
- net N$25: now also U20.8; no longer IC7.8
- net N$26: now also U20.5; no longer IC7.5
- net N$27: now also U20.1; no longer IC7.1
- net N$28: now also U20.4; no longer IC7.4
- net N$29: now also U21.8; no longer IC8.8
- net N$30: now also U21.5; no longer IC8.5
- net N$31: now also U21.1; no longer IC8.1
- net N$32: now also U21.4; no longer IC8.4
- net N$40: now also U22.8; no longer IC13.8
- net N$41: now also U22.5; no longer IC13.5
- net N$42: now also U22.1; no longer IC13.1
- net N$43: now also U22.4; no longer IC13.4
- net N$44: now also U23.8; no longer IC14.8
- net N$45: now also U23.5; no longer IC14.5
- net N$46: now also U23.1; no longer IC14.1
- net N$47: now also U23.4; no longer IC14.4
- net N$48: now also U24.8; no longer IC15.8
- net N$49: now also U24.5; no longer IC15.5
- net N$50: now also U24.1; no longer IC15.1
- net N$51: now also U24.4; no longer IC15.4
- net N$52: now also U25.8; no longer IC16.8
- net N$53: now also U25.5; no longer IC16.5
- net N$54: now also U25.1; no longer IC16.1
- net N$55: now also U25.4; no longer IC16.4
- net N$56: now also U26.8; no longer IC17.8
- net N$57: now also U26.5; no longer IC17.5
- net N$58: now also U26.1; no longer IC17.1
- net N$59: now also U26.4; no longer IC17.4
- net N$60: now also U27.8; no longer IC18.8
- net N$61: now also U27.5; no longer IC18.5
- net N$62: now also U27.1; no longer IC18.1
- net N$63: now also U27.4; no longer IC18.4
- net N$64: now also U28.8; no longer IC19.8
- net N$65: now also U28.5; no longer IC19.5
- net N$66: now also U28.1; no longer IC19.1
- net N$67: now also U28.4; no longer IC19.4
- net N$68: now also U29.8; no longer IC20.8
- net N$69: now also U29.5; no longer IC20.5
- net N$70: now also U29.1; no longer IC20.1
- net N$71: now also U29.4; no longer IC20.4
- net N$79: now also U30.8; no longer IC22.8
- net N$80: now also U30.5; no longer IC22.5
- net N$81: now also U30.1; no longer IC22.1
- net N$82: now also U30.4; no longer IC22.4
- net N$83: now also U31.8; no longer IC23.8
- net N$84: now also U31.5; no longer IC23.5
- net N$85: now also U31.1; no longer IC23.1
- net N$86: now also U31.4; no longer IC23.4
- net N$87: now also U32.8; no longer IC24.8
- net N$88: now also U32.5; no longer IC24.5
- net N$89: now also U32.1; no longer IC24.1
- net N$9: now also U16.8; no longer IC3.8
- net N$90: now also U32.4; no longer IC24.4
- net N$91: now also U33.8; no longer IC25.8
- net N$92: now also U33.5; no longer IC25.5
- net N$93: now also U33.1; no longer IC25.1
- net N$94: now also U33.4; no longer IC25.4
- net VCOM1: now also U16.2, U17.2, U18.2, U19.2, U20.2, U21.2; no longer IC3.2, IC4.2, IC5.2, IC6.2, IC7.2, IC8.2
- net VCOM2: now also U22.2, U23.2, U24.2, U25.2, U26.2, U27.2, U28.2, U29.2; no longer IC13.2, IC14.2, IC15.2, IC16.2, IC17.2, IC18.2, IC19.2, IC20.2
- net VCOM3: now also U30.2, U31.2, U32.2, U33.2; no longer IC22.2, IC23.2, IC24.2, IC25.2
Routing:
- net +3V3: track 281.2 -> 360.1 mm
- net AINN1_1: track 3.04 -> 72.6 mm
- net AINN1_2: track 3.28 -> 48.5 mm, vias 0 -> 2
- net +5V: track 539.7 -> 584.9 mm
- net +12V: track 705.2 -> 677.8 mm
- net -12V: track 647.7 -> 621.5 mm
- net AINN1_8: track 29.1 -> 49.8 mm, vias 0 -> 2
- net AINP1_8: track 28.5 -> 47.6 mm
- net DRDY1: track 39.0 -> 56.3 mm
- net VCOM2: track 195.7 -> 179.2 mm
- net SCLK1: track 41.5 -> 57.8 mm
- net AINN1_3: track 45.2 -> 60.7 mm, vias 0 -> 2
- net CLK1: track 37.8 -> 53.1 mm
- net AINP1_1: track 77.4 -> 64.0 mm, vias 0 -> 2
- net AINN3_1: track 49.5 -> 62.8 mm
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
Commit message: tarjeta_v17
Parts:
- moved C117 167.9 mm to (138.2, 71.0), turned to 270 degrees
- moved U12 161.2 mm to (133.4, 70.0), turned to 270 degrees
- moved C116 159.3 mm to (129.6, 71.7), turned to 90 degrees
- moved C119 98.8 mm to (67.0, 62.8), flipped to the bottom
- moved C118 97.7 mm to (67.8, 55.2), flipped to the bottom, turned to 180 degrees
- moved U6 97.5 mm to (65.3, 38.1), flipped to the bottom, turned to 0 degrees
- moved U13 94.6 mm to (67.1, 58.8), flipped to the bottom
- moved U22 74.5 mm to (68.9, 91.3), flipped to the bottom
- moved U23 73.3 mm to (68.8, 73.9), flipped to the bottom
- moved U24 60.9 mm to (52.0, 91.6), flipped to the bottom
- moved U25 57.8 mm to (52.5, 73.7), flipped to the bottom
- moved U26 52.5 mm to (37.2, 91.5), flipped to the bottom
- moved U28 48.2 mm to (21.0, 91.0), flipped to the bottom
- moved U27 45.5 mm to (36.7, 74.0), flipped to the bottom
- moved U29 37.9 mm to (20.9, 73.5), flipped to the bottom
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Connections:
- removed net N$75: U6.31
- net +3V3: now also U6.31
- net AINN2_1: now also R56.1, R57.1; no longer R59.1, R60.1
- net AINN2_2: now also R62.1, R63.1; no longer R65.1, R66.1
- net AINN2_3: now also R68.1, R69.1; no longer R71.1, R72.1
- net AINN2_4: now also R74.1, R75.1; no longer R77.1, R78.1
- net AINN2_5: now also R80.1, R81.1; no longer R83.1, R84.1
- net AINN2_6: now also R86.1, R87.1; no longer R89.1, R90.1
- net AINN2_7: now also R92.1, R93.1; no longer R95.1, R96.1
- net AINN2_8: now also R98.1, R99.1; no longer R101.1, R102.1
- net AINN3_3: now also R122.1, R123.1; no longer R125.1, R126.1
- net AINN3_4: now also R128.1, R129.1; no longer R131.1, R132.1
- net AINP2_1: now also R59.1, R60.1; no longer R56.1, R57.1
- net AINP2_2: now also R65.1, R66.1; no longer R62.1, R63.1
- net AINP2_3: now also R71.1, R72.1; no longer R68.1, R69.1
- net AINP2_4: now also R77.1, R78.1; no longer R74.1, R75.1
- net AINP2_5: now also R83.1, R84.1; no longer R80.1, R81.1
- net AINP2_6: now also R89.1, R90.1; no longer R86.1, R87.1
- net AINP2_7: now also R95.1, R96.1; no longer R92.1, R93.1
- net AINP2_8: now also R101.1, R102.1; no longer R98.1, R99.1
- net AINP3_3: now also R125.1, R126.1; no longer R122.1, R123.1
- net AINP3_4: now also R131.1, R132.1; no longer R128.1, R129.1
Routing:
- net -12V: track 621.5 -> 13.7 mm, vias 24 -> 0
- net +5V: track 584.9 -> 1077.0 mm, vias 9 -> 30
- net +12V: track 677.8 -> 224.2 mm, vias 25 -> 0
- net DOUT2_5: track 53.9 -> 107.3 mm
- net SYNC2: track 63.6 -> 114.7 mm
- net DOUT2_8: track 65.6 -> 115.6 mm
- net DOUT2_7: track 62.1 -> 110.8 mm
- net DOUT2_6: track 64.5 -> 112.0 mm
- net +3V3: track 360.1 -> 402.8 mm, vias 4 -> 5
- net AINN2_6: track 21.4 -> 59.1 mm, vias 0 -> 2
- net AINN2_8: track 33.5 -> 71.1 mm, vias 0 -> 2
- net DOUT2_4: track 55.1 -> 92.5 mm
- net AINN2_5: track 45.1 -> 82.0 mm, vias 0 -> 2
- net DOUT2_3: track 52.4 -> 89.1 mm
- net AINN2_7: track 49.2 -> 85.7 mm, vias 0 -> 2
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
Commit message: tarjeta_v18
Parts:
- removed C108, C109, C110, C111: 20nF, rcl:C0805
- removed IC12: PCF8523, myProyects:PCF8523
- added IC1: DS3231, myProyects:DS3231
- added JP5: (no value), pinhead:1X03
- added R103, R133, R137, R49: 50M, rcl:R0805
- added R107, R164, R165, R53: 1K, rcl:R0805
- R143, R144, R145, R146: value 10M -> 100M
- moved R143 24.3 mm to (159.5, 7.37), flipped to the bottom, turned to 0 degrees
- moved R144 18.2 mm to (159.5, 9.90), flipped to the bottom, turned to 0 degrees
- moved R145 13.2 mm to (159.5, 12.5), flipped to the bottom, turned to 0 degrees
- moved R146 9.83 mm to (159.5, 14.9), flipped to the bottom, turned to 0 degrees
- moved IC31 2.76 mm to (140.8, 27.9), turned to 90 degrees
- moved IC34 2.50 mm to (162.1, 28.6), turned to 90 degrees
- moved IC32 2.36 mm to (148.0, 27.9), turned to 90 degrees
- moved IC33 2.30 mm to (155.0, 28.0), turned to 90 degrees
Connections:
- removed net SQW: IC12.5
- removed net TX: JP1.8
- new net 5V_RPI: JP1.4, JP5.3
- new net N$111: IC34.4, R137.1, R164.2
- new net N$75: IC33.4, R133.1, R165.2
- new net N$97: IC31.4, R49.1, R53.2
- new net N$98: IC32.4, R103.1, R107.2
- new net SIGNAL: JP1.8, JP5.1
- net +3V3: now also IC31.5, IC32.5, IC33.5, IC34.5
- net +5V: no longer IC31.5, IC32.5, IC33.5, IC34.5
- net 3.3V_RPI: now also IC1.VIN; no longer IC12.2
- net DOBLE1: now also IC31.3, R143.1; no longer C108.1, IC31.4, R143.2
- net DOBLE2: now also IC32.3, R144.1; no longer C109.1, IC32.4, R144.2
- net DOBLE3: now also IC33.3, R145.1; no longer C110.1, IC33.4, R145.2
- net DOBLE4: now also IC34.3, R146.1; no longer C111.1, IC34.4, R146.2
- net GND: now also IC1.GND, JP5.2, R107.1, R143.2, R144.2, R145.2, R146.2, R164.1, R165.1, R53.1; no longer IC12.1, IC31.3, IC32.3, IC33.3, IC34.3
- net INPUT17+: now also R49.2; no longer C108.2, R143.1
- net INPUT18+: now also R103.2; no longer C109.2, R144.1
- net INPUT19+: now also R133.2; no longer C110.2, R145.1
- net INPUT20+: now also R137.2; no longer C111.2, R146.1
- net SCL: now also IC1.SCL; no longer IC12.4
- net SDA: now also IC1.SDA; no longer IC12.3
Routing:
- net +5V: track 1077.0 -> 1012.1 mm, vias 30 -> 29
- net +3V3: track 402.8 -> 446.4 mm, vias 5 -> 9
- net 3.3V_RPI: track 204.0 -> 226.9 mm
- net SIGNAL: track 0.00 -> 18.1 mm
- net 5V_RPI: track 0.00 -> 13.8 mm
- net SCL: track 87.6 -> 78.8 mm
- net INPUT17+: track 18.3 -> 10.3 mm, vias 2 -> 0
- net SDA: track 89.8 -> 82.7 mm
- net DOBLE1: track 35.2 -> 41.2 mm
- net N$111: track 0.00 -> 5.49 mm
- net N$97: track 0.00 -> 5.21 mm
- net N$75: track 0.00 -> 4.52 mm
- net N$98: track 0.00 -> 4.48 mm
- net DOBLE3: track 21.0 -> 25.4 mm
- net INPUT19+: track 21.6 -> 17.8 mm, vias 2 -> 0
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Other:
- board text added: "S"
