File: DATALOGGER_ADS_V1/DATALOGGER_ADS_V1.sch (EAGLE design)
At the start: 119 parts, among them IC1 OPA1632DR, IC10 DE10-NANO, IC11 RASPBERRY_PI_4, IC12 PCF8523, IC2 OPA1632DR, IC3 OPA1632DR, IC4 OPA1632DR, IC5 OPA1632DR, IC6 OPA1632DR, IC7 OPA1632DR, IC8 OPA1632DR, IC9 REF1004U, J1 22-29-2021, J2 22-29-2021, U1 OPA350EA/2K5, U2 OPA350EA/2K5, U3 ADS1178IPAPT

Commit message: tarjeta_v2
Parts:
- added C100, C75: 100uF, rcl:C-USC1206
- added C101, C102, C104, C44, C48, C52, C56, C60, C64, C68, C72, C74, C76, C77, C79, C85, C89, C93, C97, C99: 0.1uF, rcl:C-USC0603
- added C103, C105, C106, C107, C78, C80, C81, C82: 10uF, rcl:C-USC0603
- added C42, C45, C46, C49, C50, C53, C54, C57, C58, C61, C62, C65, C66, C69, C70, C73, C83, C86, C87, C90, C91, C94, C95, C98: 2.7nF, rcl:C-USC0603
- added C43, C47, C51, C55, C59, C63, C67, C71, C84, C88, C92, C96: 2.2nF, rcl:C-USC0603
- added IC13, IC14, IC15, IC16, IC17, IC18, IC19, IC20, IC22, IC23, IC24, IC25: OPA1632DR, SamacSys_Parts:OPA1632DR
- added IC21, IC26: REF1004U, burr-brown:REF1004U
- added R100, R101, R104, R106, R109, R110, R112, R113, R115, R116, R118, R119, R121, R122, R124, R125, R127, R128, R130, R131, R134, R136, R55, R56, R58, R59, R61, R62, R64, R65, R67, R68, R70, R71, R73, R74, R76, R77, R79, R80, R82, R83, R85, R86, R88, R89, R91, R92, R94, R95, R97, R98: 1K, rcl:R-US_R0603
- added R102, R111, R114, R117, R120, R123, R126, R129, R132, R57, R60, R63, R66, R69, R72, R75, R78, R81, R84, R87, R90, R93, R96, R99: 49.9, rcl:R-US_R0603
- added R103, R105, R108, R133, R135, R138: 100, rcl:R-US_R0603
- added R107, R137: 20K, rcl:R-US_R0603
- added U4, U5, U7, U8: OPA350EA/2K5, OPA350EA_2K5:OPA350EA/2K5
- added U6, U9: ADS1178IPAPT, ADS1178IPAPT:ADS1178IPAPT
Connections:
- new net AINN2_1: C43.2, R59.1, R60.1, U6.AINN1
- new net AINN2_2: C47.2, R65.1, R66.1, U6.AINN2
- new net AINN2_3: C51.2, R71.1, R72.1, U6.AINN3
- new net AINN2_4: C55.2, R77.1, R78.1, U6.AINN4
- new net AINN2_5: C59.2, R83.1, R84.1, U6.AINN5
- new net AINN2_6: C63.2, R89.1, R90.1, U6.AINN6
- new net AINN2_7: C67.2, R95.1, R96.1, U6.AINN7
- new net AINN2_8: C71.2, R101.1, R102.1, U6.AINN8
- new net AINN3_1: C84.2, R113.1, R114.1, U9.AINN1
- new net AINN3_2: C88.2, R119.1, R120.1, U9.AINN2
- new net AINN3_3: C92.2, R125.1, R126.1, U9.AINN3
- new net AINN3_4: C96.2, R131.1, R132.1, U9.AINN4
- new net AINN3_5: U9.AINN5
- new net AINN3_6: U9.AINN6
- new net AINN3_7: U9.AINN7
- new net AINN3_8: U9.AINN8
- new net AINP2_1: C43.1, R56.1, R57.1, U6.AINP1
- new net AINP2_2: C47.1, R62.1, R63.1, U6.AINP2
- new net AINP2_3: C51.1, R68.1, R69.1, U6.AINP3
- new net AINP2_4: C55.1, R74.1, R75.1, U6.AINP4
- new net AINP2_5: C59.1, R80.1, R81.1, U6.AINP5
- new net AINP2_6: C63.1, R86.1, R87.1, U6.AINP6
- new net AINP2_7: C67.1, R92.1, R93.1, U6.AINP7
- new net AINP2_8: C71.1, R98.1, R99.1, U6.AINP8
- new net AINP3_1: C84.1, R110.1, R111.1, U9.AINP1
- new net AINP3_2: C88.1, R116.1, R117.1, U9.AINP2
- new net AINP3_3: C92.1, R122.1, R123.1, U9.AINP3
- new net AINP3_4: C96.1, R128.1, R129.1, U9.AINP4
- new net AINP3_5: U9.AINP5
- new net AINP3_6: U9.AINP6
- new net AINP3_7: U9.AINP7
- new net AINP3_8: U9.AINP8
- new net CLK2: U6.CLK
- new net CLK3: U9.CLK
- new net DOUT2_1: U6.DOUT1
- new net DOUT2_2: U6.DOUT2
- new net DOUT2_3: U6.DOUT3
- new net DOUT2_4: U6.DOUT4
- new net DOUT2_5: U6.DOUT5
- new net DOUT2_6: U6.DOUT6
- new net DOUT2_7: U6.DOUT7
- new net DOUT2_8: U6.DOUT8
- new net DOUT3_1: U9.DOUT1
- new net DOUT3_2: U9.DOUT2
- new net DOUT3_3: U9.DOUT3
- new net DOUT3_4: U9.DOUT4
- new net DOUT3_5: U9.DOUT5
- new net DOUT3_6: U9.DOUT6
- new net DOUT3_7: U9.DOUT7
- new net DOUT3_8: U9.DOUT8
- new net DRDY2: U6.!DRDY/FSYNC
- new net DRDY3: U9.!DRDY/FSYNC
- new net INPUT10+: R61.2
- new net INPUT10-: R64.2
- new net INPUT11+: R67.2
- new net INPUT11-: R70.2
- new net INPUT12+: R73.2
- new net INPUT12-: R76.2
- new net INPUT13+: R79.2
- new net INPUT13-: R82.2
- new net INPUT14+: R85.2
- new net INPUT14-: R88.2
- new net INPUT15+: R91.2
- new net INPUT15-: R94.2
- new net INPUT16+: R97.2
- new net INPUT16-: R100.2
- new net INPUT17+: R109.2
- new net INPUT17-: R112.2
- new net INPUT18+: R115.2
- new net INPUT18-: R118.2
- new net INPUT19+: R121.2
- new net INPUT19-: R124.2
- new net INPUT20+: R127.2
- new net INPUT20-: R130.2
- new net INPUT9+: R55.2
- new net INPUT9-: R58.2
- new net N$100: C101.2, R135.1, U7.OUTPUT
- new net N$101: R138.1, U8.IN-, U8.OUTPUT
- new net N$40: C42.1, IC13.VIN+, R55.1, R56.2
- new net N$41: C42.2, IC13.VOUT-, R57.2
- new net N$42: C45.1, IC13.VIN-, R58.1, R59.2
- new net N$43: C45.2, IC13.VOUT+, R60.2
- new net N$44: C46.1, IC14.VIN+, R61.1, R62.2
- new net N$45: C46.2, IC14.VOUT-, R63.2
- new net N$46: C49.1, IC14.VIN-, R64.1, R65.2
- new net N$47: C49.2, IC14.VOUT+, R66.2
- new net N$48: C50.1, IC15.VIN+, R67.1, R68.2
- new net N$49: C50.2, IC15.VOUT-, R69.2
- new net N$50: C53.1, IC15.VIN-, R70.1, R71.2
- new net N$51: C53.2, IC15.VOUT+, R72.2
- new net N$52: C54.1, IC16.VIN+, R73.1, R74.2
- new net N$53: C54.2, IC16.VOUT-, R75.2
- new net N$54: C57.1, IC16.VIN-, R76.1, R77.2
- new net N$55: C57.2, IC16.VOUT+, R78.2
- new net N$56: C58.1, IC17.VIN+, R79.1, R80.2
- new net N$57: C58.2, IC17.VOUT-, R81.2
- new net N$58: C61.1, IC17.VIN-, R82.1, R83.2
- new net N$59: C61.2, IC17.VOUT+, R84.2
- new net N$60: C62.1, IC18.VIN+, R85.1, R86.2
- new net N$61: C62.2, IC18.VOUT-, R87.2
- new net N$62: C65.1, IC18.VIN-, R88.1, R89.2
- new net N$63: C65.2, IC18.VOUT+, R90.2
- new net N$64: C66.1, IC19.VIN+, R91.1, R92.2
- new net N$65: C66.2, IC19.VOUT-, R93.2
- new net N$66: C69.1, IC19.VIN-, R94.1, R95.2
- new net N$67: C69.2, IC19.VOUT+, R96.2
- new net N$68: C70.1, IC20.VIN+, R97.1, R98.2
- new net N$69: C70.2, IC20.VOUT-, R99.2
- new net N$70: C73.1, IC20.VIN-, R100.1, R101.2
- new net N$71: C73.2, IC20.VOUT+, R102.2
- new net N$72: R103.2, U4.IN+
- new net N$73: C74.1, C75.1, R103.1, R104.2
- new net N$74: IC21.C, R104.1
- new net N$75: IC21.C1, R107.1
- new net N$76: C76.1, R106.1, U4.IN-
- new net N$77: C76.2, R105.1, U4.OUTPUT
- new net N$78: R108.1, U5.IN-, U5.OUTPUT
- new net N$79: C83.1, IC22.VIN+, R109.1, R110.2
- new net N$80: C83.2, IC22.VOUT-, R111.2
- new net N$81: C86.1, IC22.VIN-, R112.1, R113.2
- new net N$82: C86.2, IC22.VOUT+, R114.2
- new net N$83: C87.1, IC23.VIN+, R115.1, R116.2
- new net N$84: C87.2, IC23.VOUT-, R117.2
- new net N$85: C90.1, IC23.VIN-, R118.1, R119.2
- new net N$86: C90.2, IC23.VOUT+, R120.2
- new net N$87: C91.1, IC24.VIN+, R121.1, R122.2
- new net N$88: C91.2, IC24.VOUT-, R123.2
- new net N$89: C94.1, IC24.VIN-, R124.1, R125.2
- new net N$90: C94.2, IC24.VOUT+, R126.2
- new net N$91: C95.1, IC25.VIN+, R127.1, R128.2
- new net N$92: C95.2, IC25.VOUT-, R129.2
- new net N$93: C98.1, IC25.VIN-, R130.1, R131.2
- new net N$94: C98.2, IC25.VOUT+, R132.2
- new net N$95: R133.2, U7.IN+
- new net N$96: C100.1, C99.1, R133.1, R134.2
- new net N$97: IC26.C, R134.1
- new net N$98: IC26.C1, R137.1
- new net N$99: C101.1, R136.1, U7.IN-
- new net SCLK2: U6.SCLK
- new net SCLK3: U9.SCLK
- new net SYNC2: U6.!SYNC
- new net SYNC3: U9.!SYNC
- new net VCOM2: C44.1, C48.1, C52.1, C56.1, C60.1, C64.1, C68.1, C72.1, IC13.VOCM, IC14.VOCM, IC15.VOCM, IC16.VOCM, IC17.VOCM, IC18.VOCM, IC19.VOCM, IC20.VOCM, R108.2
- new net VCOM3: C85.1, C89.1, C93.1, C97.1, IC22.VOCM, IC23.VOCM, IC24.VOCM, IC25.VOCM, R138.2
- new net VCOMM2: C79.1, U5.IN+, U6.VCOM
- new net VCOMM3: C104.1, U8.IN+, U9.VCOM
- new net VREFN2: C77.2, C78.2, U6.VREFN
- new net VREFN3: C102.2, C103.2, U9.VREFN
- new net VREFP2: C77.1, C78.1, R105.2, R106.2, U6.VREFP
- new net VREFP3: C102.1, C103.1, R135.2, R136.2, U9.VREFP
- net +12V: now also IC13.V+, IC14.V+, IC15.V+, IC16.V+, IC17.V+, IC18.V+, IC19.V+, IC20.V+, IC22.V+, IC23.V+, IC24.V+, IC25.V+
- net +1V8: now also C107.1, C82.1, U6.DVDD, U9.DVDD
- net +3V3: now also C106.1, C81.1, U6.!PWDN1, U6.!PWDN2, U6.!PWDN3, U6.!PWDN4, U6.!PWDN5, U6.!PWDN6, U6.!PWDN7, U6.!PWDN8, U6.CLKDIV, U6.FORMAT1, U6.IOVDD, U6.IOVDD_2, U9.!PWDN1, U9.!PWDN2, U9.!PWDN3, U9.!PWDN4, U9.!PWDN5, U9.!PWDN6, U9.!PWDN7, U9.!PWDN8, U9.CLKDIV, U9.FORMAT1, U9.IOVDD, U9.IOVDD_2
- net +5V: now also C105.1, C80.1, R107.2, R137.2, U4.V+, U5.V+, U6.AVDD, U6.AVDD_2, U6.AVDD_3, U6.AVDD_4, U7.V+, U8.V+, U9.AVDD, U9.AVDD_2, U9.AVDD_3, U9.AVDD_4
- net -12V: now also IC13.V-, IC14.V-, IC15.V-, IC16.V-, IC17.V-, IC18.V-, IC19.V-, IC20.V-, IC22.V-, IC23.V-, IC24.V-, IC25.V-
- net GND: now also C100.2, C104.2, C105.2, C106.2, C107.2, C44.2, C48.2, C52.2, C56.2, C60.2, C64.2, C68.2, C72.2, C74.2, C75.2, C79.2, C80.2, C81.2, C82.2, C85.2, C89.2, C93.2, C97.2, C99.2, IC21.A, IC26.A, U4.V-, U5.V-, U6.AGND, U6.AGND_2, U6.AGND_3, U6.AGND_4, U6.AGND_5, U6.DGND, U6.DGND_2, U6.DGND_3, U6.DGND_4, U6.DIN, U6.EPAD, U6.FORMAT0, U6.FORMAT2, U6.MODE, U6.TEST0, U6.TEST1, U7.V-, U8.V-, U9.AGND, U9.AGND_2, U9.AGND_3, U9.AGND_4, U9.AGND_5, U9.DGND, U9.DGND_2, U9.DGND_3, U9.DGND_4, U9.DIN, U9.EPAD, U9.FORMAT0, U9.FORMAT2, U9.MODE, U9.TEST0, U9.TEST1

Commit message: tarjeta_v3
Parts:
- removed JP5: (no value), pinhead:PINHD-2X4
- removed JP7: (no value), pinhead:PINHD-2X5
- added IC27: D36V28F5-5V-3.2A, myProyects:D36V28F5-5V-3.2A
- added IC28: D24V5F1-1.8V-500MA, myProyects:D24V5F1-1.8V-500MA
- added IC29: D24V10F3-3.3V-1A, myProyects:D24V10F3-3.3V-1A
- added IC30: D24V25F5-5V-2.5A, myProyects:D24V25F5-5V-2.5A
- added J3: 1985027, SamacSys_Parts:1985027
- added J4: 1989764, 1989764:1989764
- added J5: 1755736, 1755736:1755736
Changed lines of the file:
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@@
 <?xml version="1.0" encoding="utf-8"?>
 <!DOCTYPE eagle SYSTEM "eagle.dtd">
-<eagle version="9.5.2">
+<eagle version="9.6.2">
 <drawing>
 <settings>
@@
 <part name="JP4" library="pinhead" library_urn="urn:adsk.eagle:library:325" deviceset="PINHD-2X20" device="" package3d_urn="urn:adsk.eagle:package:22443/2"/>
 <part name="IC12" library="myProyects" deviceset="PCF8523" device=""/>
-<part name="JP5" library="pinhead" library_urn="urn:adsk.eagle:library:325" deviceset="PINHD-2X4" device="" package3d_urn="urn:adsk.eagle:package:22461/2"/>
 <part name="JP6" library="pinhead" library_urn="urn:adsk.eagle:library:325" deviceset="PINHD-2X4" device="" package3d_urn="urn:adsk.eagle:package:22461/2"/>
-<part name="JP7" library="pinhead" library_urn="urn:adsk.eagle:library:325" deviceset="PINHD-2X5" device="" package3d_urn="urn:adsk.eagle:package:22470/2"/>
 <part name="J1" library="SamacSys_Parts" deviceset="22-29-2021" device=""/>
 <part name="J2" library="SamacSys_Parts" deviceset="22-29-2021" device=""/>
@@
 <part name="P+40" library="supply1" library_urn="urn:adsk.eagle:library:371" deviceset="+5V" device=""/>
 <part name="P+41" library="supply1" library_urn="urn:adsk.eagle:library:371" deviceset="+5V" device=""/>
+<part name="FRAME19" library="frames" library_urn="urn:adsk.eagle:library:229" deviceset="A4L-LOC" device=""/>
+<part name="J3" library="SamacSys_Parts" deviceset="1985027" device=""/>
+<part name="FRAME20" library="frames" library_urn="urn:adsk.eagle:library:229" deviceset="A4L-LOC" device=""/>
+<part name="J4" library="1989764" deviceset="1989764" device=""/>
+<part name="FRAME21" library="frames" library_urn="urn:adsk.eagle:library:229" deviceset="A4L-LOC" device=""/>
+<part name="IC27" library="myProyects" deviceset="D36V28F5-5V-3.2A" device=""/>
+<part name="SUPPLY84" library="supply2" library_urn="urn:adsk.eagle:library:372" deviceset="GND" device=""/>
+<part name="IC28" library="myProyects" deviceset="D24V5F1-1.8V-500MA" device=""/>
+<part name="IC29" library="myProyects" deviceset="D24V10F3-3.3V-1A" device=""/>
+<part name="IC30" library="myProyects" deviceset="D24V25F5-5V-2.5A" device=""/>
+<part name="J5" library="1755736" deviceset="1755736" device=""/>
 </parts>
 <sheets>
@@
 <attribute name="VALUE" x="199.39" y="101.6" size="1.778" layer="96"/>
 </instance>
-<instance part="JP5" gate="A" x="203.2" y="60.96" smashed="yes">
-<attribute name="NAME" x="196.85" y="69.215" size="1.778" layer="95"/>
-<attribute name="VALUE" x="196.85" y="53.34" size="1.778" layer="96"/>
-</instance>
 <instance part="JP6" gate="A" x="160.02" y="60.96" smashed="yes">
 <attribute name="NAME" x="153.67" y="69.215" size="1.778" layer="95"/>
 <attribute name="VALUE" x="153.67" y="53.34" size="1.778" layer="96"/>
 </instance>
-<instance part="JP7" gate="A" x="81.28" y="40.64" smashed="yes">
-<attribute name="NAME" x="74.93" y="48.895" size="1.778" layer="95"/>
-<attribute name="VALUE" x="74.93" y="30.48" size="1.778" layer="96"/>
-</instance>
 <instance part="J1" gate="G$1" x="73.66" y="27.94" smashed="yes">
 <attribute name="NAME" x="90.17" y="35.56" size="1.778" layer="95" align="center-left"/>
@@
 </nets>
 </sheet>
+<sheet>
+<plain>
+</plain>
+<instances>
+<instance part="FRAME19" gate="G$1" x="0" y="0" smashed="yes">
+<attribute name="DRAWING_NAME" x="217.17" y="15.24" size="2.54" layer="94"/>
+<attribute name="LAST_DATE_TIME" x="217.17" y="10.16" size="2.286" layer="94"/>
+<attribute name="SHEET" x="230.505" y="5.08" size="2.54" layer="94"/>
+</instance>
+<instance part="J3" gate="G$1" x="63.5" y="137.16" smashed="yes">
+<attribute name="NAME" x="80.01" y="144.78" size="1.778" layer="95" align="center-left"/>
+<attribute name="VALUE" x="80.01" y="142.24" size="1.778" layer="96" align="center-left"/>
+</instance>
+</instances>
+<busses>
+</busses>
+<nets>
+</nets>
+</sheet>
+<sheet>
+<plain>
+</plain>
+<instances>
+<instance part="FRAME20" gate="G$1" x="0" y="0" smashed="yes">
+<attribute name="DRAWING_NAME" x="217.17" y="15.24" size="2.54" layer="94"/>
+<attribute name="LAST_DATE_TIME" x="217.17" y="10.16" size="2.286" layer="94"/>
+<attribute name="SHEET" x="230.505" y="5.08" size="2.54" layer="94"/>
+</instance>
+<instance part="J4" gate="A" x="50.8" y="81.28" smashed="yes">
+<attribute name="NAME" x="54.9656" y="86.5886" size="2.0828" layer="95" ratio="6" rot="SR0"/>
+</instance>
+</instances>
+<busses>
+</busses>
+<nets>
+</nets>
+</sheet>
+<sheet>
+<plain>
+</plain>
+<instances>
+<instance part="FRAME21" gate="G$1" x="0" y="0" smashed="yes">
+<attribute name="DRAWING_NAME" x="217.17" y="15.24" size="2.54" layer="94"/>
+<attribute name="LAST_DATE_TIME" x="217.17" y="10.16" size="2.286" layer="94"/>
+<attribute name="SHEET" x="230.505" y="5.08" size="2.54" layer="94"/>
+</instance>
+<instance part="IC27" gate="A" x="30.48" y="134.62" smashed="yes">
+<attribute name="NAME" x="30.48" y="152.4" size="1.27" layer="95"/>
+<attribute name="VALUE" x="30.48" y="132.08" size="1.27" layer="96"/>
+</instance>
+<instance part="SUPPLY84" gate="GND" x="15.24" y="134.62" smashed="yes">
+<attribute name="VALUE" x="13.335" y="131.445" size="1.778" layer="96"/>
+</instance>
+<instance part="IC28" gate="G$1" x="33.02" y="101.6" smashed="yes">
+<attribute name="NAME" x="33.02" y="116.84" size="1.27" layer="95"/>
+<attribute name="VALUE" x="33.02" y="99.06" size="1.27" layer="96"/>
+</instance>
+<instance part="IC29" gate="A" x="71.12" y="132.08" smashed="yes">
+<attribute name="NAME" x="71.12" y="149.86" size="1.27" layer="95"/>
+<attribute name="VALUE" x="71.12" y="129.54" size="1.27" layer="96"/>
+</instance>
+<instance part="IC30" gate="A" x="71.12" y="104.14" smashed="yes">
+<attribute name="NAME" x="71.12" y="119.38" size="1.778" layer="95"/>
+<attribute name="VALUE" x="71.12" y="101.6" size="1.778" layer="96"/>
+</instance>
+<instance part="J5" gate="A" x="38.1" y="81.28" smashed="yes">
+<attribute name="NAME" x="42.2656" y="86.5886" size="2.0828" layer="95" ratio="6" rot="SR0"/>
+</instance>
+</instances>
+<busses>
+</busses>
+<nets>
+</nets>
+</sheet>

Commit message: tarjeta_v4
Parts:
- added C108, C109, C110, C111: (no value), rcl:C-USC0805
- added IC31, IC32, IC33, IC34: TLV2771CDBVR, SamacSys_Parts:TLV2771CDBVR
- added IC35, IC36, IC37, IC38, IC39, IC40, IC41, IC42: FODM217DV, SamacSys_Parts:FODM217DV
- added R139, R140, R141, R142: (no value), rcl:R-US_R0603
- added R143, R144, R145, R146, R147, R148, R149, R150, R151, R152, R153, R154, R155, R156, R157, R158, R159, R160, R161, R162: (no value), rcl:R-US_R0805
Connections:
- new net 3.3V_RPI: IC12.VCC, JP1.1
- new net 5V_2.5A: J2.1
- new net 5V_3.2A: J1.1
- new net DOBLE1: C108.1, IC31.IN-, J4.1, R143.2
- new net DOBLE2: C109.1, IC32.IN-, J4.2, R144.2
- new net DOBLE3: C110.1, IC33.IN-, J4.3, R145.2
- new net DOBLE4: C111.1, IC34.IN-, J4.4, R146.2
- new net GPIO0_0: JP3.1
- new net GPIO0_1: JP3.2
- new net GPIO0_10: JP3.13
- new net GPIO0_11: JP3.14
- new net GPIO0_12: JP3.15
- new net GPIO0_13: JP3.16
- new net GPIO0_14: JP3.17
- new net GPIO0_15: JP3.18
- new net GPIO0_16: JP3.19
- new net GPIO0_17: JP3.20
- new net GPIO0_18: JP3.21
- new net GPIO0_19: JP3.22
- new net GPIO0_2: JP3.3
- new net GPIO0_20: JP3.23
- new net GPIO0_21: JP3.24
- new net GPIO0_22: JP3.25
- new net GPIO0_23: JP3.26
- new net GPIO0_24: JP3.27
- new net GPIO0_25: JP3.28
- new net GPIO0_26: JP3.31
- new net GPIO0_27: JP3.32
- new net GPIO0_28: JP3.33
- new net GPIO0_29: JP3.34
- new net GPIO0_3: JP3.4
- new net GPIO0_30: JP3.35
- new net GPIO0_31: JP3.36
- new net GPIO0_32: JP3.37
- new net GPIO0_33: JP3.38
- new net GPIO0_34: JP3.39
- new net GPIO0_35: JP3.40
- new net GPIO0_4: JP3.5
- new net GPIO0_5: JP3.6
- new net GPIO0_6: JP3.7
- new net GPIO0_7: JP3.8
- new net GPIO0_8: JP3.9
- new net GPIO0_9: JP3.10
- new net GPIO10: JP1.19
- new net GPIO17: JP1.11, R140.1
- new net GPIO1_0: JP2.1
- new net GPIO1_1: JP2.2
- new net GPIO1_10: JP2.13
- new net GPIO1_11: JP2.14
- new net GPIO1_12: JP2.15
- new net GPIO1_13: JP2.16
- new net GPIO1_14: JP2.17
- new net GPIO1_15: JP2.18
- new net GPIO1_16: JP2.19
- new net GPIO1_17: JP2.20
- new net GPIO1_18: JP2.21
- new net GPIO1_19: JP2.22
- new net GPIO1_2: JP2.3
- new net GPIO1_20: JP2.23
- new net GPIO1_21: JP2.24
- new net GPIO1_22: JP2.25
- new net GPIO1_23: JP2.26
- new net GPIO1_24: JP2.27
- new net GPIO1_25: JP2.28
- new net GPIO1_26: JP2.31
- new net GPIO1_27: JP2.32
- new net GPIO1_28: JP2.33
- new net GPIO1_29: JP2.34
- new net GPIO1_3: JP2.4
- new net GPIO1_30: JP2.35
- new net GPIO1_31: JP2.36
- new net GPIO1_32: JP2.37
- new net GPIO1_33: JP2.38
- new net GPIO1_34: JP2.39
- new net GPIO1_35: JP2.40
- new net GPIO1_4: JP2.5
- new net GPIO1_5: JP2.6
- new net GPIO1_6: JP2.7
- new net GPIO1_7: JP2.8
- new net GPIO1_8: JP2.9
- new net GPIO1_9: JP2.10
- new net GPIO22: JP1.15, R142.1
- new net GPIO27: JP1.13, R141.1
- new net GPIO4: JP1.7, R139.1
- new net GPIO9: JP1.21
- new net LAZO1: IC35.COLLECTOR, R148.1
- new net LAZO2: IC36.COLLECTOR, R150.1
- new net LAZO3: IC37.COLLECTOR, R152.1
- new net LAZO4: IC38.COLLECTOR, R154.1
- new net LAZO5: IC39.COLLECTOR, R156.1
- new net LAZO6: IC40.COLLECTOR, R158.1
- new net LAZO7: IC41.COLLECTOR, R160.1
- new net LAZO8: IC42.COLLECTOR, R162.1
- new net LOOP1: IC35.CATHODE, J3.1
- new net LOOP2: IC36.CATHODE, J3.2
- new net LOOP3: IC37.CATHODE, J3.3
- new net LOOP4: IC38.CATHODE, J3.4
- new net LOOP5: IC39.CATHODE, J3.5
- new net LOOP6: IC40.CATHODE, J3.6
- new net LOOP7: IC41.CATHODE, J3.7
- new net LOOP8: IC42.CATHODE, J3.8
- new net N$102: IC35.ANODE, R147.2
- new net N$104: IC36.ANODE, R149.2
- new net N$105: JP4.35, JP4.39
- new net N$106: JP6.1, R139.2
- new net N$107: JP6.3, R140.2
- new net N$108: JP6.5, R141.2
- new net N$109: JP6.7, R142.2
- new net N$110: JP4.33, JP4.37
- new net N$112: IC37.ANODE, R151.2
- new net N$114: JP4.36, JP4.40
- new net N$115: JP4.34, JP4.38
- new net N$116: IC38.ANODE, R153.2
- new net N$118: IC39.ANODE, R155.2
- new net N$120: IC40.ANODE, R157.2
- new net N$122: IC41.ANODE, R159.2
- new net N$124: IC42.ANODE, R161.2
- new net RX: JP1.10
- new net SCL: IC12.SCL, JP1.5
- new net SDA: IC12.SDA, JP1.3
- new net SQW: IC12.SQW
- new net TX: JP1.8
- net +3V3: now also R148.2, R150.2, R152.2, R154.2, R156.2, R158.2, R160.2, R162.2
- net +5V: now also IC31.VDD, IC32.VDD, IC33.VDD, IC34.VDD, R147.1, R149.1, R151.1, R153.1, R155.1, R157.1, R159.1, R161.1
- net GND: now also IC12.GND, IC31.GND, IC31.IN+, IC32.GND, IC32.IN+, IC33.GND, IC33.IN+, IC34.GND, IC34.IN+, IC35.EMITTER, IC36.EMITTER, IC37.EMITTER, IC38.EMITTER, IC39.EMITTER, IC40.EMITTER, IC41.EMITTER, IC42.EMITTER, J1.2, J2.2, JP1.14, JP1.20, JP1.25, JP1.30, JP1.34, JP1.39, JP1.6, JP1.9, JP2.12, JP2.30, JP3.12, JP3.30, JP6.2, JP6.4, JP6.6, JP6.8
- net INPUT1+: now also JP4.1
- net INPUT1-: now also JP4.2
- net INPUT10+: now also JP4.19
- net INPUT10-: now also JP4.20
- net INPUT11+: now also JP4.21
- net INPUT11-: now also JP4.22
- net INPUT12+: now also JP4.23
- net INPUT12-: now also JP4.24
- net INPUT13+: now also JP4.25
- net INPUT13-: now also JP4.26
- net INPUT14+: now also JP4.27
- net INPUT14-: now also JP4.28
- net INPUT15+: now also JP4.29
- net INPUT15-: now also JP4.30
- net INPUT16+: now also JP4.31
- net INPUT16-: now also JP4.32
- net INPUT17+: now also C108.2, IC31.OUT, R143.1
- net INPUT18+: now also C109.2, IC32.OUT, R144.1
- net INPUT19+: now also C110.2, IC33.OUT, R145.1
- net INPUT2+: now also JP4.3
- net INPUT2-: now also JP4.4
- net INPUT20+: now also C111.2, IC34.OUT, R146.1
- net INPUT3+: now also JP4.5
- net INPUT3-: now also JP4.6
- net INPUT4+: now also JP4.7
- net INPUT4-: now also JP4.8
- net INPUT5+: now also JP4.9
- net INPUT5-: now also JP4.10
- net INPUT6+: now also JP4.11
- net INPUT6-: now also JP4.12
- net INPUT7+: now also JP4.13
- net INPUT7-: now also JP4.14
- net INPUT8+: now also JP4.15
- net INPUT8-: now also JP4.16
- net INPUT9+: now also JP4.17
- net INPUT9-: now also JP4.18
Other:
- moved on the sheet: J1, J3, J4, JP4

Commit message: tarjeta_v5
Parts:
- added C112: 10uF, rcl:C-USC1206
- added C113: 22uF, rcl:C-USC1206
- added IC43: D24V25F5-5V-2.5A, myProyects:D24V25F5-5V-2.5A
- added U$4: D36V6F12-12V-600MA, myProyects:D36V6F12-12V-600MA
- added U10: VXO78012-500, VXO78012-500:VXO78012-500
Connections:
- new net +24V: C112.1, IC27.VIN, IC28.VIN, IC29.VIN, IC30.VIN, IC43.VIN, J5.1, U$4.VIN, U10.+VIN
- net +12V: now also U$4.VOUT
- net +1V8: now also IC28.VOUT
- net +3V3: now also IC29.VOUT
- net +5V: now also IC43.VOUT
- net -12V: now also C113.2, U10.GND/-VOUT
- net 5V_2.5A: now also IC30.VOUT
- net 5V_3.2A: now also IC27.VOUT
- net GND: now also C112.2, C113.1, IC27.GND, IC28.GND, IC29.GND, IC30.GND, IC43.GND, J5.2, U$4.GND, U10.+VOUT/GND
Other:
- moved on the sheet: IC27, IC28, IC29, IC30, J5
