File: DATALOGGER_ADS_V1/DATALOGGER_ADS_V1.sch (EAGLE design)
At the start: 339 parts, among them IC1 OPA1632DR, IC10 DE10-NANO, IC11 RASPBERRY_PI_4, IC12 PCF8523, IC13 OPA1632DR, IC14 OPA1632DR, IC15 OPA1632DR, IC16 OPA1632DR, IC17 OPA1632DR, IC18 OPA1632DR, IC19 OPA1632DR, IC2 OPA1632DR, IC20 OPA1632DR, IC21 REF1004U, IC22 OPA1632DR, IC23 OPA1632DR, IC24 OPA1632DR, IC25 OPA1632DR, IC26 REF1004U, IC27 D36V28F5-5V-3.2A, IC28 D24V5F1-1.8V-500MA, IC29 D24V10F3-3.3V-1A, IC3 OPA1632DR, IC30 D24V25F5-5V-2.5A, IC31 TLV2771CDBVR, IC32 TLV2771CDBVR, IC33 TLV2771CDBVR, IC34 TLV2771CDBVR, IC35 FODM217DV, IC36 FODM217DV, IC37 FODM217DV, IC38 FODM217DV, IC39 FODM217DV, IC4 OPA1632DR, IC40 FODM217DV, IC41 FODM217DV, IC42 FODM217DV, IC43 D24V25F5-5V-2.5A, IC5 OPA1632DR, IC6 OPA1632DR, IC7 OPA1632DR, IC8 OPA1632DR, IC9 REF1004U, J1 22-29-2021, J2 22-29-2021, J3 1985027, J4 1989764, J5 1755736, U1 OPA350EA/2K5, U10 VXO78012-500, U2 OPA350EA/2K5, U3 ADS1178IPAPT, U4 OPA350EA/2K5, U5 OPA350EA/2K5, U6 ADS1178IPAPT, U7 OPA350EA/2K5, U8 OPA350EA/2K5, U9 ADS1178IPAPT

Commit message: tarjeta_v7
Connections:
- removed net INPUT17-: R112.2
- removed net INPUT18-: R118.2
- removed net INPUT19-: R124.2
- removed net INPUT20-: R130.2
- net GND: now also R112.2, R118.2, R124.2, R130.2
Changed lines of the file:
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@@
 <?xml version="1.0" encoding="utf-8"?>
 <!DOCTYPE eagle SYSTEM "eagle.dtd">
-<eagle version="9.5.2">
+<eagle version="9.6.2">
 <drawing>
 <settings>
@@
 <part name="SUPPLY121" library="supply2" library_urn="urn:adsk.eagle:library:372" deviceset="GND" device=""/>
 <part name="P-21" library="supply1" library_urn="urn:adsk.eagle:library:371" deviceset="-12V" device=""/>
+<part name="SUPPLY122" library="supply2" library_urn="urn:adsk.eagle:library:372" deviceset="GND" device=""/>
+<part name="SUPPLY123" library="supply2" library_urn="urn:adsk.eagle:library:372" deviceset="GND" device=""/>
+<part name="SUPPLY124" library="supply2" library_urn="urn:adsk.eagle:library:372" deviceset="GND" device=""/>
+<part name="SUPPLY125" library="supply2" library_urn="urn:adsk.eagle:library:372" deviceset="GND" device=""/>
 </parts>
 <sheets>
@@
 <attribute name="VALUE" x="72.644" y="59.309" size="1.778" layer="96" rot="MR0"/>
 </instance>
+<instance part="SUPPLY122" gate="GND" x="43.18" y="137.16" smashed="yes">
+<attribute name="VALUE" x="41.275" y="133.985" size="1.778" layer="96"/>
+</instance>
+<instance part="SUPPLY123" gate="GND" x="43.18" y="73.66" smashed="yes">
+<attribute name="VALUE" x="41.275" y="70.485" size="1.778" layer="96"/>
+</instance>
 </instances>
 <busses>
@@
 <wire x1="93.98" y1="66.04" x2="93.98" y2="63.5" width="0.1524" layer="91"/>
 </segment>
+<segment>
+<pinref part="R112" gate="G$1" pin="2"/>
+<wire x1="45.72" y1="142.24" x2="43.18" y2="142.24" width="0.1524" layer="91"/>
+<wire x1="43.18" y1="142.24" x2="43.18" y2="139.7" width="0.1524" layer="91"/>
+<pinref part="SUPPLY122" gate="GND" pin="GND"/>
+</segment>
+<segment>
+<pinref part="R118" gate="G$1" pin="2"/>
+<wire x1="45.72" y1="78.74" x2="43.18" y2="78.74" width="0.1524" layer="91"/>
+<wire x1="43.18" y1="78.74" x2="43.18" y2="76.2" width="0.1524" layer="91"/>
+<pinref part="SUPPLY123" gate="GND" pin="GND"/>
+</segment>
 </net>
 <net name="N$81" class="0">
@@
 </segment>
 </net>
-<net name="INPUT17-" class="0">
-<segment>
-<pinref part="R112" gate="G$1" pin="2"/>
-<wire x1="45.72" y1="142.24" x2="43.18" y2="142.24" width="0.1524" layer="91"/>
-<label x="43.18" y="142.24" size="1.778" layer="95" rot="MR0" xref="yes"/>
-</segment>
-</net>
 <net name="INPUT17+" class="0">
 <segment>
@@
 </segment>
 </net>
-<net name="INPUT18-" class="0">
-<segment>
-<pinref part="R118" gate="G$1" pin="2"/>
-<wire x1="45.72" y1="78.74" x2="43.18" y2="78.74" width="0.1524" layer="91"/>
-<label x="43.18" y="78.74" size="1.778" layer="95" rot="MR0" xref="yes"/>
-</segment>
-</net>
 <net name="INPUT18+" class="0">
 <segment>
@@
 <attribute name="VALUE" x="72.644" y="59.309" size="1.778" layer="96" rot="MR0"/>
 </instance>
+<instance part="SUPPLY124" gate="GND" x="43.18" y="137.16" smashed="yes">
+<attribute name="VALUE" x="41.275" y="133.985" size="1.778" layer="96"/>
+</instance>
+<instance part="SUPPLY125" gate="GND" x="43.18" y="73.66" smashed="yes">
+<attribute name="VALUE" x="41.275" y="70.485" size="1.778" layer="96"/>
+</instance>
 </instances>
 <busses>
@@
 <wire x1="93.98" y1="66.04" x2="93.98" y2="63.5" width="0.1524" layer="91"/>
 </segment>
+<segment>
+<pinref part="R124" gate="G$1" pin="2"/>
+<wire x1="45.72" y1="142.24" x2="43.18" y2="142.24" width="0.1524" layer="91"/>
+<wire x1="43.18" y1="142.24" x2="43.18" y2="139.7" width="0.1524" layer="91"/>
+<pinref part="SUPPLY124" gate="GND" pin="GND"/>
+</segment>
+<segment>
+<pinref part="R130" gate="G$1" pin="2"/>
+<wire x1="45.72" y1="78.74" x2="43.18" y2="78.74" width="0.1524" layer="91"/>
+<wire x1="43.18" y1="78.74" x2="43.18" y2="76.2" width="0.1524" layer="91"/>
+<pinref part="SUPPLY125" gate="GND" pin="GND"/>
+</segment>
 </net>
 <net name="N$89" class="0">
@@
 </segment>
 </net>
-<net name="INPUT19-" class="0">
-<segment>
-<pinref part="R124" gate="G$1" pin="2"/>
-<wire x1="45.72" y1="142.24" x2="43.18" y2="142.24" width="0.1524" layer="91"/>
-<label x="43.18" y="142.24" size="1.778" layer="95" rot="MR0" xref="yes"/>
-</segment>
-</net>
 <net name="INPUT19+" class="0">
 <segment>
@@
 </segment>
 </net>
-<net name="INPUT20-" class="0">
-<segment>
-<pinref part="R130" gate="G$1" pin="2"/>
-<wire x1="45.72" y1="78.74" x2="43.18" y2="78.74" width="0.1524" layer="91"/>
-<label x="43.18" y="78.74" size="1.778" layer="95" rot="MR0" xref="yes"/>
-</segment>
-</net>

Commit message: tarjeta_v8
Connections:
- removed net GPIO0_0: JP3.1
- removed net GPIO0_1: JP3.2
- removed net GPIO0_10: JP3.13
- removed net GPIO0_11: JP3.14
- removed net GPIO0_2: JP3.3
- removed net GPIO0_3: JP3.4
- removed net GPIO0_4: JP3.5
- removed net GPIO0_5: JP3.6
- removed net GPIO0_6: JP3.7
- removed net GPIO0_7: JP3.8
- removed net GPIO0_8: JP3.9
- removed net GPIO0_9: JP3.10
- removed net VREFN1: C36.2, C37.2, U3.VREFN
- removed net VREFN2: C77.2, C78.2, U6.VREFN
- removed net VREFN3: C102.2, C103.2, U9.VREFN
- net CLK1: now also JP3.3
- net DOUT1_1: now also JP3.4
- net DOUT1_2: now also JP3.5
- net DOUT1_3: now also JP3.6
- net DOUT1_4: now also JP3.7
- net DOUT1_5: now also JP3.8
- net DOUT1_6: now also JP3.9
- net DOUT1_7: now also JP3.10
- net DOUT1_8: now also JP3.13
- net DRDY1: now also JP3.1
- net GND: now also C102.2, C103.2, C36.2, C37.2, C77.2, C78.2, U3.VREFN, U6.VREFN, U9.VREFN
- net INPUT10+: now also JP4.29; no longer JP4.19
- net INPUT10-: now also JP4.30; no longer JP4.20
- net INPUT11+: now also JP4.27; no longer JP4.21
- net INPUT11-: now also JP4.28; no longer JP4.22
- net INPUT12+: now also JP4.25; no longer JP4.23
- net INPUT12-: now also JP4.26; no longer JP4.24
- net INPUT13+: now also JP4.23; no longer JP4.25
- net INPUT13-: now also JP4.24; no longer JP4.26
- net INPUT14+: now also JP4.21; no longer JP4.27
- net INPUT14-: now also JP4.22; no longer JP4.28
- net INPUT15+: now also JP4.19; no longer JP4.29
- net INPUT15-: now also JP4.20; no longer JP4.30
- net INPUT16+: now also JP4.17; no longer JP4.31
- net INPUT16-: now also JP4.18; no longer JP4.32
- net INPUT9+: now also JP4.31; no longer JP4.17
- net INPUT9-: now also JP4.32; no longer JP4.18
- net SCLK1: now also JP3.2
- net SYNC1: now also JP3.14

Commit message: tarjeta_v9
Connections:
- net GPIO1_29 renamed LAZO_8
- removed net GPIO0_12: JP3.15
- removed net GPIO0_13: JP3.16
- removed net GPIO0_14: JP3.17
- removed net GPIO0_15: JP3.18
- removed net GPIO0_16: JP3.19
- removed net GPIO0_17: JP3.20
- removed net GPIO0_18: JP3.21
- removed net GPIO0_19: JP3.22
- removed net GPIO0_20: JP3.23
- removed net GPIO0_21: JP3.24
- removed net GPIO0_22: JP3.25
- removed net GPIO0_23: JP3.26
- removed net GPIO1_0: JP2.1
- removed net GPIO1_1: JP2.2
- removed net GPIO1_10: JP2.13
- removed net GPIO1_11: JP2.14
- removed net GPIO1_12: JP2.15
- removed net GPIO1_13: JP2.16
- removed net GPIO1_15: JP2.18
- removed net GPIO1_2: JP2.3
- removed net GPIO1_3: JP2.4
- removed net GPIO1_4: JP2.5
- removed net GPIO1_5: JP2.6
- removed net GPIO1_6: JP2.7
- removed net GPIO1_7: JP2.8
- removed net GPIO1_8: JP2.9
- removed net GPIO1_9: JP2.10
- removed net N$105: JP4.35, JP4.39
- removed net N$110: JP4.33, JP4.37
- removed net N$114: JP4.36, JP4.40
- removed net N$115: JP4.34, JP4.38
- net CLK2: now also JP3.24
- net CLK3: now also JP2.9
- net DOUT2_1: now also JP3.23
- net DOUT2_2: now also JP3.22
- net DOUT2_3: now also JP3.21
- net DOUT2_4: now also JP3.20
- net DOUT2_5: now also JP3.19
- net DOUT2_6: now also JP3.18
- net DOUT2_7: now also JP3.17
- net DOUT2_8: now also JP3.16
- net DOUT3_1: now also JP2.13
- net DOUT3_2: now also JP2.16
- net DOUT3_3: now also JP2.15
- net DOUT3_4: now also JP2.18
- net DRDY2: now also JP3.26
- net DRDY3: now also JP2.14
- net LAZO1: now also JP2.2
- net LAZO2: now also JP2.1
- net LAZO3: now also JP2.4
- net LAZO4: now also JP2.3
- net LAZO5: now also JP2.6
- net LAZO6: now also JP2.5
- net LAZO7: now also JP2.8
- net LAZO8: now also JP2.7
- net SCLK2: now also JP3.25
- net SCLK3: now also JP2.10
- net SYNC2: now also JP3.15
Changed lines of the file:
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@@
 <?xml version="1.0" encoding="utf-8"?>
 <!DOCTYPE eagle SYSTEM "eagle.dtd">
-<eagle version="9.6.2">
+<eagle version="9.5.2">
 <drawing>
 <settings>
@@
 </segment>
 </net>
-<net name="GPIO1_0" class="0">
+<net name="LAZO2" class="0">
 <segment>
 <pinref part="JP2" gate="A" pin="1"/>
@@
 </segment>
 </net>
-<net name="GPIO1_2" class="0">
+<net name="LAZO4" class="0">
 <segment>
 <pinref part="JP2" gate="A" pin="3"/>
@@
 </segment>
 </net>
-<net name="GPIO1_4" class="0">
+<net name="LAZO6" class="0">
 <segment>
 <pinref part="JP2" gate="A" pin="5"/>
@@
 </segment>
 </net>
-<net name="GPIO1_6" class="0">
+<net name="LAZO8" class="0">
 <segment>
 <pinref part="JP2" gate="A" pin="7"/>
@@
 </segment>
 </net>
-<net name="GPIO1_8" class="0">
+<net name="CLK3" class="0">
 <segment>
 <pinref part="JP2" gate="A" pin="9"/>
@@
 </segment>
 </net>
-<net name="GPIO1_10" class="0">
+<net name="DOUT3_1" class="0">
 <segment>
 <pinref part="JP2" gate="A" pin="13"/>
@@
 </segment>
 </net>
-<net name="GPIO1_12" class="0">
+<net name="DOUT3_3" class="0">
 <segment>
 <pinref part="JP2" gate="A" pin="15"/>
@@
 </segment>
 </net>
-<net name="GPIO1_1" class="0">
+<net name="LAZO1" class="0">
 <segment>
 <pinref part="JP2" gate="A" pin="2"/>
@@
 </segment>
 </net>
-<net name="GPIO1_3" class="0">
+<net name="LAZO3" class="0">
 <segment>
 <pinref part="JP2" gate="A" pin="4"/>
@@
 </segment>
 </net>
-<net name="GPIO1_5" class="0">
+<net name="LAZO5" class="0">
 <segment>
 <pinref part="JP2" gate="A" pin="6"/>
@@
 </segment>
 </net>
-<net name="GPIO1_7" class="0">
+<net name="LAZO7" class="0">
 <segment>
 <pinref part="JP2" gate="A" pin="8"/>
@@
 </segment>
 </net>
-<net name="GPIO1_9" class="0">
+<net name="SCLK3" class="0">
 <segment>
 <pinref part="JP2" gate="A" pin="10"/>
@@
 </segment>
 </net>
-<net name="GPIO1_11" class="0">
+<net name="DRDY3" class="0">
 <segment>
 <pinref part="JP2" gate="A" pin="14"/>
@@
 </segment>
 </net>
-<net name="GPIO1_13" class="0">
+<net name="DOUT3_2" class="0">
 <segment>
 <pinref part="JP2" gate="A" pin="16"/>
@@
 </segment>
 </net>
-<net name="GPIO1_15" class="0">
+<net name="DOUT3_4" class="0">
 <segment>
 <pinref part="JP2" gate="A" pin="18"/>
@@
 </segment>
 </net>
-<net name="GPIO1_29" class="0">
+<net name="LAZO_8" class="0">
 <segment>
 <pinref part="JP2" gate="A" pin="34"/>
@@
 </segment>
 </net>
-<net name="GPIO0_14" class="0">
+<net name="DOUT2_7" class="0">
 <segment>
 <pinref part="JP3" gate="A" pin="17"/>
@@
 </segment>
 </net>
-<net name="GPIO0_16" class="0">
+<net name="DOUT2_5" class="0">
 <segment>
 <pinref part="JP3" gate="A" pin="19"/>
@@
 </segment>
 </net>
-<net name="GPIO0_18" class="0">
+<net name="DOUT2_3" class="0">
 <segment>
 <pinref part="JP3" gate="A" pin="21"/>
@@
 </segment>
 </net>
-<net name="GPIO0_20" class="0">
+<net name="DOUT2_1" class="0">
 <segment>
 <pinref part="JP3" gate="A" pin="23"/>
@@
 </segment>
 </net>
-<net name="GPIO0_22" class="0">
+<net name="SCLK2" class="0">
 <segment>
 <pinref part="JP3" gate="A" pin="25"/>
@@
 </segment>
 </net>
-<net name="GPIO0_13" class="0">
+<net name="DOUT2_8" class="0">
 <segment>
 <pinref part="JP3" gate="A" pin="16"/>
@@
 </segment>
 </net>
-<net name="GPIO0_15" class="0">
+<net name="DOUT2_6" class="0">
 <segment>
 <pinref part="JP3" gate="A" pin="18"/>
@@
 </segment>
 </net>
-<net name="GPIO0_17" class="0">
+<net name="DOUT2_4" class="0">
 <segment>
 <pinref part="JP3" gate="A" pin="20"/>
@@
 </segment>
 </net>
-<net name="GPIO0_19" class="0">
+<net name="DOUT2_2" class="0">
 <segment>
 <pinref part="JP3" gate="A" pin="22"/>
@@
 </segment>
 </net>
-<net name="GPIO0_21" class="0">
+<net name="CLK2" class="0">
 <segment>
 <pinref part="JP3" gate="A" pin="24"/>
@@
 </segment>
 </net>
-<net name="GPIO0_23" class="0">
+<net name="DRDY2" class="0">
 <segment>
 <pinref part="JP3" gate="A" pin="26"/>
@@
 </segment>
 </net>
-<net name="GPIO0_12" class="0">
+<net name="SYNC2" class="0">
 <segment>
 <pinref part="JP3" gate="A" pin="15"/>
@@
 </segment>
 </net>
-<net name="N$105" class="0">
-<segment>
-<wire x1="73.66" y1="99.06" x2="38.1" y2="99.06" width="0.1524" layer="91"/>
-<pinref part="JP4" gate="A" pin="35"/>
-</segment>
-<segment>
-<wire x1="73.66" y1="93.98" x2="38.1" y2="93.98" width="0.1524" layer="91"/>
-<pinref part="JP4" gate="A" pin="39"/>
-</segment>
-</net>
-<net name="N$110" class="0">
-<segment>
-<wire x1="73.66" y1="101.6" x2="68.58" y2="101.6" width="0.1524" layer="91"/>
-<pinref part="JP4" gate="A" pin="33"/>
-</segment>
-<segment>
-<wire x1="73.66" y1="96.52" x2="68.58" y2="96.52" width="0.1524" layer="91"/>
-<pinref part="JP4" gate="A" pin="37"/>
-</segment>
-</net>
 <net name="INPUT1-" class="0">
 <segment>
@@
 </segment>
 </net>
-<net name="N$114" class="0">
-<segment>
-<wire x1="81.28" y1="99.06" x2="116.84" y2="99.06" width="0.1524" layer="91"/>
-<pinref part="JP4" gate="A" pin="36"/>
-</segment>
-<segment>
-<wire x1="81.28" y1="93.98" x2="116.84" y2="93.98" width="0.1524" layer="91"/>
-<pinref part="JP4" gate="A" pin="40"/>
-</segment>
-</net>
-<net name="N$115" class="0">
-<segment>
-<wire x1="81.28" y1="101.6" x2="86.36" y2="101.6" width="0.1524" layer="91"/>
-<pinref part="JP4" gate="A" pin="34"/>
-</segment>
-<segment>
-<wire x1="81.28" y1="96.52" x2="86.36" y2="96.52" width="0.1524" layer="91"/>
-<pinref part="JP4" gate="A" pin="38"/>
-</segment>
-</net>

Commit message: tarjeta_v10
Parts:
- U$4: value D36V6F12-12V-600MA -> D24V22F12-12V-2.2A; device myProyects:D36V6F12-12V-600MA -> myProyects:D24V22F12-12V-2.2A
Connections:
- net +12V: now also JP4.35, JP4.36
- net +5V: now also JP4.39, JP4.40
- net GND: now also JP4.33, JP4.34, JP4.37, JP4.38
