File: DATALOGGER_ADS_V1/DATALOGGER_ADS_V1.sch (EAGLE design)
At the start: 339 parts, among them IC1 OPA1632DR, IC10 DE10-NANO, IC11 RASPBERRY_PI_4, IC12 PCF8523, IC13 OPA1632DR, IC14 OPA1632DR, IC15 OPA1632DR, IC16 OPA1632DR, IC17 OPA1632DR, IC18 OPA1632DR, IC19 OPA1632DR, IC2 OPA1632DR, IC20 OPA1632DR, IC21 REF1004U, IC22 OPA1632DR, IC23 OPA1632DR, IC24 OPA1632DR, IC25 OPA1632DR, IC26 REF1004U, IC27 D36V28F5-5V-3.2A, IC28 D24V5F1-1.8V-500MA, IC29 D24V10F3-3.3V-1A, IC3 OPA1632DR, IC30 D24V25F5-5V-2.5A, IC31 TLV2771CDBVR, IC32 TLV2771CDBVR, IC33 TLV2771CDBVR, IC34 TLV2771CDBVR, IC35 FODM217DV, IC36 FODM217DV, IC37 FODM217DV, IC38 FODM217DV, IC39 FODM217DV, IC4 OPA1632DR, IC40 FODM217DV, IC41 FODM217DV, IC42 FODM217DV, IC43 D24V25F5-5V-2.5A, IC5 OPA1632DR, IC6 OPA1632DR, IC7 OPA1632DR, IC8 OPA1632DR, IC9 REF1004U, J1 22-29-2021, J2 22-29-2021, J3 1985027, J4 1989764, J5 1755736, U1 OPA350EA/2K5, U10 VXO78012-500, U2 OPA350EA/2K5, U3 ADS1178IPAPT, U4 OPA350EA/2K5, U5 OPA350EA/2K5, U6 ADS1178IPAPT, U7 OPA350EA/2K5, U8 OPA350EA/2K5, U9 ADS1178IPAPT

Commit message: tarjeta_v11
Parts:
- added J6: 22-29-2021, SamacSys_Parts:22-29-2021
Connections:
- net +12V: now also J6.1
- net GND: now also J6.2
Other:
- moved on the sheet: J5

Commit message: tarjeta_v13
Parts:
- added R163: (no value), rcl:R-US_R0603
- JP6: device pinhead:PINHD-2X4 -> pinhead:PINHD-2X5
Connections:
- new net N$105: JP6.9, R163.2
- net 3.3V_RPI: now also R163.1
- net GND: now also JP6.10
Changed lines of the file:
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@@
 <?xml version="1.0" encoding="utf-8"?>
 <!DOCTYPE eagle SYSTEM "eagle.dtd">
-<eagle version="9.5.2">
+<eagle version="9.6.2">
 <drawing>
 <settings>
@@
 <part name="JP4" library="pinhead" library_urn="urn:adsk.eagle:library:325" deviceset="PINHD-2X20" device="" package3d_urn="urn:adsk.eagle:package:22443/2"/>
 <part name="IC12" library="myProyects" deviceset="PCF8523" device=""/>
-<part name="JP6" library="pinhead" library_urn="urn:adsk.eagle:library:325" deviceset="PINHD-2X4" device="" package3d_urn="urn:adsk.eagle:package:22461/2"/>
+<part name="JP6" library="pinhead" library_urn="urn:adsk.eagle:library:325" deviceset="PINHD-2X5" device="" package3d_urn="urn:adsk.eagle:package:22470/2"/>
 <part name="J1" library="SamacSys_Parts" deviceset="22-29-2021" device=""/>
 <part name="J2" library="SamacSys_Parts" deviceset="22-29-2021" device=""/>
@@
 <part name="SUPPLY130" library="supply2" library_urn="urn:adsk.eagle:library:372" deviceset="GND" device=""/>
 <part name="P+68" library="supply1" library_urn="urn:adsk.eagle:library:371" deviceset="+12V" device=""/>
+<part name="R163" library="rcl" library_urn="urn:adsk.eagle:library:334" deviceset="R-US_" device="R0603" package3d_urn="urn:adsk.eagle:package:23555/3"/>
 </parts>
 <sheets>
@@
 <attribute name="VALUE" x="199.39" y="101.6" size="1.778" layer="96"/>
 </instance>
-<instance part="JP6" gate="A" x="160.02" y="60.96" smashed="yes">
-<attribute name="NAME" x="153.67" y="69.215" size="1.778" layer="95"/>
-<attribute name="VALUE" x="153.67" y="53.34" size="1.778" layer="96"/>
+<instance part="JP6" gate="A" x="172.72" y="60.96" smashed="yes">
+<attribute name="NAME" x="166.37" y="69.215" size="1.778" layer="95"/>
+<attribute name="VALUE" x="166.37" y="53.34" size="1.778" layer="96"/>
 </instance>
 <instance part="J1" gate="G$1" x="73.66" y="33.02" smashed="yes">
@@
 <attribute name="VALUE" x="192.405" y="118.745" size="1.778" layer="96" rot="R270"/>
 </instance>
-<instance part="SUPPLY100" gate="GND" x="172.72" y="53.34" smashed="yes">
-<attribute name="VALUE" x="170.815" y="50.165" size="1.778" layer="96"/>
+<instance part="SUPPLY100" gate="GND" x="185.42" y="50.8" smashed="yes">
+<attribute name="VALUE" x="183.515" y="47.625" size="1.778" layer="96"/>
 </instance>
 <instance part="R139" gate="G$1" x="142.24" y="73.66" smashed="yes">
@@
 <attribute name="VALUE" x="68.58" y="53.34" size="1.778" layer="96" rot="R90"/>
 </instance>
+<instance part="R163" gate="G$1" x="142.24" y="43.18" smashed="yes">
+<attribute name="NAME" x="138.43" y="44.6786" size="1.778" layer="95"/>
+<attribute name="VALUE" x="138.43" y="39.878" size="1.778" layer="96"/>
+</instance>
 </instances>
 <busses>
@@
 <pinref part="JP6" gate="A" pin="2"/>
 <pinref part="SUPPLY100" gate="GND" pin="GND"/>
-<wire x1="165.1" y1="66.04" x2="172.72" y2="66.04" width="0.1524" layer="91"/>
-<wire x1="172.72" y1="66.04" x2="172.72" y2="63.5" width="0.1524" layer="91"/>
+<wire x1="177.8" y1="66.04" x2="185.42" y2="66.04" width="0.1524" layer="91"/>
+<wire x1="185.42" y1="66.04" x2="185.42" y2="63.5" width="0.1524" layer="91"/>
 <pinref part="JP6" gate="A" pin="4"/>
-<wire x1="172.72" y1="63.5" x2="172.72" y2="60.96" width="0.1524" layer="91"/>
-<wire x1="172.72" y1="60.96" x2="172.72" y2="58.42" width="0.1524" layer="91"/>
-<wire x1="172.72" y1="58.42" x2="172.72" y2="55.88" width="0.1524" layer="91"/>
-<wire x1="165.1" y1="63.5" x2="172.72" y2="63.5" width="0.1524" layer="91"/>
-<junction x="172.72" y="63.5"/>
+<wire x1="185.42" y1="63.5" x2="185.42" y2="60.96" width="0.1524" layer="91"/>
+<wire x1="185.42" y1="60.96" x2="185.42" y2="58.42" width="0.1524" layer="91"/>
+<wire x1="185.42" y1="58.42" x2="185.42" y2="55.88" width="0.1524" layer="91"/>
+<wire x1="185.42" y1="55.88" x2="185.42" y2="53.34" width="0.1524" layer="91"/>
+<wire x1="177.8" y1="63.5" x2="185.42" y2="63.5" width="0.1524" layer="91"/>
+<junction x="185.42" y="63.5"/>
 <pinref part="JP6" gate="A" pin="6"/>
-<wire x1="165.1" y1="60.96" x2="172.72" y2="60.96" width="0.1524" layer="91"/>
-<junction x="172.72" y="60.96"/>
+<wire x1="177.8" y1="60.96" x2="185.42" y2="60.96" width="0.1524" layer="91"/>
+<junction x="185.42" y="60.96"/>
 <pinref part="JP6" gate="A" pin="8"/>
-<wire x1="165.1" y1="58.42" x2="172.72" y2="58.42" width="0.1524" layer="91"/>
-<junction x="172.72" y="58.42"/>
+<wire x1="177.8" y1="58.42" x2="185.42" y2="58.42" width="0.1524" layer="91"/>
+<junction x="185.42" y="58.42"/>
+<pinref part="JP6" gate="A" pin="10"/>
+<wire x1="177.8" y1="55.88" x2="185.42" y2="55.88" width="0.1524" layer="91"/>
+<junction x="185.42" y="55.88"/>
 </segment>
 <segment>
@@
 <label x="180.34" y="114.3" size="1.778" layer="95" rot="R180" xref="yes"/>
 </segment>
+<segment>
+<pinref part="R163" gate="G$1" pin="1"/>
+<wire x1="137.16" y1="43.18" x2="134.62" y2="43.18" width="0.1524" layer="91"/>
+<label x="134.62" y="43.18" size="1.778" layer="95" rot="R180" xref="yes"/>
+</segment>
 </net>
 <net name="SDA" class="0">
@@
 <segment>
 <pinref part="JP6" gate="A" pin="1"/>
-<wire x1="157.48" y1="66.04" x2="152.4" y2="66.04" width="0.1524" layer="91"/>
+<wire x1="170.18" y1="66.04" x2="152.4" y2="66.04" width="0.1524" layer="91"/>
 <wire x1="152.4" y1="66.04" x2="152.4" y2="73.66" width="0.1524" layer="91"/>
 <pinref part="R139" gate="G$1" pin="2"/>
@@
 <segment>
 <pinref part="JP6" gate="A" pin="3"/>
-<wire x1="157.48" y1="63.5" x2="149.86" y2="63.5" width="0.1524" layer="91"/>
+<wire x1="170.18" y1="63.5" x2="149.86" y2="63.5" width="0.1524" layer="91"/>
 <wire x1="149.86" y1="63.5" x2="149.86" y2="66.04" width="0.1524" layer="91"/>
 <pinref part="R140" gate="G$1" pin="2"/>
@@
 <segment>
 <pinref part="JP6" gate="A" pin="5"/>
-<wire x1="157.48" y1="60.96" x2="149.86" y2="60.96" width="0.1524" layer="91"/>
+<wire x1="170.18" y1="60.96" x2="149.86" y2="60.96" width="0.1524" layer="91"/>
 <pinref part="R141" gate="G$1" pin="2"/>
 <wire x1="149.86" y1="60.96" x2="149.86" y2="58.42" width="0.1524" layer="91"/>
@@
 <segment>
 <pinref part="JP6" gate="A" pin="7"/>
-<wire x1="157.48" y1="58.42" x2="152.4" y2="58.42" width="0.1524" layer="91"/>
+<wire x1="170.18" y1="58.42" x2="152.4" y2="58.42" width="0.1524" layer="91"/>
 <pinref part="R142" gate="G$1" pin="2"/>
 <wire x1="152.4" y1="58.42" x2="152.4" y2="50.8" width="0.1524" layer="91"/>
@@
 </segment>
 </net>
+<net name="N$105" class="0">
+<segment>
+<pinref part="R163" gate="G$1" pin="2"/>
+<wire x1="147.32" y1="43.18" x2="154.94" y2="43.18" width="0.1524" layer="91"/>
+<wire x1="154.94" y1="43.18" x2="154.94" y2="55.88" width="0.1524" layer="91"/>
+<pinref part="JP6" gate="A" pin="9"/>
+<wire x1="154.94" y1="55.88" x2="170.18" y2="55.88" width="0.1524" layer="91"/>
+</segment>
+</net>

Commit message: tarjeta_v15
Parts:
- R139, R140, R141, R142, R163: value (none) -> 330R
- R147, R148, R149, R150, R151, R152, R153, R154, R155, R156, R157, R158, R159, R160, R161, R162: value (none) -> 220R

Commit message: tarjeta_v17
Parts:
- removed IC1, IC2: OPA1632DR, SamacSys_Parts:OPA1632DR
- removed IC21, IC26, IC9: REF1004U, burr-brown:REF1004U
- removed R103, R133, R49: 100, rcl:R-US_R0603
- removed R107, R137, R53: 20K, rcl:R-US_R0603
- added C114, C115, C116, C117, C118, C119: 1uF, rcl:C-USC0603
- added U11: ADS1278IPAPR, ADS1278IPAPR:ADS1278IPAPR
- added U12, U13: REF5025AID, REF5025:REF5025AID
- added U14, U15: THS4521IDGKT, THS4521IDGKT:THS4521IDGKT
- C33, C74, C99: value 0.1uF -> 10uF
- U3: value ADS1178IPAPT -> REF5025AID; device ADS1178IPAPT:ADS1178IPAPT -> REF5025:REF5025AID
- U6, U9: value ADS1178IPAPT -> ADS1278IPAPR; device ADS1178IPAPT:ADS1178IPAPT -> ADS1278IPAPR:ADS1278IPAPR
Connections:
- removed net N$98: IC26.C1, R137.1
- new net N$103: U11.FORMAT1
- net +12V: no longer IC1.V+, IC2.V+
- net +1V8: now also U11.DVDD; no longer U3.DVDD
- net +3V3: now also U11.!PWDN1, U11.!PWDN2, U11.!PWDN3, U11.!PWDN4, U11.!PWDN5, U11.!PWDN6, U11.!PWDN7, U11.!PWDN8, U11.CLKDIV_2, U11.IOVDD, U11.IOVDD_2, U6.CLKDIV_2, U9.CLKDIV_2; no longer U3.!PWDN1, U3.!PWDN2, U3.!PWDN3, U3.!PWDN4, U3.!PWDN5, U3.!PWDN6, U3.!PWDN7, U3.!PWDN8, U3.CLKDIV, U3.FORMAT1, U3.IOVDD, U3.IOVDD_2, U6.CLKDIV, U6.FORMAT1, U9.CLKDIV, U9.FORMAT1
- net +5V: now also C114.1, C117.1, C119.1, U11.AVDD, U11.AVDD_2, U11.AVDD_3, U11.AVDD_4, U12.VIN, U13.VIN, U14.VS+, U15.VS+, U3.VIN; no longer R107.2, R137.2, R53.2, U3.AVDD, U3.AVDD_2, U3.AVDD_3, U3.AVDD_4
- net -12V: no longer IC1.V-, IC2.V-
- net AINN1_1: now also R2.1, R3.1, U11.AINN1; no longer R5.1, R6.1, U3.AINN1
- net AINN1_2: now also R8.1, R9.1, U11.AINN2; no longer R11.1, R12.1, U3.AINN2
- net AINN1_3: now also U11.AINN3; no longer U3.AINN3
- net AINN1_4: now also U11.AINN4; no longer U3.AINN4
- net AINN1_5: now also U11.AINN5; no longer U3.AINN5
- net AINN1_6: now also U11.AINN6; no longer U3.AINN6
- net AINN1_7: now also U11.AINN7; no longer U3.AINN7
- net AINN1_8: now also U11.AINN8; no longer U3.AINN8
- net AINP1_1: now also R5.1, R6.1, U11.AINP1; no longer R2.1, R3.1, U3.AINP1
- net AINP1_2: now also R11.1, R12.1, U11.AINP2; no longer R8.1, R9.1, U3.AINP2
- net AINP1_3: now also U11.AINP3; no longer U3.AINP3
- net AINP1_4: now also U11.AINP4; no longer U3.AINP4
- net AINP1_5: now also U11.AINP5; no longer U3.AINP5
- net AINP1_6: now also U11.AINP6; no longer U3.AINP6
- net AINP1_7: now also U11.AINP7; no longer U3.AINP7
- net AINP1_8: now also U11.AINP8; no longer U3.AINP8
- net CLK1: now also U11.CLKDIV; no longer U3.CLK
- net CLK2: now also U6.CLKDIV; no longer U6.CLK
- net CLK3: now also U9.CLKDIV; no longer U9.CLK
- net DOUT1_1: now also U11.DOUT1; no longer U3.DOUT1
- net DOUT1_2: now also U11.DOUT2; no longer U3.DOUT2
- net DOUT1_3: now also U11.DOUT3; no longer U3.DOUT3
- net DOUT1_4: now also U11.DOUT4; no longer U3.DOUT4
- net DOUT1_5: now also U11.DOUT5; no longer U3.DOUT5
- net DOUT1_6: now also U11.DOUT6; no longer U3.DOUT6
- net DOUT1_7: now also U11.DOUT7; no longer U3.DOUT7
- net DOUT1_8: now also U11.DOUT8; no longer U3.DOUT8
- net DRDY1: now also U11.!DRDY/FSYNC; no longer U3.!DRDY/FSYNC
- net GND: now also C114.2, C115.2, C116.2, C117.2, C118.2, C119.2, U11.AGND, U11.AGND_2, U11.AGND_3, U11.AGND_4, U11.AGND_5, U11.DGND, U11.DGND_2, U11.DGND_3, U11.DGND_4, U11.DIN, U11.EPAD, U11.FORMAT0, U11.FORMAT2, U11.MODE0, U11.MODE1, U11.TEST0, U11.TEST1, U11.VREFN, U12.GND, U13.GND, U14.VS-, U15.VS-, U3.GND, U6.MODE0, U6.MODE1, U9.MODE0, U9.MODE1; no longer IC21.A, IC26.A, IC9.A, U3.AGND, U3.AGND_2, U3.AGND_3, U3.AGND_4, U3.AGND_5, U3.DGND, U3.DGND_2, U3.DGND_3, U3.DGND_4, U3.DIN, U3.EPAD, U3.FORMAT0, U3.FORMAT2, U3.MODE, U3.TEST0, U3.TEST1, U3.VREFN, U6.MODE, U9.MODE
- net N$1: now also U14.VIN-; no longer IC1.VIN-
- net N$2: now also U14.VIN+; no longer IC1.VIN+
- net N$3: now also U14.VOUT-; no longer IC1.VOUT-
- net N$33: now also C34.1, R50.2; no longer R49.2
- net N$34: now also C99.1, R134.1, U12.VOUT; no longer C33.1, C34.1, R49.1, R50.2
- net N$35: now also C115.1, U3.TRIM/NR; no longer IC9.C, R50.1
- net N$36: now also C33.1, R50.1, U3.VOUT; no longer IC9.C1, R53.1
- net N$4: now also U14.VOUT+; no longer IC1.VOUT+
- net N$5: now also U15.VIN+; no longer IC2.VIN+
- net N$6: now also U15.VOUT-; no longer IC2.VOUT-
- net N$7: now also U15.VIN-; no longer IC2.VIN-
- net N$72: now also C75.1, R104.2; no longer R103.2
- net N$73: now also R104.1, U13.VOUT; no longer C75.1, R103.1, R104.2
- net N$74: now also C118.1, U13.TRIM/NR; no longer IC21.C, R104.1
- net N$75: now also U6.FORMAT1; no longer IC21.C1, R107.1
- net N$8: now also U15.VOUT+; no longer IC2.VOUT+
- net N$95: now also C100.1, R134.2; no longer R133.2
- net N$96: now also C116.1, U12.TRIM/NR; no longer C100.1, C99.1, R133.1, R134.2
- net N$97: now also U9.FORMAT1; no longer IC26.C, R134.1
- net SCLK1: now also U11.SCLK; no longer U3.SCLK
- net SYNC1: now also U11.!SYNC; no longer U3.!SYNC
- net VCOM1: now also U14.VOCM, U15.VOCM; no longer IC1.VOCM, IC2.VOCM
- net VCOMM1: now also U11.VCOM; no longer U3.VCOM
- net VREFP1: now also U11.VREFP; no longer U3.VREFP
Other:
- moved on the sheet: C1, C100, C101, C102, C103, C2, C3, C33, C34, C35, C36, C37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

Commit message: tarjeta_v17
Parts:
- removed IC13, IC14, IC15, IC16, IC17, IC18, IC19, IC20, IC22, IC23, IC24, IC25, IC3, IC4, IC5, IC6, IC7, IC8: OPA1632DR, SamacSys_Parts:OPA1632DR
- added U16, U17, U18, U19, U20, U21, U22, U23, U24, U25, U26, U27, U28, U29, U30, U31, U32, U33: THS4521IDGKT, THS4521IDGKT:THS4521IDGKT
- C108, C109, C110, C111: value (none) -> 20nF
- R143, R144, R145, R146: value (none) -> 10M
Connections:
- removed net N$103: U11.FORMAT1
- removed net N$97: U9.FORMAT1
- net +12V: no longer IC13.V+, IC14.V+, IC15.V+, IC16.V+, IC17.V+, IC18.V+, IC19.V+, IC20.V+, IC22.V+, IC23.V+, IC24.V+, IC25.V+, IC3.V+, IC4.V+, IC5.V+, IC6.V+, IC7.V+, IC8.V+
- net +3V3: now also U11.FORMAT1, U9.FORMAT1
- net +5V: now also U16.VS+, U17.VS+, U18.VS+, U19.VS+, U20.VS+, U21.VS+, U22.VS+, U23.VS+, U24.VS+, U25.VS+, U26.VS+, U27.VS+, U28.VS+, U29.VS+, U30.VS+, U31.VS+, U32.VS+, U33.VS+
- net -12V: no longer IC13.V-, IC14.V-, IC15.V-, IC16.V-, IC17.V-, IC18.V-, IC19.V-, IC20.V-, IC22.V-, IC23.V-, IC24.V-, IC25.V-, IC3.V-, IC4.V-, IC5.V-, IC6.V-, IC7.V-, IC8.V-
- net AINN1_3: now also R14.1, R15.1; no longer R17.1, R18.1
- net AINN1_4: now also R20.1, R21.1; no longer R23.1, R24.1
- net AINN1_5: now also R26.1, R27.1; no longer R29.1, R30.1
- net AINN1_6: now also R32.1, R33.1; no longer R35.1, R36.1
- net AINN1_7: now also R38.1, R39.1; no longer R41.1, R42.1
- net AINN1_8: now also R44.1, R45.1; no longer R47.1, R48.1
- net AINN3_1: now also R110.1, R111.1; no longer R113.1, R114.1
- net AINN3_2: now also R116.1, R117.1; no longer R119.1, R120.1
- net AINP1_3: now also R17.1, R18.1; no longer R14.1, R15.1
- net AINP1_4: now also R23.1, R24.1; no longer R20.1, R21.1
- net AINP1_5: now also R29.1, R30.1; no longer R26.1, R27.1
- net AINP1_6: now also R35.1, R36.1; no longer R32.1, R33.1
- net AINP1_7: now also R41.1, R42.1; no longer R38.1, R39.1
- net AINP1_8: now also R47.1, R48.1; no longer R44.1, R45.1
- net AINP3_1: now also R113.1, R114.1; no longer R110.1, R111.1
- net AINP3_2: now also R119.1, R120.1; no longer R116.1, R117.1
- net GND: now also U16.VS-, U17.VS-, U18.VS-, U19.VS-, U20.VS-, U21.VS-, U22.VS-, U23.VS-, U24.VS-, U25.VS-, U26.VS-, U27.VS-, U28.VS-, U29.VS-, U30.VS-, U31.VS-, U32.VS-, U33.VS-
- net N$10: now also U16.VOUT-; no longer IC3.VOUT-
- net N$11: now also U16.VIN-; no longer IC3.VIN-
- net N$12: now also U16.VOUT+; no longer IC3.VOUT+
- net N$13: now also U17.VIN+; no longer IC4.VIN+
- net N$14: now also U17.VOUT-; no longer IC4.VOUT-
- net N$15: now also U17.VIN-; no longer IC4.VIN-
- net N$16: now also U17.VOUT+; no longer IC4.VOUT+
- net N$17: now also U18.VIN+; no longer IC5.VIN+
- net N$18: now also U18.VOUT-; no longer IC5.VOUT-
- net N$19: now also U18.VIN-; no longer IC5.VIN-
- net N$20: now also U18.VOUT+; no longer IC5.VOUT+
- net N$21: now also U19.VIN+; no longer IC6.VIN+
- net N$22: now also U19.VOUT-; no longer IC6.VOUT-
- net N$23: now also U19.VIN-; no longer IC6.VIN-
- net N$24: now also U19.VOUT+; no longer IC6.VOUT+
- net N$25: now also U20.VIN+; no longer IC7.VIN+
- net N$26: now also U20.VOUT-; no longer IC7.VOUT-
- net N$27: now also U20.VIN-; no longer IC7.VIN-
- net N$28: now also U20.VOUT+; no longer IC7.VOUT+
- net N$29: now also U21.VIN+; no longer IC8.VIN+
- net N$30: now also U21.VOUT-; no longer IC8.VOUT-
- net N$31: now also U21.VIN-; no longer IC8.VIN-
- net N$32: now also U21.VOUT+; no longer IC8.VOUT+
- net N$40: now also U22.VIN+; no longer IC13.VIN+
- net N$41: now also U22.VOUT-; no longer IC13.VOUT-
- net N$42: now also U22.VIN-; no longer IC13.VIN-
- net N$43: now also U22.VOUT+; no longer IC13.VOUT+
- net N$44: now also U23.VIN+; no longer IC14.VIN+
- net N$45: now also U23.VOUT-; no longer IC14.VOUT-
- net N$46: now also U23.VIN-; no longer IC14.VIN-
- net N$47: now also U23.VOUT+; no longer IC14.VOUT+
- net N$48: now also U24.VIN+; no longer IC15.VIN+
- net N$49: now also U24.VOUT-; no longer IC15.VOUT-
- net N$50: now also U24.VIN-; no longer IC15.VIN-
- net N$51: now also U24.VOUT+; no longer IC15.VOUT+
- net N$52: now also U25.VIN+; no longer IC16.VIN+
- net N$53: now also U25.VOUT-; no longer IC16.VOUT-
- net N$54: now also U25.VIN-; no longer IC16.VIN-
- net N$55: now also U25.VOUT+; no longer IC16.VOUT+
- net N$56: now also U26.VIN+; no longer IC17.VIN+
- net N$57: now also U26.VOUT-; no longer IC17.VOUT-
- net N$58: now also U26.VIN-; no longer IC17.VIN-
- net N$59: now also U26.VOUT+; no longer IC17.VOUT+
- net N$60: now also U27.VIN+; no longer IC18.VIN+
- net N$61: now also U27.VOUT-; no longer IC18.VOUT-
- net N$62: now also U27.VIN-; no longer IC18.VIN-
- net N$63: now also U27.VOUT+; no longer IC18.VOUT+
- net N$64: now also U28.VIN+; no longer IC19.VIN+
- net N$65: now also U28.VOUT-; no longer IC19.VOUT-
- net N$66: now also U28.VIN-; no longer IC19.VIN-
- net N$67: now also U28.VOUT+; no longer IC19.VOUT+
- net N$68: now also U29.VIN+; no longer IC20.VIN+
- net N$69: now also U29.VOUT-; no longer IC20.VOUT-
- net N$70: now also U29.VIN-; no longer IC20.VIN-
- net N$71: now also U29.VOUT+; no longer IC20.VOUT+
- net N$79: now also U30.VIN+; no longer IC22.VIN+
- net N$80: now also U30.VOUT-; no longer IC22.VOUT-
- net N$81: now also U30.VIN-; no longer IC22.VIN-
- net N$82: now also U30.VOUT+; no longer IC22.VOUT+
- net N$83: now also U31.VIN+; no longer IC23.VIN+
- net N$84: now also U31.VOUT-; no longer IC23.VOUT-
- net N$85: now also U31.VIN-; no longer IC23.VIN-
- net N$86: now also U31.VOUT+; no longer IC23.VOUT+
- net N$87: now also U32.VIN+; no longer IC24.VIN+
- net N$88: now also U32.VOUT-; no longer IC24.VOUT-
- net N$89: now also U32.VIN-; no longer IC24.VIN-
- net N$9: now also U16.VIN+; no longer IC3.VIN+
- net N$90: now also U32.VOUT+; no longer IC24.VOUT+
- net N$91: now also U33.VIN+; no longer IC25.VIN+
- net N$92: now also U33.VOUT-; no longer IC25.VOUT-
- net N$93: now also U33.VIN-; no longer IC25.VIN-
- net N$94: now also U33.VOUT+; no longer IC25.VOUT+
- net VCOM1: now also U16.VOCM, U17.VOCM, U18.VOCM, U19.VOCM, U20.VOCM, U21.VOCM; no longer IC3.VOCM, IC4.VOCM, IC5.VOCM, IC6.VOCM, IC7.VOCM, IC8.VOCM
- net VCOM2: now also U22.VOCM, U23.VOCM, U24.VOCM, U25.VOCM, U26.VOCM, U27.VOCM, U28.VOCM, U29.VOCM; no longer IC13.VOCM, IC14.VOCM, IC15.VOCM, IC16.VOCM, IC17.VOCM, IC18.VOCM, IC19.VOCM, IC20.VOCM
- net VCOM3: now also U30.VOCM, U31.VOCM, U32.VOCM, U33.VOCM; no longer IC22.VOCM, IC23.VOCM, IC24.VOCM, IC25.VOCM
Other:
- moved on the sheet: C10, C11, C12, C13, C14, C15, C16, C17, C18, C19, C20, C21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

Commit message: tarjeta_v17
Connections:
- removed net N$75: U6.FORMAT1
- net +3V3: now also U6.FORMAT1
- net AINN2_1: now also R56.1, R57.1; no longer R59.1, R60.1
- net AINN2_2: now also R62.1, R63.1; no longer R65.1, R66.1
- net AINN2_3: now also R68.1, R69.1; no longer R71.1, R72.1
- net AINN2_4: now also R74.1, R75.1; no longer R77.1, R78.1
- net AINN2_5: now also R80.1, R81.1; no longer R83.1, R84.1
- net AINN2_6: now also R86.1, R87.1; no longer R89.1, R90.1
- net AINN2_7: now also R92.1, R93.1; no longer R95.1, R96.1
- net AINN2_8: now also R98.1, R99.1; no longer R101.1, R102.1
- net AINN3_3: now also R122.1, R123.1; no longer R125.1, R126.1
- net AINN3_4: now also R128.1, R129.1; no longer R131.1, R132.1
- net AINP2_1: now also R59.1, R60.1; no longer R56.1, R57.1
- net AINP2_2: now also R65.1, R66.1; no longer R62.1, R63.1
- net AINP2_3: now also R71.1, R72.1; no longer R68.1, R69.1
- net AINP2_4: now also R77.1, R78.1; no longer R74.1, R75.1
- net AINP2_5: now also R83.1, R84.1; no longer R80.1, R81.1
- net AINP2_6: now also R89.1, R90.1; no longer R86.1, R87.1
- net AINP2_7: now also R95.1, R96.1; no longer R92.1, R93.1
- net AINP2_8: now also R101.1, R102.1; no longer R98.1, R99.1
- net AINP3_3: now also R125.1, R126.1; no longer R122.1, R123.1
- net AINP3_4: now also R131.1, R132.1; no longer R128.1, R129.1

Commit message: tarjeta_v18
Parts:
- removed C108, C109, C110, C111: 20nF, rcl:C-USC0805
- removed IC12: PCF8523, myProyects:PCF8523
- added IC1: DS3231, myProyects:DS3231
- added JP5: (no value), pinhead:PINHD-1X3
- added R103, R133, R137, R49: 50M, rcl:R-US_R0805
- added R107, R164, R165, R53: 1K, rcl:R-US_R0805
- R143, R144, R145, R146: value 10M -> 100M
Connections:
- removed net SQW: IC12.SQW
- removed net TX: JP1.8
- new net 5V_RPI: JP1.4, JP5.3
- new net N$111: IC34.IN-, R137.1, R164.2
- new net N$75: IC33.IN-, R133.1, R165.2
- new net N$97: IC31.IN-, R49.1, R53.2
- new net N$98: IC32.IN-, R103.1, R107.2
- new net SIGNAL: JP1.8, JP5.1
- net +3V3: now also IC31.VDD, IC32.VDD, IC33.VDD, IC34.VDD
- net +5V: no longer IC31.VDD, IC32.VDD, IC33.VDD, IC34.VDD
- net 3.3V_RPI: now also IC1.VIN; no longer IC12.VCC
- net DOBLE1: now also IC31.IN+, R143.1; no longer C108.1, IC31.IN-, R143.2
- net DOBLE2: now also IC32.IN+, R144.1; no longer C109.1, IC32.IN-, R144.2
- net DOBLE3: now also IC33.IN+, R145.1; no longer C110.1, IC33.IN-, R145.2
- net DOBLE4: now also IC34.IN+, R146.1; no longer C111.1, IC34.IN-, R146.2
- net GND: now also IC1.GND, JP5.2, R107.1, R143.2, R144.2, R145.2, R146.2, R164.1, R165.1, R53.1; no longer IC12.GND, IC31.IN+, IC32.IN+, IC33.IN+, IC34.IN+
- net INPUT17+: now also R49.2; no longer C108.2, R143.1
- net INPUT18+: now also R103.2; no longer C109.2, R144.1
- net INPUT19+: now also R133.2; no longer C110.2, R145.1
- net INPUT20+: now also R137.2; no longer C111.2, R146.1
- net SCL: now also IC1.SCL; no longer IC12.SCL
- net SDA: now also IC1.SDA; no longer IC12.SDA
Other:
- moved on the sheet: R143, R144, R145, R146
