File: DATALOGGER_ADS_V1/DATALOGGER_ADS_V1.sch (EAGLE design)
At the start: 343 parts, among them IC1 DS3231, IC10 DE10-NANO, IC11 RASPBERRY_PI_4, IC27 D36V28F5-5V-3.2A, IC28 D24V5F1-1.8V-500MA, IC29 D24V10F3-3.3V-1A, IC30 D24V25F5-5V-2.5A, IC31 TLV2771CDBVR, IC32 TLV2771CDBVR, IC33 TLV2771CDBVR, IC34 TLV2771CDBVR, IC35 FODM217DV, IC36 FODM217DV, IC37 FODM217DV, IC38 FODM217DV, IC39 FODM217DV, IC40 FODM217DV, IC41 FODM217DV, IC42 FODM217DV, IC43 D24V25F5-5V-2.5A, J1 22-29-2021, J2 22-29-2021, J3 1985027, J4 1989764, J5 1755736, J6 22-29-2021, U1 OPA350EA/2K5, U11 ADS1278IPAPR, U12 REF5025AID, U13 REF5025AID, U14 THS4521IDGKT, U15 THS4521IDGKT, U16 THS4521IDGKT, U17 THS4521IDGKT, U18 THS4521IDGKT, U19 THS4521IDGKT, U2 OPA350EA/2K5, U20 THS4521IDGKT, U21 THS4521IDGKT, U22 THS4521IDGKT, U23 THS4521IDGKT, U24 THS4521IDGKT, U25 THS4521IDGKT, U26 THS4521IDGKT, U27 THS4521IDGKT, U28 THS4521IDGKT, U29 THS4521IDGKT, U3 REF5025AID, U30 THS4521IDGKT, U31 THS4521IDGKT, U32 THS4521IDGKT, U33 THS4521IDGKT, U4 OPA350EA/2K5, U5 OPA350EA/2K5, U6 ADS1278IPAPR, U7 OPA350EA/2K5, U8 OPA350EA/2K5, U9 ADS1278IPAPR

Commit message: datalogger_ads_v2
Connections:
- removed net GPIO1_14: JP2.17
- net SYNC3: now also JP2.17
Changed lines of the file:
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@@
 </segment>
 </net>
-<net name="GPIO1_14" class="0">
+<net name="SYNC3" class="0">
 <segment>
 <pinref part="JP2" gate="A" pin="17"/>
