File: DATALOGGER_CA_V1/DATALOGGER_CA_ADC_V1.brd (EAGLE design)
At the start: 160 x 100 mm, 131 parts, among them IC1 TLV2771CDBVR, IC10 MCP601OT, IC11 TLV2771CDBVR, IC12 MCP601OT, IC13 TLV2771CDBVR, IC14 MCP601OT, IC15 TLV2771CDBVR, IC16 MCP601OT, IC17 TLV2771CDBVR, IC18 MCP601OT, IC19 TLV2771CDBVR, IC2 TLV2771CDBVR, IC20 MCP601OT, IC21 TLV2771CDBVR, IC22 MCP601OT, IC23 TLV2771CDBVR, IC24 MCP601OT, IC25 TLV2771CDBVR, IC26 MCP601OT, IC27 TLV2771CDBVR, IC28 MCP601OT, IC29 TLV2771CDBVR, IC3 MCP601OT, IC30 MCP601OT, IC31 TLV2771CDBVR, IC32 MCP601OT, IC4 MCP601OT, IC5 TLV2771CDBVR, IC6 MCP601OT, IC7 TLV2771CDBVR, IC8 MCP601OT, IC9 TLV2771CDBVR, J1 1985027, J2 1985027

Commit message: tarjeta_v13
Parts:
- moved C47 174.6 mm to (68.8, 30.7), flipped to the bottom, turned to 270 degrees
- moved C46 171.8 mm to (69.9, 23.5), flipped to the bottom
- moved IC29 166.5 mm to (68.0, 20.3), turned to 270 degrees
- moved C45 159.4 mm to (66.9, 34.8), turned to 90 degrees
- moved C33 157.7 mm to (54.0, 34.8), turned to 90 degrees
- moved C44 156.8 mm to (69.2, 30.7), turned to 270 degrees
- moved IC26 156.7 mm to (63.1, 34.9)
- moved R38 154.8 mm to (60.5, 30.8), turned to 90 degrees
- moved C32 154.8 mm to (56.3, 30.7), turned to 270 degrees
- moved C43 152.1 mm to (68.1, 23.5)
- moved C31 149.8 mm to (55.2, 23.5)
- moved IC19 149.4 mm to (50.8, 20.4), flipped to the bottom, turned to 270 degrees
- moved IC27 149.0 mm to (63.5, 20.4), flipped to the bottom, turned to 270 degrees
- moved R28 148.8 mm to (50.8, 25.6), flipped to the bottom
- moved R35 144.8 mm to (58.1, 30.7), flipped to the bottom, turned to 90 degrees
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Routing:
- net +5V: track 0.00 -> 213.7 mm, vias 0 -> 17
- net INPUT1+: track 0.00 -> 87.6 mm
- net INPUT9+: track 0.00 -> 87.0 mm
- net INPUT10+: track 0.00 -> 86.8 mm, vias 0 -> 2
- net INPUT3+: track 0.00 -> 85.3 mm
- net INPUT2+: track 0.00 -> 85.0 mm
- net INPUT5+: track 0.00 -> 83.7 mm
- net INPUT4+: track 0.00 -> 83.7 mm, vias 0 -> 2
- net INPUT7+: track 0.00 -> 82.6 mm
- net INPUT6+: track 0.00 -> 82.1 mm, vias 0 -> 2
- net INPUT8+: track 0.00 -> 80.3 mm, vias 0 -> 2
- net INPUT16+: track 0.00 -> 43.1 mm, vias 0 -> 6
- net INPUT15+: track 0.00 -> 40.5 mm, vias 0 -> 4
- net INPUT14+: track 0.00 -> 33.4 mm, vias 0 -> 4
- net INPUT13+: track 0.00 -> 30.5 mm, vias 0 -> 2
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- added copper zone on layer 1, net GND
- added copper zone on layer 16, net GND
Other:
- board size 160 x 100 mm -> 81.7 x 54 mm
