File: DATALOGGER_CA_V1/DATALOGGER_CA_ADC_V1.brd (EAGLE design)
At the start: 134 x 50 mm, 229 parts, among them IC1 TLV2771CDBVR, IC10 MCP601OT, IC11 TLV2771CDBVR, IC12 MCP601OT, IC13 TLV2771CDBVR, IC14 MCP601OT, IC15 TLV2771CDBVR, IC16 MCP601OT, IC17 TLV2771CDBVR, IC18 MCP601OT, IC19 TLV2771CDBVR, IC2 TLV2771CDBVR, IC20 MCP601OT, IC21 TLV2771CDBVR, IC22 MCP601OT, IC23 TLV2771CDBVR, IC24 MCP601OT, IC25 TLV2771CDBVR, IC26 MCP601OT, IC27 TLV2771CDBVR, IC28 MCP601OT, IC29 TLV2771CDBVR, IC3 MCP601OT, IC30 MCP601OT, IC31 TLV2771CDBVR, IC32 MCP601OT, IC4 MCP601OT, IC5 TLV2771CDBVR, IC6 MCP601OT, IC7 TLV2771CDBVR, IC8 MCP601OT, IC9 TLV2771CDBVR, J1 1985027, J2 1985027, J3 1985027, J4 1985027, U1 REF5025AID, U10 REF5025AID, U11 REF5025AID, U12 REF5025AID, U13 REF5025AID, U14 REF5025AID, U15 REF5025AID, U16 REF5025AID, U2 REF5025AID, U3 REF5025AID, U4 REF5025AID, U5 REF5025AID, U6 REF5025AID, U7 REF5025AID, U8 REF5025AID, U9 REF5025AID

Commit message: tarjeta_v22
Parts:
- C11, C14, C17, C2, C20, C23, C26, C29, C32, C35, C38, C41, C44, C47, C5, C8: value 18uF -> 0.018uF
- R10: value 200M -> 10M
- moved C21 0.41 mm to (54.1, 36.2)
- moved R50 0.38 mm to (10.5, 18.2)
- moved C19 0.32 mm to (61.7, 26.1)
- moved R19 0.32 mm to (61.7, 28.2)
- moved C7 0.31 mm to (30.3, 27.5)
- moved R7 0.31 mm to (30.3, 25.4)
- moved C54 0.29 mm to (30.3, 29.6)
- moved C53 0.28 mm to (30.3, 31.8)
- moved C64 0.24 mm to (61.7, 30.3)
- moved R31 0.22 mm to (91.7, 27.8)
- moved C31 0.20 mm to (91.7, 25.7)
- moved C70 0.18 mm to (91.7, 29.9)
- moved R27 0.18 mm to (72.6, 28.9)
- moved C63 0.17 mm to (61.7, 32.3)
- moved C12 0.13 mm to (31.0, 35.2)
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Routing:
- net +5V: track 559.3 -> 562.0 mm
- net INPUT1+: track 204.4 -> 206.3 mm
- net N$1: track 20.5 -> 21.6 mm
- net N$31: track 47.3 -> 48.2 mm
