File: DATALOGGER_CA_V1/DATALOGGER_CA_ADC_V1.sch (EAGLE design)
At the start: 131 parts, among them IC1 TLV2771CDBVR, IC10 MCP601OT, IC11 TLV2771CDBVR, IC12 MCP601OT, IC13 TLV2771CDBVR, IC14 MCP601OT, IC15 TLV2771CDBVR, IC16 MCP601OT, IC17 TLV2771CDBVR, IC18 MCP601OT, IC19 TLV2771CDBVR, IC2 TLV2771CDBVR, IC20 MCP601OT, IC21 TLV2771CDBVR, IC22 MCP601OT, IC23 TLV2771CDBVR, IC24 MCP601OT, IC25 TLV2771CDBVR, IC26 MCP601OT, IC27 TLV2771CDBVR, IC28 MCP601OT, IC29 TLV2771CDBVR, IC3 MCP601OT, IC30 MCP601OT, IC31 TLV2771CDBVR, IC32 MCP601OT, IC4 MCP601OT, IC5 TLV2771CDBVR, IC6 MCP601OT, IC7 TLV2771CDBVR, IC8 MCP601OT, IC9 TLV2771CDBVR, J1 1985027, J2 1985027

Commit message: TARJETA_V20
Parts:
- added C49, C51, C53, C55, C57, C59, C61, C63: 18nF, rcl:C-USC0805
- added C50, C52, C54, C56, C58, C60, C62, C64: 12nF, rcl:C-USC0805
- added C65, C66, C67, C68: 20nF, rcl:C-USC0805
- added R49, R50, R51, R52, R53, R54, R55, R56: 1K, rcl:R-US_R0805
- added R57, R58: 200M, rcl:R-US_R0805
- C1, C10, C13, C16, C19, C22, C4, C7: value 20nF -> 150nF
- R1, R13, R16, R19, R22, R4, R7: value 200M -> 10M
Connections:
- new net N$49: C4.1, C51.1, C52.1, IC2.IN-, R4.1, R50.2
- new net N$50: C1.1, C49.1, C50.1, IC1.IN-, R1.1, R49.2
- new net N$51: C53.1, C54.1, C7.1, IC5.IN-, R51.2, R7.1
- new net N$52: C10.1, C55.1, C56.1, IC7.IN-, R10.1, R52.2
- new net N$53: C13.1, C57.1, C58.1, IC9.IN-, R13.1, R53.2
- new net N$54: C19.1, C63.1, C64.1, IC13.IN-, R19.1, R55.2
- new net N$55: C22.1, C61.1, C62.1, IC15.IN-, R22.1, R56.2
- new net N$56: C16.1, C59.1, C60.1, IC11.IN-, R16.1, R54.2
- new net REF_S1: IC1.IN+
- new net REF_S2: IC2.IN+
- new net REF_S3: IC5.IN+
- new net REF_S4: IC7.IN+
- new net REF_S5: IC9.IN+
- new net REF_S6: IC11.IN+
- new net REF_S7: IC13.IN+
- new net REF_S8: IC15.IN+
- net GND: no longer IC1.IN+, IC11.IN+, IC13.IN+, IC15.IN+, IC17.GND, IC17.IN+, IC19.GND, IC19.IN+, IC2.IN+, IC5.IN+, IC7.IN+, IC9.IN+
- net N$1: now also C53.2, C54.2
- net N$10: now also C55.2, C56.2
- net N$13: now also C57.2, C58.2
- net N$16: now also C59.2, C60.2
- net N$19: now also C63.2, C64.2
- net N$2: now also C49.2, C50.2
- net N$22: now also C61.2, C62.2
- net N$6: now also C51.2, C52.2
- net S1: now also R49.1; no longer C1.1, IC1.IN-, R1.1
- net S10: no longer C28.1, IC19.IN-, R28.1
- net S2: now also R50.1; no longer C4.1, IC2.IN-, R4.1
- net S3: now also R51.1; no longer C7.1, IC5.IN-, R7.1
- net S4: now also R52.1; no longer C10.1, IC7.IN-, R10.1
- net S5: now also R53.1; no longer C13.1, IC9.IN-, R13.1
- net S6: now also R54.1; no longer C16.1, IC11.IN-, R16.1
- net S7: now also R55.1; no longer C19.1, IC13.IN-, R19.1
- net S8: now also R56.1; no longer C22.1, IC15.IN-, R22.1
- net S9: no longer C25.1, IC17.IN-, R25.1
Other:
- moved on the sheet: C1, C10, C11, C12, C13, C14, C15, C16, C17, C18, C19, C2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
