File: DATALOGGER_CA_V1/DATALOGGER_CA_ADC_V1.sch (EAGLE design)
At the start: 229 parts, among them IC1 TLV2771CDBVR, IC10 MCP601OT, IC11 TLV2771CDBVR, IC12 MCP601OT, IC13 TLV2771CDBVR, IC14 MCP601OT, IC15 TLV2771CDBVR, IC16 MCP601OT, IC17 TLV2771CDBVR, IC18 MCP601OT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

Commit message: tarjeta_v22
Parts:
- C11, C14, C17, C2, C20, C23, C26, C29, C32, C35, C38, C41, C44, C47, C5, C8: value 18uF -> 0.018uF
- R10: value 200M -> 10M
