File: DATALOGGER_BP_V1/DATALOGGER_BP_V1.brd (EAGLE design)
At the start: 130 x 50 mm, 36 parts, among them J1 1985247, J2 1985247, J3 1985247, J4 1985247, J5 1985247, J6 1985247, J7 1985247, J8 1985247, J9 1755736

Commit message: tarjeta_v16
Parts:
- added C10, C11, C12, C13, C14, C15, C16, C17, C18, C19, C20, C21, C22, C23, C24, C9: 0.01uF, rcl:C0805
Connections:
- net GND: now also C10.2, C11.2, C12.2, C13.2, C14.2, C15.2, C16.2, C17.2, C18.2, C19.2, C20.2, C21.2, C22.2, C23.2, C24.2, C9.2
- net INPUT1+: now also C10.1
- net INPUT1-: now also C9.1
- net INPUT2+: now also C12.1
- net INPUT2-: now also C11.1
- net INPUT3+: now also C14.1
- net INPUT3-: now also C13.1
- net INPUT4+: now also C16.1
- net INPUT4-: now also C15.1
- net INPUT5+: now also C18.1
- net INPUT5-: now also C17.1
- net INPUT6+: now also C20.1
- net INPUT6-: now also C19.1
- net INPUT7+: now also C22.1
- net INPUT7-: now also C21.1
- net INPUT8+: now also C24.1
- net INPUT8-: now also C23.1
Routing:
- net INPUT5-: track 125.3 -> 136.0 mm
- net INPUT5+: track 116.3 -> 125.3 mm
- net INPUT7+: track 77.3 -> 84.8 mm
- net INPUT7-: track 72.6 -> 80.0 mm
- net INPUT3-: track 74.4 -> 80.4 mm
- net INPUT6+: track 94.4 -> 99.8 mm
- net INPUT8-: track 43.1 -> 47.9 mm
- net INPUT3+: track 65.6 -> 69.5 mm
- net INPUT2+: track 98.9 -> 102.1 mm
- net INPUT1+: track 123.4 -> 126.4 mm
- net INPUT2-: track 102.9 -> 105.6 mm
- net INPUT4-: track 49.9 -> 52.5 mm
- net INPUT8+: track 45.9 -> 48.5 mm
- net INPUT4+: track 49.5 -> 52.0 mm
- net INPUT6-: track 104.7 -> 107.0 mm
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
Commit message: tarjeta_v18
Parts:
- added IC1, IC2, IC3, IC4, IC5, IC6, IC7, IC8: AD620R, analog-devices:SO8
- added R17, R18, R19, R20, R21, R22, R23, R24: 34.8, rcl:R0805
- added U$1: TMH2412D, TMH 2412D:TMH2412D
- moved C12 20.4 mm to (85.2, 48.1), turned to 180 degrees
- moved C16 18.4 mm to (25.0, 48.2), turned to 180 degrees
- moved C9 18.4 mm to (111.8, 48.2), turned to 180 degrees
- moved C4 16.1 mm to (31.6, 48.1)
- moved C1 14.7 mm to (104.8, 48.2)
- moved C3 14.7 mm to (51.5, 48.1)
- moved C2 14.6 mm to (78.4, 48.1)
- moved C6 14.5 mm to (76.9, 27.6), turned to 270 degrees
- moved R5 14.1 mm to (58.5, 48.1), turned to 0 degrees
- moved R2 12.9 mm to (101.6, 47.3)
- moved R8 12.9 mm to (21.6, 47.3)
- moved R3 12.8 mm to (81.9, 47.3)
- moved R1 12.8 mm to (108.6, 47.3)
- moved R6 12.8 mm to (48.2, 47.3)
- moved R7 12.8 mm to (28.5, 47.2)
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Connections:
- new net -12V: IC1.4, IC2.4, IC3.4, IC4.4, IC5.4, IC6.4, IC7.4, IC8.4, U$1.P$3
- new net N$17: IC1.8, R17.1
- new net N$18: IC1.1, R17.2
- new net N$19: IC3.1, R19.2
- new net N$20: IC3.8, R19.1
- new net N$21: IC2.1, R18.2
- new net N$22: IC2.8, R18.1
- new net N$23: IC4.8, R20.1
- new net N$24: IC4.1, R20.2
- new net N$25: IC5.8, R21.1
- new net N$26: IC5.1, R21.2
- new net N$27: IC6.1, R22.2
- new net N$28: IC6.8, R22.1
- new net N$29: IC7.1, R23.2
- new net N$30: IC7.8, R23.1
- new net N$33: IC8.8, R24.1
- new net N$34: IC8.1, R24.2
- new net SIG1+: C1.2, C10.1, IC1.3, R2.1
- new net SIG1-: C1.1, C9.1, IC1.2, R1.1
- new net SIG2+: C12.1, C2.2, IC2.3, R4.1
- new net SIG2-: C11.1, C2.1, IC2.2, R3.1
- new net SIG3+: C14.1, C3.2, IC3.3, R6.1
- new net SIG3-: C13.1, C3.1, IC3.2, R5.1
- new net SIG4+: C16.1, C4.2, IC4.3, R8.1
- new net SIG4-: C15.1, C4.1, IC4.2, R7.1
- new net SIG5+: C18.1, C5.2, IC5.3, R10.1
- new net SIG5-: C17.1, C5.1, IC5.2, R9.1
- new net SIG6+: C20.1, C6.2, IC6.3, R12.1
- new net SIG6-: C19.1, C6.1, IC6.2, R11.1
- new net SIG7+: C22.1, C7.2, IC7.3, R14.1
- new net SIG7-: C21.1, C7.1, IC7.2, R13.1
- new net SIG8+: C24.1, C8.2, IC8.3, R16.1
- new net SIG8-: C23.1, C8.1, IC8.2, R15.1
- net +12V: now also IC1.7, IC2.7, IC3.7, IC4.7, IC5.7, IC6.7, IC7.7, IC8.7, U$1.P$1
- net GND: now also IC1.5, IC2.5, IC3.5, IC4.5, IC5.5, IC6.5, IC7.5, IC8.5, JP1.2, U$1.P$2, U$1.P$4
- net INPUT1+: now also IC1.6; no longer C1.2, C10.1, R2.1
- net INPUT1-: no longer C1.1, C9.1, JP1.2, R1.1
- net INPUT2+: now also IC2.6; no longer C12.1, C2.2, R4.1
- net INPUT2-: no longer C11.1, C2.1, R3.1
- net INPUT3+: now also IC3.6; no longer C14.1, C3.2, R6.1
- net INPUT3-: no longer C13.1, C3.1, R5.1
- net INPUT4+: now also IC4.6; no longer C16.1, C4.2, R8.1
- net INPUT4-: no longer C15.1, C4.1, R7.1
- net INPUT5+: now also IC5.6; no longer C18.1, C5.2, R10.1
- net INPUT5-: no longer C17.1, C5.1, R9.1
- net INPUT6+: now also IC6.6; no longer C20.1, C6.2, R12.1
- net INPUT6-: no longer C19.1, C6.1, R11.1
- net INPUT7+: now also IC7.6, IC8.6; no longer C22.1, C7.2, R14.1
- net INPUT7-: no longer C21.1, C7.1, R13.1
- net INPUT8+: no longer C24.1, C8.2, R16.1
- net INPUT8-: no longer C23.1, C8.1, R15.1
Routing:
- net +12V: track 2.63 -> 160.8 mm, vias 0 -> 4
- net -12V: track 0.00 -> 133.7 mm, vias 0 -> 8
- net INPUT1-: track 123.7 -> 0.00 mm, vias 1 -> 0
- net SIG1-: track 0.00 -> 118.5 mm, vias 0 -> 2
- net SIG1+: track 0.00 -> 115.5 mm, vias 0 -> 2
- net SIG8+: track 0.00 -> 113.4 mm, vias 0 -> 2
- net INPUT5-: track 136.0 -> 24.8 mm, vias 1 -> 2
- net SIG8-: track 0.00 -> 97.5 mm, vias 0 -> 2
- net INPUT2-: track 105.6 -> 14.0 mm, vias 2 -> 0
- net INPUT1+: track 126.4 -> 37.6 mm, vias 1 -> 0
- net INPUT6-: track 107.0 -> 29.2 mm, vias 3 -> 2
- net SIG2-: track 0.00 -> 75.0 mm, vias 0 -> 2
- net SIG2+: track 0.00 -> 72.5 mm, vias 0 -> 3
- net INPUT7+: track 84.8 -> 149.2 mm, vias 1 -> 3
- net SIG7-: track 0.00 -> 63.0 mm
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Other:
- board text added: "Calle Kellogs N° 10, Fracc. Ind. El Pueblito, Corregidora, Querétaro CP: 76905 (442) 192 9600 | www.ipc.com.mx | www.win-systems.com"
- board text removed: "ver 1.0"

Commit message: tarjeta_v19
Parts:
- removed IC1, IC2, IC3, IC4, IC5, IC6, IC7, IC8: AD620R, analog-devices:SO8
- removed U$1: TMH2412D, TMH 2412D:TMH2412D
- added U1, U2, U3, U4, U5, U6, U7, U8: AD620ARZ-REEL7, AD620ARZ-REEL7:R_8_ADI
- R17, R18, R19, R20, R21, R22, R23, R24: value 34.8 -> 34R
- moved R24 148.7 mm to (12.1, -76.7), flipped to the top, turned to 0 degrees
- moved R23 140.6 mm to (7.00, -76.7), flipped to the top, turned to 0 degrees
- moved R22 137.1 mm to (1.88, -76.7), flipped to the top, turned to 0 degrees
- moved R21 112.6 mm to (19.9, -69.8), flipped to the top, turned to 0 degrees
- moved R20 91.1 mm to (7.00, -43.1), flipped to the top, turned to 0 degrees
- moved R19 84.5 mm to (1.88, -43.1), flipped to the top, turned to 0 degrees
- moved R18 61.8 mm to (1.88, -23.1), flipped to the top, turned to 0 degrees
- moved R17 43.0 mm to (1.88, -10.1), flipped to the top, turned to 0 degrees
- moved C12 20.4 mm to (76.2, 29.7), turned to 270 degrees
- moved C16 18.4 mm to (21.9, 30.0), turned to 270 degrees
- moved C9 18.4 mm to (108.1, 30.2), turned to 270 degrees
- moved C4 16.1 mm to (25.1, 33.4)
- moved C1 14.7 mm to (105.0, 33.5)
- moved C3 14.7 mm to (51.7, 33.5)
- moved C2 14.6 mm to (78.4, 33.5)
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Connections:
- removed net INPUT1-: JP2.2
- removed net INPUT10-: JP1.20, JP3.4
- removed net INPUT11-: JP1.22, JP3.6
- removed net INPUT12-: JP1.24, JP3.8
- removed net INPUT13-: JP1.26, JP3.10
- removed net INPUT14-: JP1.28, JP3.12
- removed net INPUT15-: JP1.30, JP3.14
- removed net INPUT16-: JP1.32, JP3.16
- removed net INPUT2-: JP1.4, JP2.4
- removed net INPUT3-: JP1.6, JP2.6
- removed net INPUT4-: JP1.8, JP2.8
- removed net INPUT5-: JP1.10, JP2.10
- removed net INPUT6-: JP1.12, JP2.12
- removed net INPUT7-: JP1.14, JP2.14
- removed net INPUT8-: JP1.16, JP2.16
- removed net INPUT9-: JP1.18, JP3.2
- removed net N$33: IC8.8, R24.1
- removed net N$34: IC8.1, R24.2
- new net N$31: R24.1, U8.1
- new net N$32: R24.2, U8.8
- net +12V: now also U1.7, U2.7, U3.7, U4.7, U5.7, U6.7, U7.7, U8.7; no longer IC1.7, IC2.7, IC3.7, IC4.7, IC5.7, IC6.7, IC7.7, IC8.7, U$1.P$1
- net -12V: now also U1.4, U2.4, U3.4, U4.4, U5.4, U6.4, U7.4, U8.4; no longer IC1.4, IC2.4, IC3.4, IC4.4, IC5.4, IC6.4, IC7.4, IC8.4, U$1.P$3
- net GND: now also JP1.10, JP1.12, JP1.14, JP1.16, JP1.18, JP1.20, JP1.22, JP1.24, JP1.26, JP1.28, JP1.30, JP1.32, JP1.4, JP1.6, JP1.8, JP2.10, JP2.12, JP2.14, JP2.16, JP2.2, JP2.4, JP2.6, JP2.8, JP3.10, JP3.12, JP3.14, JP3.16, JP3.2, JP3.4, JP3.6, JP3.8, U1.5, U2.5, U3.5, U4.5, U5.5, U6.5, U7.5, U8.5; no longer IC1.5, IC2.5, IC3.5, IC4.5, IC5.5, IC6.5, IC7.5, IC8.5, U$1.P$2, U$1.P$4
- net INPUT1+: now also U1.6; no longer IC1.6
- net INPUT2+: now also U2.6; no longer IC2.6
- net INPUT3+: now also U3.6; no longer IC3.6
- net INPUT4+: now also U4.6; no longer IC4.6
- net INPUT5+: now also U5.6; no longer IC5.6
- net INPUT6+: now also U6.6; no longer IC6.6
- net INPUT7+: now also U7.6; no longer IC7.6, IC8.6
- net INPUT8+: now also U8.6
- net N$17: now also U1.1; no longer IC1.8
- net N$18: now also U1.8; no longer IC1.1
- net N$19: now also R18.1, U2.1; no longer IC3.1, R19.2
- net N$20: now also R18.2, U2.8; no longer IC3.8, R19.1
- net N$21: now also R19.1, U3.1; no longer IC2.1, R18.2
- net N$22: now also R19.2, U3.8; no longer IC2.8, R18.1
- net N$23: now also U4.1; no longer IC4.8
- net N$24: now also U4.8; no longer IC4.1
- net N$25: now also U5.1; no longer IC5.8
- net N$26: now also U5.8; no longer IC5.1
- net N$27: now also R22.1, U6.1; no longer IC6.1, R22.2
- net N$28: now also R22.2, U6.8; no longer IC6.8, R22.1
- net N$29: now also R23.1, U7.1; no longer IC7.1, R23.2
- net N$30: now also R23.2, U7.8; no longer IC7.8, R23.1
- net SIG1+: now also U1.3; no longer IC1.3
- net SIG1-: now also U1.2; no longer IC1.2
- net SIG2+: now also U2.3; no longer IC2.3
- net SIG2-: now also U2.2; no longer IC2.2
- net SIG3+: now also U3.3; no longer IC3.3
- net SIG3-: now also U3.2; no longer IC3.2
- net SIG4+: now also U4.3; no longer IC4.3
- net SIG4-: now also U4.2; no longer IC4.2
- net SIG5+: now also U5.3; no longer IC5.3
- net SIG5-: now also U5.2; no longer IC5.2
- net SIG6+: now also U6.3; no longer IC6.3
- net SIG6-: now also U6.2; no longer IC6.2
- net SIG7+: now also U7.3; no longer IC7.3
- net SIG7-: now also U7.2; no longer IC7.2
- net SIG8+: now also U8.3; no longer IC8.3
- net SIG8-: now also U8.2; no longer IC8.2
Routing:
- net +5V: track 289.1 -> 0.00 mm, vias 3 -> 0
- net +12V: track 160.8 -> 0.00 mm, vias 4 -> 0
- net INPUT7+: track 149.2 -> 0.00 mm, vias 3 -> 0
- net -12V: track 133.7 -> 0.00 mm, vias 8 -> 0
- net SIG1-: track 118.5 -> 0.00 mm, vias 2 -> 0
- net SIG1+: track 115.5 -> 0.00 mm, vias 2 -> 0
- net SIG8+: track 113.4 -> 0.00 mm, vias 2 -> 0
- net INPUT6+: track 109.1 -> 0.00 mm, vias 2 -> 0
- net INPUT11+: track 104.6 -> 0.00 mm
- net INPUT15+: track 104.2 -> 0.00 mm, vias 1 -> 0
- net INPUT10+: track 104.1 -> 0.00 mm, vias 1 -> 0
- net INPUT9+: track 103.9 -> 0.00 mm, vias 1 -> 0
- net INPUT13+: track 103.5 -> 0.00 mm, vias 1 -> 0
- net INPUT14+: track 103.2 -> 0.00 mm, vias 1 -> 0
- net INPUT16+: track 102.9 -> 0.00 mm
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Other:
- board text added: "ver 1.0"
- board text removed: "Calle Kellogs N° 10, Fracc. Ind. El Pueblito, Corregidora, Querétaro CP: 76905 (442) 192 9600 | www.ipc.com.mx | www.win-systems.com"

Commit message: tarjeta_v21
Parts:
- added IC1: TRV1-1222M, TRV 1-1222M:TRV1-1222M
- C1, C2, C3, C4, C5, C6, C7, C8: value 0.1uF -> 4.7nF
- R1, R10, R11, R12, R13, R14, R15, R16, R2, R3, R4, R5, R6, R7, R8, R9: value 100R -> 300R
- moved U5 119.1 mm to (104.9, 12.3), flipped to the bottom, turned to 270 degrees
- moved R21 115.4 mm to (100.9, 12.5), flipped to the bottom, turned to 270 degrees
- moved R22 114.2 mm to (74.2, 11.7), flipped to the bottom, turned to 270 degrees
- moved U1 107.9 mm to (105.0, 32.8), flipped to the bottom, turned to 270 degrees
- moved R17 107.6 mm to (100.6, 32.7), flipped to the bottom, turned to 270 degrees
- moved U6 101.6 mm to (78.3, 11.8), flipped to the bottom, turned to 270 degrees
- moved R23 98.2 mm to (47.6, 12.6), flipped to the bottom, turned to 270 degrees
- moved R18 91.4 mm to (74.1, 32.8), flipped to the bottom, turned to 270 degrees
- moved U7 90.4 mm to (51.7, 12.6), flipped to the bottom, turned to 270 degrees
- moved U2 89.9 mm to (78.3, 32.7), flipped to the bottom, turned to 270 degrees
- moved R24 89.7 mm to (20.9, 12.6), flipped to the bottom, turned to 270 degrees
- moved R19 88.5 mm to (47.6, 32.7), flipped to the bottom, turned to 270 degrees
- moved U8 86.1 mm to (25.0, 12.5), flipped to the bottom, turned to 270 degrees
- moved U3 79.3 mm to (51.7, 32.7), flipped to the bottom, turned to 270 degrees
- moved R20 76.3 mm to (20.9, 32.0), flipped to the bottom, turned to 270 degrees
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Connections:
- net +12V: now also IC1.1, JP2.20, JP3.20
- net +5V: no longer JP2.20, JP3.20
- net -12V: now also IC1.7
- net GND: now also IC1.2, IC1.8
Routing:
- net +5V: track 0.00 -> 278.8 mm, vias 0 -> 1
- net +12V: track 0.00 -> 263.2 mm, vias 0 -> 4
- net -12V: track 0.00 -> 211.5 mm, vias 0 -> 1
- net INPUT9+: track 0.00 -> 137.0 mm
- net INPUT5+: track 0.00 -> 136.3 mm, vias 0 -> 1
- net INPUT1+: track 0.00 -> 121.9 mm, vias 0 -> 2
- net INPUT11+: track 0.00 -> 117.5 mm, vias 0 -> 1
- net INPUT10+: track 0.00 -> 114.3 mm, vias 0 -> 3
- net INPUT12+: track 0.00 -> 113.1 mm, vias 0 -> 3
- net INPUT13+: track 0.00 -> 105.4 mm, vias 0 -> 1
- net INPUT14+: track 0.00 -> 102.7 mm, vias 0 -> 1
- net INPUT16+: track 0.00 -> 101.9 mm, vias 0 -> 1
- net INPUT15+: track 0.00 -> 100.8 mm, vias 0 -> 2
- net INPUT2+: track 0.00 -> 99.4 mm, vias 0 -> 2
- net INPUT6+: track 0.00 -> 94.0 mm, vias 0 -> 2
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Other:
- board size 130 x 50 mm -> 140 x 50 mm
- board text added: "AGND"

Commit message: tarjeta_v22
Parts:
- removed R24: 34R, rcl:R0805
- added R25: 200R, 22AR200LFTR:RES3_22A_TTE
- R17, R18, R19, R20, R21, R22, R23: value 34R -> 200R; device rcl:R0805 -> 22AR200LFTR:RES3_22A_TTE
- moved R20 79.5 mm to (98.0, 12.6), turned to 0 degrees
- moved R22 30.1 mm to (44.1, 12.6), turned to 0 degrees
- moved R21 29.8 mm to (71.1, 14.6), turned to 0 degrees
- moved R23 29.4 mm to (18.2, 12.5), turned to 0 degrees
- moved R18 29.3 mm to (44.9, 32.8), turned to 0 degrees
- moved R19 29.2 mm to (18.4, 32.2), turned to 0 degrees
- moved R17 28.3 mm to (72.3, 32.7), turned to 0 degrees
Connections:
- net N$17: now also R25.1; no longer R17.1
- net N$18: now also R25.2, R25.3; no longer R17.2
- net N$19: now also R17.1; no longer R18.1
- net N$20: now also R17.2, R17.3; no longer R18.2
- net N$21: now also R18.1; no longer R19.1
- net N$22: now also R18.2, R18.3; no longer R19.2
- net N$23: now also R19.1; no longer R20.1
- net N$24: now also R19.2, R19.3; no longer R20.2
- net N$25: now also R20.1; no longer R21.1
- net N$26: now also R20.2, R20.3; no longer R21.2
- net N$27: now also R21.1; no longer R22.1
- net N$28: now also R21.2, R21.3; no longer R22.2
- net N$29: now also R22.1; no longer R23.1
- net N$30: now also R22.2, R22.3; no longer R23.2
- net N$31: now also R23.1; no longer R24.1
- net N$32: now also R23.2, R23.3; no longer R24.2
Routing:
- net N$28: track 3.07 -> 9.04 mm
- net N$30: track 2.75 -> 8.07 mm
- net N$26: track 2.90 -> 7.65 mm
- net N$22: track 2.93 -> 7.38 mm
- net N$24: track 3.07 -> 7.49 mm
- net N$32: track 2.88 -> 7.28 mm
- net N$18: track 3.06 -> 7.37 mm
- net N$20: track 3.11 -> 6.63 mm
- net N$29: track 5.00 -> 7.13 mm
- net N$27: track 2.88 -> 4.44 mm
- net -12V: track 211.5 -> 213.0 mm
- net N$25: track 2.75 -> 4.07 mm
- net N$31: track 2.86 -> 3.96 mm
- net N$21: track 2.93 -> 3.96 mm
- net INPUT6+: track 94.0 -> 93.3 mm
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