File: DATALOGGER_BP_V1/DATALOGGER_BP_V1.sch (EAGLE design)
At the start: 36 parts, among them J1 1985247, J2 1985247, J3 1985247, J4 1985247, J5 1985247, J6 1985247, J7 1985247, J8 1985247, J9 1755736

Commit message: tarjeta_v14
Connections:
- new net +12V: JP1.35, JP1.36
- new net INPUT10+: JP1.19, JP3.3
- new net INPUT10-: JP1.20, JP3.4
- new net INPUT11+: JP1.21, JP3.5
- new net INPUT11-: JP1.22, JP3.6
- new net INPUT12+: JP1.23, JP3.7
- new net INPUT12-: JP1.24, JP3.8
- new net INPUT13+: JP1.25, JP3.9
- new net INPUT13-: JP1.26, JP3.10
- new net INPUT14+: JP1.27, JP3.11
- new net INPUT14-: JP1.28, JP3.12
- new net INPUT15+: JP1.29, JP3.13
- new net INPUT15-: JP1.30, JP3.14
- new net INPUT16+: JP1.31, JP3.15
- new net INPUT16-: JP1.32, JP3.16
- new net INPUT9+: JP1.17, JP3.1
- new net INPUT9-: JP1.18, JP3.2
- net +5V: now also JP1.39, JP1.40, JP2.19, JP2.20, JP3.19, JP3.20
- net GND: now also JP1.33, JP1.34, JP1.37, JP1.38, JP2.17, JP2.18, JP3.17, JP3.18
- net GNDA: now also J9.1, J9.2
- net INPUT1+: now also JP1.1, JP2.1
- net INPUT1-: now also JP1.2, JP2.2
- net INPUT2+: now also JP1.3, JP2.3
- net INPUT2-: now also JP1.4, JP2.4
- net INPUT3+: now also JP1.5, JP2.5
- net INPUT3-: now also JP1.6, JP2.6
- net INPUT4+: now also JP1.7, JP2.7
- net INPUT4-: now also JP1.8, JP2.8
- net INPUT5+: now also JP1.9, JP2.9
- net INPUT5-: now also JP1.10, JP2.10
- net INPUT6+: now also JP1.11, JP2.11
- net INPUT6-: now also JP1.12, JP2.12
- net INPUT7+: now also JP1.13, JP2.13
- net INPUT7-: now also JP1.14, JP2.14
- net INPUT8+: now also JP1.15, JP2.15
- net INPUT8-: now also JP1.16, JP2.16

Commit message: tarjeta_v16
Parts:
- added C10, C11, C12, C13, C14, C15, C16, C17, C18, C19, C20, C21, C22, C23, C24, C9: 0.01uF, rcl:C-USC0805
Connections:
- net GND: now also C10.2, C11.2, C12.2, C13.2, C14.2, C15.2, C16.2, C17.2, C18.2, C19.2, C20.2, C21.2, C22.2, C23.2, C24.2, C9.2
- net INPUT1+: now also C10.1
- net INPUT1-: now also C9.1
- net INPUT2+: now also C12.1
- net INPUT2-: now also C11.1
- net INPUT3+: now also C14.1
- net INPUT3-: now also C13.1
- net INPUT4+: now also C16.1
- net INPUT4-: now also C15.1
- net INPUT5+: now also C18.1
- net INPUT5-: now also C17.1
- net INPUT6+: now also C20.1
- net INPUT6-: now also C19.1
- net INPUT7+: now also C22.1
- net INPUT7-: now also C21.1
- net INPUT8+: now also C24.1
- net INPUT8-: now also C23.1

Commit message: tarjeta_v18
Parts:
- added IC1, IC2, IC3, IC4, IC5, IC6, IC7, IC8: AD620R, analog-devices:AD620R
- added R17, R18, R19, R20, R21, R22, R23, R24: 34.8, rcl:R-US_R0805
- added U$1: TMH2412D, TMH 2412D:TMH2412D
Connections:
- new net -12V: IC1.-V, IC2.-V, IC3.-V, IC4.-V, IC5.-V, IC6.-V, IC7.-V, IC8.-V, U$1.-VOUT
- new net N$17: IC1.RG@2, R17.1
- new net N$18: IC1.RG@1, R17.2
- new net N$19: IC3.RG@1, R19.2
- new net N$20: IC3.RG@2, R19.1
- new net N$21: IC2.RG@1, R18.2
- new net N$22: IC2.RG@2, R18.1
- new net N$23: IC4.RG@2, R20.1
- new net N$24: IC4.RG@1, R20.2
- new net N$25: IC5.RG@2, R21.1
- new net N$26: IC5.RG@1, R21.2
- new net N$27: IC6.RG@1, R22.2
- new net N$28: IC6.RG@2, R22.1
- new net N$29: IC7.RG@1, R23.2
- new net N$30: IC7.RG@2, R23.1
- new net N$33: IC8.RG@2, R24.1
- new net N$34: IC8.RG@1, R24.2
- new net SIG1+: C1.2, C10.1, IC1.+, R2.1
- new net SIG1-: C1.1, C9.1, IC1.-, R1.1
- new net SIG2+: C12.1, C2.2, IC2.+, R4.1
- new net SIG2-: C11.1, C2.1, IC2.-, R3.1
- new net SIG3+: C14.1, C3.2, IC3.+, R6.1
- new net SIG3-: C13.1, C3.1, IC3.-, R5.1
- new net SIG4+: C16.1, C4.2, IC4.+, R8.1
- new net SIG4-: C15.1, C4.1, IC4.-, R7.1
- new net SIG5+: C18.1, C5.2, IC5.+, R10.1
- new net SIG5-: C17.1, C5.1, IC5.-, R9.1
- new net SIG6+: C20.1, C6.2, IC6.+, R12.1
- new net SIG6-: C19.1, C6.1, IC6.-, R11.1
- new net SIG7+: C22.1, C7.2, IC7.+, R14.1
- new net SIG7-: C21.1, C7.1, IC7.-, R13.1
- new net SIG8+: C24.1, C8.2, IC8.+, R16.1
- new net SIG8-: C23.1, C8.1, IC8.-, R15.1
- net +12V: now also IC1.+V, IC2.+V, IC3.+V, IC4.+V, IC5.+V, IC6.+V, IC7.+V, IC8.+V, U$1.VCC
- net GND: now also IC1.REF, IC2.REF, IC3.REF, IC4.REF, IC5.REF, IC6.REF, IC7.REF, IC8.REF, JP1.2, U$1.COMMON, U$1.GND
- net INPUT1+: now also IC1.OUT; no longer C1.2, C10.1, R2.1
- net INPUT1-: no longer C1.1, C9.1, JP1.2, R1.1
- net INPUT2+: now also IC2.OUT; no longer C12.1, C2.2, R4.1
- net INPUT2-: no longer C11.1, C2.1, R3.1
- net INPUT3+: now also IC3.OUT; no longer C14.1, C3.2, R6.1
- net INPUT3-: no longer C13.1, C3.1, R5.1
- net INPUT4+: now also IC4.OUT; no longer C16.1, C4.2, R8.1
- net INPUT4-: no longer C15.1, C4.1, R7.1
- net INPUT5+: now also IC5.OUT; no longer C18.1, C5.2, R10.1
- net INPUT5-: no longer C17.1, C5.1, R9.1
- net INPUT6+: now also IC6.OUT; no longer C20.1, C6.2, R12.1
- net INPUT6-: no longer C19.1, C6.1, R11.1
- net INPUT7+: now also IC7.OUT, IC8.OUT; no longer C22.1, C7.2, R14.1
- net INPUT7-: no longer C21.1, C7.1, R13.1
- net INPUT8+: no longer C24.1, C8.2, R16.1
- net INPUT8-: no longer C23.1, C8.1, R15.1

Commit message: tarjeta_v19
Parts:
- removed IC1, IC2, IC3, IC4, IC5, IC6, IC7, IC8: AD620R, analog-devices:AD620R
- removed U$1: TMH2412D, TMH 2412D:TMH2412D
- added U1, U2, U3, U4, U5, U6, U7, U8: AD620ARZ-REEL7, AD620ARZ-REEL7:AD620ARZ-REEL7
- R17, R18, R19, R20, R21, R22, R23, R24: value 34.8 -> 34R
Connections:
- removed net INPUT1-: JP2.2
- removed net INPUT10-: JP1.20, JP3.4
- removed net INPUT11-: JP1.22, JP3.6
- removed net INPUT12-: JP1.24, JP3.8
- removed net INPUT13-: JP1.26, JP3.10
- removed net INPUT14-: JP1.28, JP3.12
- removed net INPUT15-: JP1.30, JP3.14
- removed net INPUT16-: JP1.32, JP3.16
- removed net INPUT2-: JP1.4, JP2.4
- removed net INPUT3-: JP1.6, JP2.6
- removed net INPUT4-: JP1.8, JP2.8
- removed net INPUT5-: JP1.10, JP2.10
- removed net INPUT6-: JP1.12, JP2.12
- removed net INPUT7-: JP1.14, JP2.14
- removed net INPUT8-: JP1.16, JP2.16
- removed net INPUT9-: JP1.18, JP3.2
- removed net N$33: IC8.RG@2, R24.1
- removed net N$34: IC8.RG@1, R24.2
- new net N$31: R24.1, U8.RG_2
- new net N$32: R24.2, U8.RG
- net +12V: now also U1.+VS, U2.+VS, U3.+VS, U4.+VS, U5.+VS, U6.+VS, U7.+VS, U8.+VS; no longer IC1.+V, IC2.+V, IC3.+V, IC4.+V, IC5.+V, IC6.+V, IC7.+V, IC8.+V, U$1.VCC
- net -12V: now also U1.-VS, U2.-VS, U3.-VS, U4.-VS, U5.-VS, U6.-VS, U7.-VS, U8.-VS; no longer IC1.-V, IC2.-V, IC3.-V, IC4.-V, IC5.-V, IC6.-V, IC7.-V, IC8.-V, U$1.-VOUT
- net GND: now also JP1.10, JP1.12, JP1.14, JP1.16, JP1.18, JP1.20, JP1.22, JP1.24, JP1.26, JP1.28, JP1.30, JP1.32, JP1.4, JP1.6, JP1.8, JP2.10, JP2.12, JP2.14, JP2.16, JP2.2, JP2.4, JP2.6, JP2.8, JP3.10, JP3.12, JP3.14, JP3.16, JP3.2, JP3.4, JP3.6, JP3.8, U1.REF, U2.REF, U3.REF, U4.REF, U5.REF, U6.REF, U7.REF, U8.REF; no longer IC1.REF, IC2.REF, IC3.REF, IC4.REF, IC5.REF, IC6.REF, IC7.REF, IC8.REF, U$1.COMMON, U$1.GND
- net INPUT1+: now also U1.OUTPUT; no longer IC1.OUT
- net INPUT2+: now also U2.OUTPUT; no longer IC2.OUT
- net INPUT3+: now also U3.OUTPUT; no longer IC3.OUT
- net INPUT4+: now also U4.OUTPUT; no longer IC4.OUT
- net INPUT5+: now also U5.OUTPUT; no longer IC5.OUT
- net INPUT6+: now also U6.OUTPUT; no longer IC6.OUT
- net INPUT7+: now also U7.OUTPUT; no longer IC7.OUT, IC8.OUT
- net INPUT8+: now also U8.OUTPUT
- net N$17: now also U1.RG_2; no longer IC1.RG@2
- net N$18: now also U1.RG; no longer IC1.RG@1
- net N$19: now also R18.1, U2.RG_2; no longer IC3.RG@1, R19.2
- net N$20: now also R18.2, U2.RG; no longer IC3.RG@2, R19.1
- net N$21: now also R19.1, U3.RG_2; no longer IC2.RG@1, R18.2
- net N$22: now also R19.2, U3.RG; no longer IC2.RG@2, R18.1
- net N$23: now also U4.RG_2; no longer IC4.RG@2
- net N$24: now also U4.RG; no longer IC4.RG@1
- net N$25: now also U5.RG_2; no longer IC5.RG@2
- net N$26: now also U5.RG; no longer IC5.RG@1
- net N$27: now also R22.1, U6.RG_2; no longer IC6.RG@1, R22.2
- net N$28: now also R22.2, U6.RG; no longer IC6.RG@2, R22.1
- net N$29: now also R23.1, U7.RG_2; no longer IC7.RG@1, R23.2
- net N$30: now also R23.2, U7.RG; no longer IC7.RG@2, R23.1
- net SIG1+: now also U1.+IN; no longer IC1.+
- net SIG1-: now also U1.-IN; no longer IC1.-
- net SIG2+: now also U2.+IN; no longer IC2.+
- net SIG2-: now also U2.-IN; no longer IC2.-
- net SIG3+: now also U3.+IN; no longer IC3.+
- net SIG3-: now also U3.-IN; no longer IC3.-
- net SIG4+: now also U4.+IN; no longer IC4.+
- net SIG4-: now also U4.-IN; no longer IC4.-
- net SIG5+: now also U5.+IN; no longer IC5.+
- net SIG5-: now also U5.-IN; no longer IC5.-
- net SIG6+: now also U6.+IN; no longer IC6.+
- net SIG6-: now also U6.-IN; no longer IC6.-
- net SIG7+: now also U7.+IN; no longer IC7.+
- net SIG7-: now also U7.-IN; no longer IC7.-
- net SIG8+: now also U8.+IN; no longer IC8.+
- net SIG8-: now also U8.-IN; no longer IC8.-

Commit message: tarjeta_v21
Parts:
- added IC1: TRV1-1222M, TRV 1-1222M:TRV1-1222M
- C1, C2, C3, C4, C5, C6, C7, C8: value 0.1uF -> 4.7nF
- R1, R10, R11, R12, R13, R14, R15, R16, R2, R3, R4, R5, R6, R7, R8, R9: value 100R -> 300R
Connections:
- net +12V: now also IC1.VCC, JP2.20, JP3.20
- net +5V: no longer JP2.20, JP3.20
- net -12V: now also IC1.-VOUT
- net GND: now also IC1.COM, IC1.GND

Commit message: tarjeta_v22
Parts:
- removed R24: 34R, rcl:R-US_R0805
- added R25: 200R, 22AR200LFTR:22AR200LFTR
- R17, R18, R19, R20, R21, R22, R23: value 34R -> 200R; device rcl:R-US_R0805 -> 22AR200LFTR:22AR200LFTR
Connections:
- net N$17: now also R25.1; no longer R17.1
- net N$18: now also R25.2, R25.3; no longer R17.2
- net N$19: now also R17.1; no longer R18.1
- net N$20: now also R17.2, R17.3; no longer R18.2
- net N$21: now also R18.1; no longer R19.1
- net N$22: now also R18.2, R18.3; no longer R19.2
- net N$23: now also R19.1; no longer R20.1
- net N$24: now also R19.2, R19.3; no longer R20.2
- net N$25: now also R20.1; no longer R21.1
- net N$26: now also R20.2, R20.3; no longer R21.2
- net N$27: now also R21.1; no longer R22.1
- net N$28: now also R21.2, R21.3; no longer R22.2
- net N$29: now also R22.1; no longer R23.1
- net N$30: now also R22.2, R22.3; no longer R23.2
- net N$31: now also R23.1; no longer R24.1
- net N$32: now also R23.2, R23.3; no longer R24.2
